File: pcb/PULSER/PULSER.kicad_pcb (KiCad board)
At the start: 4 copper layers, 150 x 100 mm, 125 parts, among them J1 Screw_Terminal 2pin, J2 XH 2pin, J4 Screw_Terminal 2pin, J5 Screw_Terminal 2pin, J6 FFC 8pin, J8 Socket 20pin, 2.54mm, J9 Socket 20pin, 2.54mm, Q14 N-ch, Vds>=200V, fast switch,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, Q15 N-ch, Vds>=200V, fast switch,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, Q16 N-ch, Vds>=200V, fast switch,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, Q17 N-ch, Vds>=200V, fast switch,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, Q2 N-ch, Vds>=60V, fast switch, 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, Q6 N-ch, Vds>=60V, fast switch, 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, Q7 N-ch, Vds>=200V, fast switch,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, Q8 N-ch, Vds>=200V, fast switch,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, U1 LM5104MX/NOPB, U10 IR2104S, U12 TMP102, U2 L78M05ABDT, U3 ACS724LLCTR-30AU, U4 LT8365, U5 IR2104S, U6 REF3030, U8 IR2104S

Commit message: Fix missing 5V input
Connections:
- C3 pad 1: /Regulator 5V/VIN -> +12V
- L4 pad 3: GND -> (no net)
- U2 pad 1: /Regulator 5V/VIN -> +12V
Routing:
- net +12V: track 258.6 -> 266.0 mm
- net /Regulator 5V/VIN: track 2.24 -> 0.00 mm

Commit message: r4 DRC pass
Parts:
- removed J6: FFC 8pin, SparkAll:Molex_Connector_8pin_P1mm_526100872
- removed TP22, TP37, TP38, TP40, TP41, TP43, TP44: TestPoint_Small, TestPoint:TestPoint_Pad_D1.5mm
- added C14: 10uF 50V, Capacitor_SMD:C_1206_3216Metric, F.Cu at (136.6, 62.9)
- added C19: 100nF 50V, Capacitor_SMD:C_0603_1608Metric, F.Cu at (159.5, 84.5)
- added C27: 100nF 50V, Capacitor_SMD:C_0603_1608Metric, F.Cu at (159.5, 86.0)
- added C28: 10uF 50V, Capacitor_SMD:C_1206_3216Metric, F.Cu at (136.6, 65.3)
- added C31: 10uF 50V, Capacitor_SMD:C_1206_3216Metric, F.Cu at (145.0, 62.9)
- added C32: 10uF 50V, Capacitor_SMD:C_1206_3216Metric, F.Cu at (145.0, 65.3)
- added C33: 1nF 50V, Capacitor_SMD:C_0603_1608Metric, F.Cu at (166.9, 93.5)
- added C34: 1nF 50V, Capacitor_SMD:C_0603_1608Metric, F.Cu at (152.0, 86.2)
- added FB1: FerriteBead_Small, Inductor_SMD:L_0603_1608Metric, F.Cu at (81.7, 60.7)
- added FB2: FerriteBead_Small, Inductor_SMD:L_0603_1608Metric, F.Cu at (84.3, 60.7)
- added J7: XH 3pin, Connector_JST:JST_XH_B3B-XH-AM_1x03_P2.50mm_Vertical, F.Cu at (81.7, 54.6)
- added Q18: N-ch, Vds>=200V, fast switch, low Rds, SparkAll:Infineon-TG-TDSON-8-NMOS, F.Cu at (175.8, 88.9)
- added Q19: N-ch, Vds>=200V, fast switch, low Rds, SparkAll:Infineon-TG-TDSON-8-NMOS, F.Cu at (175.9, 121.9)
- added Q20: N-ch, Vds>=200V, fast switch, low Rds, SparkAll:Infineon-TG-TDSON-8-NMOS, F.Cu at (185.0, 88.9)
- added Q21: N-ch, Vds>=200V, fast switch, low Rds, SparkAll:Infineon-TG-TDSON-8-NMOS, F.Cu at (184.9, 121.9)
- added R32: 10, Resistor_SMD:R_0603_1608Metric, F.Cu at (187.2, 75.0)
- added R33: 10, Resistor_SMD:R_0603_1608Metric, F.Cu at (186.2, 109.7)
- added R34: 10, Resistor_SMD:R_0603_1608Metric, F.Cu at (178.6, 85.3)
- added R35: 10, Resistor_SMD:R_0603_1608Metric, F.Cu at (178.4, 118.2)
- added R36: 1, Resistor_SMD:R_1210_3225Metric, F.Cu at (167.0, 90.4)
- added R37: 1, Resistor_SMD:R_1210_3225Metric, F.Cu at (152.0, 89.6)
- moved TP27 49.3 mm to (168.3, 74.5)
- moved C30 21.9 mm to (178.2, 80.6), turned to -90 degrees
- moved U3 21.0 mm to (182.7, 81.3)
- moved C29 20.8 mm to (177.4, 82.9)
- moved C11 18.7 mm to (157.1, 77.0), turned to 0 degrees
- moved C10 18.7 mm to (157.2, 79.5), turned to 0 degrees
- moved TP24 16.7 mm to (171.3, 74.7)
- moved TP13 16.1 mm to (53.3, 99.1)
- moved Q15 15.1 mm to (184.9, 113.5)
- moved JP1 14.8 mm to (190.6, 117.7)
- moved Q14 14.7 mm to (175.9, 113.5)
- moved TP30 13.7 mm to (168.3, 71.8)
- moved Q2 13.7 mm to (162.4, 91.2), turned to -90 degrees
- moved R16 13.1 mm to (159.0, 104.9), turned to 0 degrees
- moved C15 12.7 mm to (153.0, 99.5), turned to 180 degrees
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Connections:
- J8 pad 4: /DCHG_GATE -> unconnected-(J8-Pin_4-Pad4)
- L4 pad 3: (no net) -> GND
Routing:
- net +12V: track 266.0 -> 315.6 mm, vias 9 -> 8
- net /DCHG_GATE: track 49.2 -> 0.00 mm, vias 1 -> 0
- net Net-(Q14-PadG): track 29.7 -> 2.42 mm, vias 3 -> 0
- net /Mux/VC_L: track 126.6 -> 153.9 mm
- net /Mux/V+: track 30.0 -> 4.98 mm
- net Net-(Q16-PadG): track 26.2 -> 1.70 mm
- net /Mux/V-: track 36.5 -> 12.3 mm
- net Net-(U10-HO): track 5.71 -> 29.5 mm, vias 0 -> 3
- net +5V: track 101.5 -> 122.8 mm
- net Net-(Q6-PadG): track 19.8 -> 41.0 mm, vias 0 -> 3
- net Net-(C33-Pad2): track 32.8 -> 12.6 mm
- net Net-(Q15-PadG): track 22.0 -> 5.19 mm, vias 3 -> 2
- net Net-(D6-K): track 20.7 -> 4.76 mm, vias 2 -> 0
- net Net-(U1-LO): track 15.6 -> 2.09 mm, vias 2 -> 0
- net Net-(D2-A-Pad1): track 22.5 -> 9.00 mm
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Other:
- board text added: "SCL"
- board text added: "SDA"
- board text removed: "Type-A cable"
- board text removed: "pin 1"

Commit message: LGTM
Parts:
- moved TP20 2.80 mm to (66.2, 63.6)
- moved TP18 2.29 mm to (66.3, 58.2)
- moved TP29 0.68 mm to (155.2, 68.8)
- moved R29 0.28 mm to (179.1, 110.0)
- moved R35 0.13 mm to (178.4, 118.4)
Routing:
- net Net-(Q2-PadG): track 41.2 -> 34.2 mm
- net +12V: track 315.6 -> 319.5 mm
- net /I2C_SDA: track 39.9 -> 37.7 mm
- net /Mux/V0_L: track 173.8 -> 174.8 mm
- net Net-(C10-Pad1): track 4.12 -> 3.35 mm
- net GND: vias 328 -> 486

Commit message: Bump revision to r4
Other:
- board text added: "PULSER r4"
- board text removed: "PULSER r3"
Changed lines of the file:
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@@
 	(title_block
 		(title "PULSER")
-		(date "2025-03-28")
-		(rev "3")
+		(date "2025-08-06")
+		(rev "4")
 		(company "Spark Project")
 		(comment 1 "Author: 夕月霞 (xyx)")
@@
 		)
 	)
-	(gr_text "PULSER r3"
+	(gr_text "PULSER r4"
 		(at 69.596 142.748 0)
 		(layer "F.SilkS")

Commit message: Increase current path width
Routing:
- net GND: vias 486 -> 489
Changed lines of the file:
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@@
 			"kPIBAABwptJq/H8AAAC742r8fwAAcKbSavx/AABwptJq/H8AAHCm0mr8fwAAKLPjavx/AAAwsHzT"
 			"8gEAACiz42r8fwAAAPMpkPIBAAAw8ymQ8gEAAHCWKZDyAQAA0Lrjavx/AABg8ymQ8gEAAHCm0mr8"
-			"fwAAkLvjavx/AAAwu+Nq/H8AAHCm0mr8fwAAcKbSavx/AABwptJq/H8AAHCm0mr8fwAAkA=="
+			"fwAAkLvjavx/AAAwu+Nq/H8AAHCm0mr8fwAAcKbSavx/AABwptJq/H8AAHCm0mr8fwAAkL13P4IA"
+			"CH8lJCT/Ozs7/wAAAAAAAAAAmDQWwKmH2L+YhglAggAIfyUkJP87Ozv/AAAAAAAAAACYNBbAqYfY"
+			"P5iGCUCCAAh/JSQk/zs7O/8AAAAAAAAAAOaRG8BGQuM/z713P4IACH8lJCT/Ozs7/wAAAAAAAAAA"
+			"SdcQwAzNzT+YhglAAAB/f7CpmP+rqqf/AAAAAAAAAAAe9NS/DM3NP5iGCUAAAH9/sKmY/6uqp/8A"
+			"AAAAAAAAAEnXEMAMzc0/mIYJQAAAf3+wqZj/q6qn/wAAAAAAAAAAHvTUvwzNzT+YhglAAAB/f7Cp"
+			"mP+rqqf/AAAAAAAAAAAe9NS/DM3NP5iGCUAAAH9/sKmY/6uqp/8AAAAAAAAAAEnXEMAMzc0/mIYJ"
+			"QAAAf3+wqZj/q6qn/wAAAAAAAAAAHvTUvwzNzT+YhglAAAB/f7CpmP+rqqf/AAAAAAAAAAAe9NS/"
+			"DM3Nv5iGCUAAAH9/sKmY/6uqp/8AAAAAAAAAAB701L8Mzc0/mIYJQAAAf3+wqZj/q6qn/wAAAAAA"
+			"AAAAHvTUvwzNzb+YhglAAAB/f7CpmP+rqqf/AAAAAAAAAAAe9NS/DM3Nv5iGCUAAAH9/sKmY/6uq"
+			"p/8AAAAAAAAAAB701L8Mzc0/mIYJQAAAf3+wqZj/q6qn/wAAAAAAAAAAHvTUvwzNzb+YhglAAAB/"
+			"f7CpmP+rqqf/AAAAAAAAAABJ1xDADM3Nv5iGCUAAAH9/sKmY/6uqp/8AAAAAAAAAAB701L8Mzc2/"
+			"mIYJQAAAf3+wqZj/q6qn/wAAAAAAAAAASdcQwAzNzb+YhglAAAB/f7CpmP+rqqf/AAAAAAAAAABJ"
+			"1xDADM3Nv5iGCUAAAH9/sKmY/6uqp/8AAAAAAAAAAB701L8Mzc2/mIYJQAAAf3+wqZj/q6qn/wAA"
+			"AAAAAAAASdcQwAzNzb+YhglAAAB/f7CpmP+rqqf/AAAAAAAAAABJ1xDADM3NP5iGCUAAAH9/sKmY"
+			"/6uqp/8AAAAAAAAAAEnXEMAMzc2/mIYJQAAAf3+wqZj/q6qn/wAAAAAAAAAASdcQwAzNzT+YhglA"
+			"AAB/f7CpmP+rqqf/AAAAAAAAAABJ1xDADM3NP5iGCUAAAH9/sKmY/6uqp/8AAAAAAAAAAEnXEMAM"
+			"zc2/mIYJQAAAf3+wqZj/q6qn/wAAAAAAAAAASdcQwAzNzT+YhglAAAB/f7CpmP+rqqf/AAAAAAAA"
+			"AABJ1xDADM3Nv5iGCUAAAH9/sKmY/6uqp/8AAAAAAAAAAB701L8Mzc0/mIYJQAAAf3+wqZj/q6qn"
+			"/wAAAAAAAAAASdcQwAzNzb+YhglAAAB/f7CpmP+rqqf/AAAAAAAAAAAe9NS/DM3Nv5iGCQ=="
 		)
 	)
@@
 	)
 	(via
+		(at 155.448 59.436)
+		(size 0.6)
+		(drill 0.3)
+		(layers "F.Cu" "B.Cu")
+		(free yes)
+		(net 3)
+	)
+	(via
 		(at 198.12 60.96)
 		(size 0.6)
@@
 	)
 	(via
-		(at 183.658 74.422)
+		(at 183.658 73.787)
 		(size 0.6)
 		(drill 0.3)
@@
 	)
 	(via
+		(at 157.734 59.436)
+		(size 0.6)
+		(drill 0.3)
+		(layers "F.Cu" "B.Cu")
+		(free yes)
+		(net 3)
+	)
+	(via
 		(at 96.52 96.52)
 		(size 0.6)
@@
 	)
 	(via
-		(at 182.762253 79.192575)
+		(at 181.737 79.375)
 		(size 0.6)
 		(drill 0.3)
@@
 	)
 	(via
-		(at 176.779913 79.267667)
+		(at 177.419 78.994)
 		(size 0.6)
 		(drill 0.3)
@@
 	)
 	(via
+		(at 159.893 59.436)
+		(size 0.6)
+		(drill 0.3)
+		(layers "F.Cu" "B.Cu")
+		(free yes)
+		(net 3)
+	)
+	(via
 		(at 116.84 106.68)
 		(size 0.6)
@@
 			(pts
 				(xy 154.5 65) (xy 154.5 50) (xy 190 50) (xy 190 60) (xy 200 60) (xy 200 90) (xy 195 90) (xy 195 65)
-				(xy 185 65) (xy 185 65)
+				(xy 185 65)
 			)
 		)
@@
 				(xy 154.94 60.579) (xy 145.288 60.579) (xy 145.288 66.675) (xy 157.48 66.675) (xy 157.48 82.042)
 				(xy 159.893 83.82) (xy 159.893 86.487) (xy 161.417 86.868) (xy 161.417 88.392) (xy 165.227 88.392)
-				(xy 176.911 78.359) (xy 183.642 78.359) (xy 183.642 81.026) (xy 186.182 81.026) (xy 185.928 74.93)
-				(xy 174.879 74.93) (xy 173.101 76.454) (xy 166.581666 82.042) (xy 163.322 82.042) (xy 162.56 81.28)
+				(xy 177.165 78.486) (xy 182.372 78.359) (xy 183.642 81.026) (xy 187.198 81.026) (xy 186.055 74.676)
+				(xy 175.175333 74.676) (xy 173.101 76.454) (xy 166.581666 82.042) (xy 163.322 82.042) (xy 162.56 81.28)
 				(xy 162.56 70.358) (xy 168 65) (xy 165 61)
 			)
@@
 				(xy 187.96 118.618) (xy 187.96 112.522) (xy 189.23 112.522) (xy 189.23 110.363) (xy 187.96 110.363)
 				(xy 187.96 96.266) (xy 189.23 96.266) (xy 189.23 94.107) (xy 187.96 94.107) (xy 187.96 87.757) (xy 189.357 87.757)
-				(xy 189.357 85.471) (xy 187.96 85.471) (xy 183.642 83.581875) (xy 183.642 81.28) (xy 193.294 81.788)
+				(xy 189.357 85.471) (xy 186.817 85.471) (xy 183.642 83.581875) (xy 183.642 81.534) (xy 193.294 81.788)
 				(xy 193.167 126.365) (xy 183.007 128.143)
 			)
