File: pcb/PULSER/PULSER.kicad_pcb (KiCad board)
At the start: 4 copper layers, 150 x 100 mm, 138 parts, among them J1 Screw_Terminal 2pin, J2 XH 2pin, J4 Screw_Terminal 2pin, J5 Screw_Terminal 2pin, J7 XH 3pin, J8 Socket 20pin, 2.54mm, J9 Socket 20pin, 2.54mm, Q14 N-ch, Vds>=200V, fast switch,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, Q15 N-ch, Vds>=200V, fast switch,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, Q16 N-ch, Vds>=200V, fast switch,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, Q17 N-ch, Vds>=200V, fast switch,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, Q18 N-ch, Vds>=200V, fast switch,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, Q19 N-ch, Vds>=200V, fast switch,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, Q2 N-ch, Vds>=60V, fast switch, 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, Q20 N-ch, Vds>=200V, fast switch,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, Q21 N-ch, Vds>=200V, fast switch,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, Q6 N-ch, Vds>=60V, fast switch, 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, Q7 N-ch, Vds>=200V, fast switch,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, Q8 N-ch, Vds>=200V, fast switch,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, U1 LM5104MX/NOPB, U10 IR2104S, U12 TMP102, U2 L78M05ABDT, U3 ACS724LLCTR-30AU, U4 LT8365, U5 IR2104S, U6 REF3030, U8 IR2104S

Commit message: (crit) Insert resistor to 100V line / (minor) Fix small diode foorprint
Parts:
- removed C6: 1uF 200V, Capacitor_SMD:C_1812_4532Metric
- added R2: 200, Resistor_SMD:R_2512_6332Metric, F.Cu at (135.0, 137.9)
- D10, D4, D6: footprint Diode_SMD:D_SOD-323 -> SparkAll:D_SOD-323HE
- moved C5 19.1 mm to (127.3, 139.8)
- moved NT4 16.0 mm to (121.2, 137.8)
- moved TP23 7.87 mm to (144.9, 140.0)
- moved C23 0.13 mm to (130.8, 124.5)
Connections:
- L4 pad 3: (no net) -> GND
- Q7 pad D: Net-(C5-Pad1) -> Net-(Q7-PadD)
- TP23 pad 1: Net-(C5-Pad1) -> Net-(Q7-PadD)
Routing:
- net /Pulse Shaper/Boost Converter 100V/VOUT: track 31.0 -> 13.6 mm
- net Net-(Q7-PadD): track 0.00 -> 9.98 mm
- net Net-(C5-Pad1): track 5.30 -> 8.86 mm
- net GND: vias 489 -> 484
- removed copper zone on F.Cu, net Net-(C5-Pad1)
Other:
- board text added: "PULSER r5"
- board text removed: "PULSER r4"
