File: pcb/PULSER/PULSER.kicad_sch (KiCad schematic)
At the start: 27 parts, among them J1 Screw_Terminal 2pin, J2 XH 2pin, J4 Screw_Terminal 2pin, J5 Screw_Terminal 2pin, J6 FFC 8pin, U12 TMP102

Commit message: Fix missing 5V input
Other:
- sheet Regulator 5V ports: added VIN; removed none
Changed lines of the file:
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@@
 			"eXkyVDUiDQoJCQkiTURkc0grMkJUWGU0WThjWUQxeGc0a0hIYVl6WHc3T3hQYmtZZncxMVJTdzdC"
 			"LzNkN3JFZWlKcmh5OTF0SkpCS3A5Mm14R0s4RTVHTiINCgkJCSJCNW1WRThmYWJtYlhFenJCQ3hl"
-			"bithS1FXVVlQSDYwUDBpdjVrYjNXeU9rK0RRcTVEWFZCZVVrbHduWmRnWXVYTFhlaERaLw=="
+			"bithS1FXVVlQSDYwUDBpdjVrYjNXeU9rK0RRcTVEWFZCZVVrbHduWmRnWXVYTFhlaERaLxGWCD1w"
+			"L8j4EwIAAAAAAJCEuSoeAgAA2THYsHe+J92A8gEAAAAAAJyF2yoeAgAA2JGJXCDTptlw4QAAAAAA"
+			"APBvvCoeAgAA2TH77JqVhV7AbwEAAAAAANBnuSoeAgAA2RF2nfIbvZNwkwEAAAAAAMC9rioeAgAA"
+			"21G6U6jf3q7w7QEAAAAAAMDIrioeAgAA2xEJz1YNeFDA3wEAAAAAAOyG2yoeAgAA3NHnTlUJCXBQ"
+			"4gAAAAAAANCDkCoeAgAA3dGZvZyhb5/gSgIAAAAAAIDJwyoeAgAA9JEpMmwhqgfAPQMAAAAAAJCg"
+			"uSoeAgAA7vGuJL5R9a+4NAMAAAAAAPCJwyoeAgAA7LGspHuZt/QYBgMAAAAAADz52yoeAgAA4REF"
+			"FOu30BnIrAEAAAAAABBnwyoeAgAA6dHqFK73FvOA6AIAAAAAAJwb3CoeAgAA8FFo+PX1vrxA2QIA"
+			"AAAAAJBTtyoeAgAA5LG16m4PUxzQOwEAAAAAAEDTpyoeAgAA5pGXZdsYTFl4ogAAAAAAAFC0qioe"
+			"AgAA5tE9ODfnThuwIgAAAAAAADwQ3CoeAgAA8PFAZA2TH6QgNwIAAAAAAOD+eyoeAgAA61Groo80"
+			"NKHQ/gAAAAAAADBKvCoeAgAA6nGjRbkCOrvYXgEAAAAAAADyZSoeAgAA6vFm4LyYGgzwZQEAAAAA"
+			"ALDPqioeAgAA65FMie6Hy3roQAAAAAAAAEDBrioeAgAA7FHaYMYyacdoBAIAAAAAAID9eyoeAgAA"
+			"7dE88pcS8YPw7gAAAAAAACDNtSoeAgAA7lF0dveSfmrIMQEAAAAAADBzuSoeAgAA7zEn5tepuqqo"
+			"igEAAAAAANCGuSoeAgAA8BHZ/F1iUQeQ1gEAAAAAAMC1vSoeAgAA8lHzkzXVEO4YpQIAAAAAAEym"
+			"2yoeAgAA8rFH/D1YoeQw1wAAAAAAACBhvioeAgAA89Hpmg8YbsygZAIAAAAAAKACfCoeAgAA9FFM"
+			"v5rW+vWYLgEAAAAAABDfwyoeAgAA+NHYnAjk6b5oYQMAAAAAAFC0wyoeAgAAAfLHZvmVO12ILwMA"
+			"AAAAAMB1vioeAgAA/LHXwrCfdklwfQIAAAAAADBuuSoeAgAA+DEox6gYB8VIiQEAAAAAAIBQuioe"
+			"AgAA+pFn2RbzHQbohAAAAAAAAJD2ZSoeAgAA+vHsvS3dMFWQggEAAAAAANyv2yoeAgAA+/FqT1+M"
+			"N/GQ3QAAAAAAAICDuioeAgAAAdLH+qHzDm9IvgAAAAAAADDxuioeAgAA/hHFTlOquAxQ9wAAAAAA"
+			"ABBXuioeAgAA/jEnnGfkxMVwiwAAAAAAACCDuioeAgAAAfKiEZ5uQjaYtAAAAAAAAADcrg=="
 		)
 	)
@@
 			)
 		)
+		(pin "VIN" input
+			(at 50.8 59.69 180)
+			(effects
+				(font
+					(size 1.27 1.27)
+				)
+				(justify left)
+			)
+		)

Commit message: EMI (ferrite for I2C). Simplify I2C signal
Parts:
- removed J6: FFC 8pin, SparkAll:Molex_Connector_8pin_P1mm_526100872, symbol Connector:Conn_01x08_Pin
- removed TP22: TestPoint_Small, TestPoint:TestPoint_Pad_D1.5mm, symbol Connector:TestPoint_Small
- added FB1, FB2: FerriteBead_Small, Inductor_SMD:L_0603_1608Metric, symbol Device:FerriteBead_Small
- added J7: XH 3pin, Connector_JST:JST_XH_B3B-XH-AM_1x03_P2.50mm_Vertical, symbol Connector:Conn_01x03_Pin
Connections:
- net GND: now also J7.3 (Pin_3)
- net I2C_SCL: now also FB2.2
- net I2C_SDA: now also FB1.2
- new net: FB1.1, J7.1 (Pin_1)
- new net: FB2.1, J7.2 (Pin_2)
- no-connect marks 1 -> 0
Other:
- sheet Pico2 ports: added none; removed M_GATE
- note added: "All signals are 3.3V digital"
- note removed: "1 2 3 4 5 6 7 8"
- note removed: "GND"
- note removed: "Pins are flipped for Type A (Same-side) cable. All signals are 3.3V digital"
- note removed: "VSYS (5V)"
- note removed: "pins in CTRL-MINI"
- moved on the sheet: TP18, TP20
