File: pcb/PULSER/mux_half_bridge.kicad_sch (KiCad schematic)
At the start: 12 parts, among them Q16 N-ch, Vds>=200V, fast switch,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, Q17 N-ch, Vds>=200V, fast switch,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, U10 IR2104S

Commit message: EMI reduction & heatsink simplification
EMI: MOSFET snubber, 36V pi-filter
heatsink: Parallel mux bridge
Parts:
- added Q18, Q20: N-ch, Vds>=200V, fast switch, low Rds, SparkAll:Infineon-TG-TDSON-8-NMOS, symbol Device:Q_NMOS
- added R32, R34: 10, Resistor_SMD:R_0603_1608Metric, symbol Device:R
Connections:
- net V+: now also Q18.D
- net V-: now also Q20.S
- net VOUT: now also Q18.S, Q20.D
- net at R30.2, U10.5 (LO): now also R32.2
- net at R28.2, U10.7 (HO): now also R34.2
- new net: Q18.G, R34.1
- new net: Q20.G, R32.1
Other:
- note removed: "Parts Height To make heatsink (shim) attachment easier, make sure all parts (other than the IC) is shorter than MOSFETs. BSC110N15NS5: 1.05mm UCC27288DR: 1.75mm CL10A105KB8NNNC (1uF 50V, 0603): 0.8mm CC0603KRX7R9BB104 (100nF 50V, 0603): 0.8mm RB168VAM150TR (150V diode, SOD-323): 0.6mm"
- moved on the sheet: C24, D10, R28, TP37, U10

Commit message: EMI (ferrite for I2C). Simplify I2C signal
Parts:
- TP37, TP40, TP43: now not fitted
Changed lines of the file:
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@@
 			"//8A////AP///wD///8A////AP///wD///8A////AP///wD///8A////AP///wD///8A////AP//"
 			"/wD///8A////AP///wD///8A////AP///wD///8A////AP///wD///8A////AP///wD///8A////"
-			"AP///wD///8A////AP///wD///8A////AP///wD///8A////AP///wD///8A////AP///w=="
+			"AP///wD///8A////AP///wD///8A////AP///wD///8A////AP///wD///8A////AP///wAAAAAA"
+			"AAAAAAAAAAAAAAAAAAAAAAAAAAAAAAAAAAAAAAAAAAAAAAAAAAAAAAAAAAAAAAAAAAAAAAAAAAAA"
+			"AAAAAAAAAAAAAAAAAAAAAAAAAAAAAAAAAAAAAAAAAAAAAAAAAAAAAAAAAAAAAAAAAAAAAAAAAAAA"
+			"AAAAAAAAAAAAAAAAAAAAAAAAAAAAAAAAAAAAAAAAAAAAAAAAAAAAAAAAAAAAAAAAAAAAAAAAAAAA"
+			"AAAAAAAAAAAAAAAAAAAAAAAAAAAAAAAAAAAAAAAAAAAAAAAAAAAAAAAAAAAAAAAAAAAAAAAAAAAA"
+			"AAAAAAAAAAAAAAAAAAAAAAAAAAAAAAAAAAAAAAAAAAAAAAAAAAAAAAAAAAAAAAAAAAAAAAAAAAAA"
+			"AAAAAAAAAAAAAAAAAAAAAAAAAAAAAAAAAAAAAAAAAAAAAAAAAAAAAAAAAAAAAAAAAAAAAAAAAAAA"
+			"AAAAAAAAAAAAAAAAAAAAAAAAAAAAAAAAAAAAAAAAAAAAAAAAAAAAAAAAAAAAAAAAAAAAAAAAAAAA"
+			"AAAAAAAAAAAAAAAAAAAAAAAAAAAAAAAAAAAAAAAAAAAAAAAAAAAAAAAAAAAAAAAAAAAAAAAAAAAA"
+			"AAAAAAAAAAAAAAAAAAAAAAAAAAAAAAAAAAAAAAAAAAAAAAAAAAAAAAAAAAAAAAAAAAAAAAAAAAAA"
+			"AAAAAAAAAAAAAAAAAAAAAAAAAAAAAAAAAAAAAAAAAAAAAAAAAAAAAAAAAAAAAAAAAAAAAAAAAAAA"
+			"AAAAAAAAAAAAAAAAAAAAAAAAAAAAAAAAAAAAAAAAAAAAAAAAAAAAAAAAAAAAAAAAAAAAAAAAAAAA"
+			"AAAAAAAAAAAAAAAAAAAAAAAAAAAAAAAAAAAAAAAAAAAAAAAAAAAAAAAAAAAAAAAAAAAAAAAAAAAA"
+			"AAAAAAAAAAAAAAAAAAAAAAAAAAAAAAAAAAAAAAAAAAAAAAAAAAAAAAAAAAAAAAAAAAAAAAAAAAAA"
+			"AAAAAAAAAAAAAAAAAAAAAAAAAAAAAAAAAAAAAAAAAAAAAAAAAAAAAAAAAAAAAAAAAAAAAAAAAAAA"
+			"AAAAAAAAAAAAAAAAAAAAAAAAAAAAAAAAAAAAAAAAAAAAAAAAAAAAAAAAAAAAAAAAAAAAAAAAAAAA"
+			"AAAAAAAAAAAAAAAAAAAAAAAAAAAAAAAAAAAAAAAAAAAAAAAAAAAAAAAAAAAAAAAAAAAAAAAAAAAA"
+			"AAAAAAAAAAAAAAAAAAAAAAAAAAAAAAAAAAAAAAAAAAAAAAAAAAAAAAAAAAAAAAAAAAAAAAAAAAAA"
+			"AAAAAAAAAAAAAAAAAAAAAAAAAAAAAAAAAAAAAAAAAAAAAAAAAAAAAAAAAAAAAAAAAAAAAA=="
 		)
 	)
@@
 		(exclude_from_sim no)
 		(in_bom no)
-		(on_board yes)
-		(dnp no)
+		(on_board no)
+		(dnp yes)
 		(property "Reference" "TP37"
 			(at 91.186 73.914 0)
@@
 		(exclude_from_sim no)
 		(in_bom no)
-		(on_board yes)
-		(dnp no)
+		(on_board no)
+		(dnp yes)
 		(property "Reference" "TP40"
 			(at 118.872 69.088 0)
@@
 		(exclude_from_sim no)
 		(in_bom no)
-		(on_board yes)
-		(dnp no)
+		(on_board no)
+		(dnp yes)
 		(property "Reference" "TP43"
 			(at 118.872 95.504 0)

Commit message: Fix mux MOSFET LCSC ids
Parts:
- Q16, Q17, Q18, Q20: LCSC C501501 -> C412739
Changed lines of the file:
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@@
 			"AAAAAAAAAAAAAAAAAAAAAAAAAAAAAAAAAAAAAAAAAAAAAAAAAAAAAAAAAAAAAAAAAAAAAAAAAAAA"
 			"AAAAAAAAAAAAAAAAAAAAAAAAAAAAAAAAAAAAAAAAAAAAAAAAAAAAAAAAAAAAAAAAAAAAAAAAAAAA"
-			"AAAAAAAAAAAAAAAAAAAAAAAAAAAAAAAAAAAAAAAAAAAAAAAAAAAAAAAAAAAAAAAAAAAAAA=="
+			"AAAAAAAAAAAAAAAAAAAAAAAAAAAAAAAAAAAAAAAAAAAAAAAAAAAAAAAAAAAAAAAAAAAAAL13P4IA"
+			"CH8lJCT/Ozs7/wAAAAAAAAAAmDQWwKmH2L+YhglAggAIfyUkJP87Ozv/AAAAAAAAAACYNBbAqYfY"
+			"P5iGCUCCAAh/JSQk/zs7O/8AAAAAAAAAAOaRG8BGQuM/z713P4IACH8lJCT/Ozs7/wAAAAAAAAAA"
+			"SdcQwAzNzT+YhglAAAB/f7CpmP+rqqf/AAAAAAAAAAAe9NS/DM3NP5iGCUAAAH9/sKmY/6uqp/8A"
+			"AAAAAAAAAEnXEMAMzc0/mIYJQAAAf3+wqZj/q6qn/wAAAAAAAAAAHvTUvwzNzT+YhglAAAB/f7Cp"
+			"mP+rqqf/AAAAAAAAAAAe9NS/DM3NP5iGCUAAAH9/sKmY/6uqp/8AAAAAAAAAAEnXEMAMzc0/mIYJ"
+			"QAAAf3+wqZj/q6qn/wAAAAAAAAAAHvTUvwzNzT+YhglAAAB/f7CpmP+rqqf/AAAAAAAAAAAe9NS/"
+			"DM3Nv5iGCUAAAH9/sKmY/6uqp/8AAAAAAAAAAB701L8Mzc0/mIYJQAAAf3+wqZj/q6qn/wAAAAAA"
+			"AAAAHvTUvwzNzb+YhglAAAB/f7CpmP+rqqf/AAAAAAAAAAAe9NS/DM3Nv5iGCUAAAH9/sKmY/6uq"
+			"p/8AAAAAAAAAAB701L8Mzc0/mIYJQAAAf3+wqZj/q6qn/wAAAAAAAAAAHvTUvwzNzb+YhglAAAB/"
+			"f7CpmP+rqqf/AAAAAAAAAABJ1xDADM3Nv5iGCUAAAH9/sKmY/6uqp/8AAAAAAAAAAB701L8Mzc2/"
+			"mIYJQAAAf3+wqZj/q6qn/wAAAAAAAAAASdcQwAzNzb+YhglAAAB/f7CpmP+rqqf/AAAAAAAAAABJ"
+			"1xDADM3Nv5iGCUAAAH9/sKmY/6uqp/8AAAAAAAAAAB701L8Mzc2/mIYJQAAAf3+wqZj/q6qn/wAA"
+			"AAAAAAAASdcQwAzNzb+YhglAAAB/f7CpmP+rqqf/AAAAAAAAAABJ1xDADM3NP5iGCUAAAH9/sKmY"
+			"/6uqp/8AAAAAAAAAAEnXEMAMzc2/mIYJQAAAf3+wqZj/q6qn/wAAAAAAAAAASdcQwAzNzT+YhglA"
+			"AAB/f7CpmP+rqqf/AAAAAAAAAABJ1xDADM3NP5iGCUAAAH9/sKmY/6uqp/8AAAAAAAAAAEnXEMAM"
+			"zc2/mIYJQAAAf3+wqZj/q6qn/wAAAAAAAAAASdcQwAzNzT+YhglAAAB/f7CpmP+rqqf/AAAAAAAA"
+			"AABJ1xDADM3Nv5iGCUAAAH9/sKmY/6uqp/8AAAAAAAAAAB701L8Mzc0/mIYJQAAAf3+wqZj/q6qn"
+			"/wAAAAAAAAAASdcQwAzNzb+YhglAAAB/f7CpmP+rqqf/AAAAAAAAAAAe9NS/DM3Nv5iGCQ=="
 		)
 	)
@@
 			)
 		)
-		(property "LCSC" "C501501"
+		(property "LCSC" "C412739"
 			(at 147.32 67.31 0)
 			(effects
@@
 			)
 		)
-		(property "LCSC" "C501501"
+		(property "LCSC" "C412739"
 			(at 128.27 93.98 0)
 			(effects
@@
 			)
 		)
-		(property "LCSC" "C501501"
+		(property "LCSC" "C412739"
 			(at 147.32 93.98 0)
 			(effects
@@
 			)
 		)
-		(property "LCSC" "C501501"
+		(property "LCSC" "C412739"
 			(at 128.27 67.31 0)
 			(effects

Commit message: (crit) Insert resistor to 100V line / (minor) Fix small diode foorprint
Parts:
- D10: footprint Diode_SMD:D_SOD-323 -> SparkAll:D_SOD-323HE
Changed lines of the file:
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@@
 	(title_block
 		(title "PULSER")
-		(date "2025-08-06")
-		(rev "4")
+		(date "2025-11-12")
+		(rev "5")
 		(company "Spark Project")
 		(comment 1 "Author: 夕月霞 (xyx)")
@@
 			"zc2/mIYJQAAAf3+wqZj/q6qn/wAAAAAAAAAASdcQwAzNzT+YhglAAAB/f7CpmP+rqqf/AAAAAAAA"
 			"AABJ1xDADM3Nv5iGCUAAAH9/sKmY/6uqp/8AAAAAAAAAAB701L8Mzc0/mIYJQAAAf3+wqZj/q6qn"
-			"/wAAAAAAAAAASdcQwAzNzb+YhglAAAB/f7CpmP+rqqf/AAAAAAAAAAAe9NS/DM3Nv5iGCQ=="
+			"/wAAAAAAAAAASdcQwAzNzb+YhglAAAB/f7CpmP+rqqf/AAAAAAAAAAAe9NS/DM3Nv5iGCQAAAAAA"
+			"AAAAAAAAAAAAAAAAAAAAAAAAAAAAAAAAAAAAAAAAAAAAAAAAAAAAAAAAAAAAAAAAAAAAAAAAAAAA"
+			"AAAAAAAAAAAAAAAAAAAAAAAAAAAAAAAAAAAAAAAAAAAAAAAAAAAAAAAAAAAAAAAAAAAAAAAAAAAA"
+			"AAAAAAAAAAAAAAAAAAAAAAAAAAAAAAAAAAAAAAAAAAAAAAAAAAAAAAAAAAAAAAAAAAAAAAAAAAAA"
+			"AAAAAAAAAAAAAAAAAAAAAAAAAAAAAAAAAAAAAAAAAAAAAAAAAAAAAAAAAAAAAAAAAAAAAAAAAAAA"
+			"AAAAAAAAAAAAAAAAAAAAAAAAAAAAAAAAAAAAAAAAAAAAAAAAAAAAAAAAAAAAAAAAAAAAAAAAAAAA"
+			"AAAAAAAAAAAAAAAAAAAAAAAAAAAAAAAAAAAAAAAAAAAAAAAAAAAAAAAAAAAAAAAAAAAAAAAAAAAA"
+			"AAAAAAAAAAAAAAAAAAAAAAAAAAAAAAAAAAAAAAAAAAAAAAAAAAAAAAAAAAAAAAAAAAAAAAAAAAAA"
+			"AAAAAAAAAAAAAAAAAAAAAAAAAAAAAAAAAAAAAAAAAAAAAAAAAAAAAAAAAAAAAAAAAAAAAAAAAAAA"
+			"AAAAAAAAAAAAAAAAAAAAAAAAAAAAAAAAAAAAAAAAAAAAAAAAAAAAAAAAAAAAAAAAAAAAAAAAAAAA"
+			"AAAAAAAAAAAAAAAAAAAAAAAAAAAAAAAAAAAAAAAAAAAAAAAAAAAAAAAAAAAAAAAAAAAAAAAAAAAA"
+			"AAAAAAAAAAAAAAAAAAAAAAAAAAAAAAAAAAAAAAAAAAAAAAAAAAAAAAAAAAAAAAAAAAAAAAAAAAAA"
+			"AAAAAAAAAAAAAAAAAAAAAAAAAAAAAAAAAAAAAAAAAAAAAAAAAAAAAAAAAAAAAAAAAAAAAAAAAAAA"
+			"AAAAAAAAAAAAAAAAAAAAAAAAAAAAAAAAAAAAAAAAAAAAAAAAAAAAAAAAAAAAAAAAAAAAAAAAAAAA"
+			"AAAAAAAAAAAAAAAAAAAAAAAAAAAAAAAAAAAAAAAAAAAAAAAAAAAAAAAAAAAAAAAAAAAAAAAAAAAA"
+			"AAAAAAAAAAAAAAAAAAAAAAAAAAAAAAAAAAAAAAAAAAAAAAAAAAAAAAAAAAAAAAAAAAAAAAAAAAAA"
+			"AAAAAAAAAAAAAAAAAAAAAAAAAAAAAAAAAAAAAAAAAAAAAAAAAAAAAAAAAAAAAAAAAAAAAAAAAAAA"
+			"AAAAAAAAAAAAAAAAAAAAAAAAAAAAAAAAAAAAAAAAAAAAAAAAAAAAAAAAAAAAAAAAAAAAAAAAAAAA"
+			"AAAAAAAAAAAAAAAAAAAAAAAAAAAAAAAAAAAAAAAAAAAAAAAAAAAAAAAAAAAAAAAAAAAAAA=="
 		)
 	)
@@
 			)
 		)
-		(property "Footprint" "Diode_SMD:D_SOD-323"
+		(property "Footprint" "SparkAll:D_SOD-323HE"
 			(at 76.2 69.85 0)
 			(effects
