File: pcb/PULSER/relay_mux.kicad_sch (KiCad schematic)
At the start: 0 parts

Commit message: EMI reduction & heatsink simplification
EMI: MOSFET snubber, 36V pi-filter
heatsink: Parallel mux bridge
Other:
- note added: "4W heat output Passive heatsink or no heatsink 1.1W x 4 = 4.4W On Power: (20A/2)^2 x 11mΩ = 1.1W"
- note removed: "9W heat output 4.4W x 2 = 8.8W height=1.0mm (area: 6.1x5.3), RΘJC=1C/W On Power: 20A^2 x 11mΩ = 4.4W"
Changed lines of the file:
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@@
 		)
 	)
-	(text "9W heat output\n\n4.4W x 2 = 8.8W\nheight=1.0mm (area: 6.1x5.3), RΘJC=1C/W\nOn Power: 20A^2 x 11mΩ = 4.4W\n"
+	(text "4W heat output\nPassive heatsink or no heatsink\n\n1.1W x 4 = 4.4W\nOn Power: (20A/2)^2 x 11mΩ = 1.1W\n"
 		(exclude_from_sim no)
 		(at 180.848 29.464 0)
@@
 			"AAAAAAAAAAAAAAAAAAAAAAAAAAAAAAAAAAAAAAAAAAAAAAAAAAAAAAAAAAAAAAAAAAAAAAAAAAAA"
 			"AAAAAAAAAAAAAAAAAAAAAAAAAAAAAAAAAAAAAAAAAAAAAAAAAAAAAAAAAAAAAAAAAAAAAAAAAAAA"
-			"AAAAAAAAAAAAAAAAAAAAAAAAAAAAAAAAAAAAAAAAAAAAAAAAAAAAAAAAAAAAAAAAAAAAAA=="
-		)
-	)
+			"AAAAAAAAAAAAAAAAAAAAAAAAAAAAAAAAAAAAAAAAAAAAAAAAAAAAAAAAAAAAAAAAAAAAAN7yAQAA"
+			"qxArggAHBYAAAAAAAAAAAEp8+I4AAAAA0Pwo3vIBAAClEC2CAAgFgOe0sOaYjumrlC1FeHRCAAAA"
+			"AAAAAAAAAKcQL4IACQWAAAAAAAAAAABtr+tvAAAAADAAKd7yAQAAoRAhggAKBYAGAAAAEAAAAKAC"
+			"4P//////AAAAAAAAAACjECOCAAsFgE1pY3Jvc29mdCBKaGVuZ0hlaQAAAAAAAL0QJYIADAWA5b6u"
+			"6Luf5q2j6buR6auUAAAAAAAAAAAAvxAnggANBYBOb3JtYWFsaQAAAAAAAAAAAAAAAAAAAAC5EDmC"
+			"AA4FgFN0YW5kYXJkAAAAAAAAAAAAAAAAAAAAALsQO4IADwWABgAAABAAAABQ9t///////wAAAAAA"
+			"AAAAtRA9ggAQBYBHcmFzc2V0dG8AAAAAAAAAAAAAAAAAAAC3ED+CABEFgG9iecSNZWpuw6kAAAAA"
+			"AAAAAAAAAAAAALEQMYIAEgWA77yt77yzIOOCtOOCt+ODg+OCrwAAAAAAsxAzggATBYAGAAAAEAAA"
+			"AOAH4P//////AAAAAAAAAACNEDWCABQFgAYAAAAQAAAAANnf//////8AAAAAAAAAAI8QN4IAFQWA"
+			"BgAAABAAAADAK+D//////wAAAAAAAAAAiRBJggAWBYBvYnnEjWVqbsOpAAAAAAAAAAAAAAAAAACL"
+			"EEuCABcFgEbDqWxrw7Z2w6lyAAAAAAAAAAAAAAAAAIUQTYIAGAWAU3RhbmRhcmQAAAAAAAAAAAAA"
+			"AAAAAAAAhxBPggAZBYDQntCx0YvRh9C90YvQuQAAAAAAAAAAAACBEEGCABoFgE15YW5tYXIgVGV4"
+			"dAAAAAAAAAAAAAAAAIMQQ4IAGwWATGloYXZvaXR1AAAAAAAAAAAAAAAAAAAAnRBFggAcBYBTdGFu"
+			"ZGFhcmQAAAAAAAAAAAAAAAAAAACfEEeCAB0FgAAAAAAAAAAABUSvhAAAAAAQAine8gEAAJkQWYIA"
+			"HgWAAAAAAAAAAACH/Ic5AAAAAHABKd7yAQAAmxBbggAfBYAAAAAAAAAAABBKWqQAAAAA8Pso3vIB"
+			"AACVEF2CACAFgAAAAAAAAAAA0vxhvAAAAABw/Sje8gEAAJcQX4IAIQWAUG9ncnViaW9ueQAAAAAA"
+			"AAAAAAAAAAAAkRBRggAiBYBOb3JtYWxueQAAAAAAAAAAAAAAAAAAAACTEFOCACMFgFN0YW5kYWFy"
+			"ZAAAAAAAAAAAAAAAAAAAAG0PVYIAJAWATm9ybcOhbG5lAAAAAAAAAAAAAAAAAAAAbw9XggAlBYAG"
+			"AAAAEAAAAFDN3///////AAAAAAAAAABpD2mCACYFgFBNaW5nTGlVLUV4dEIAAAAAAAAAAA=="
+		)
+	)
