File: pcb/PULSER/pulse_shaper.kicad_sch (KiCad schematic)
At the start: 46 parts, among them Q2 N-ch, Vds>=60V, fast switch, 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, Q6 N-ch, Vds>=60V, fast switch, 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, Q7 N-ch, Vds>=200V, fast switch,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, Q8 N-ch, Vds>=200V, fast switch,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, U1 LM5104MX/NOPB, U3 ACS724LLCTR-30AU, U5 IR2104S

Commit message: EMI reduction & heatsink simplification
EMI: MOSFET snubber, 36V pi-filter
heatsink: Parallel mux bridge
Parts:
- added C14, C28, C31, C32: 10uF 50V, Capacitor_SMD:C_1206_3216Metric, symbol Device:C
- added C19, C27: 100nF 50V, Capacitor_SMD:C_0603_1608Metric, symbol Device:C
- added C33, C34: 1nF 50V, Capacitor_SMD:C_0603_1608Metric, symbol Device:C
- added R36, R37: 1, Resistor_SMD:R_1210_3225Metric, symbol Device:R
Connections:
- net GND: now also C14.2, C19.1, C27.1, C28.2, C31.2, C32.2, R36.2
- net VPWR: now also C14.1, C28.1, C31.1, C32.1
- net at L4.2, NT6.1, Q2.D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: now also C33.2, R37.2
- net at C10.1, C11.1, C12.1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: now also C19.2, C27.2, C34.2
- new net: C34.1, R37.1
- new net: C33.1, R36.1
Other:
- note added: "P=1nF x (36V)^2 x 500kHz = 0.6W"

Commit message: (crit) Insert resistor to 100V line / (minor) Fix small diode foorprint
Parts:
- removed C6: 1uF 200V, Capacitor_SMD:C_1812_4532Metric, symbol Device:C
- added R2: 200, Resistor_SMD:R_2512_6332Metric, symbol Device:R
- D4: footprint Diode_SMD:D_SOD-323 -> SparkAll:D_SOD-323HE
Connections:
- net at Q7.D, TP23.1: now also R2.2; no longer C5.1, NT4.2
- new net: C5.1, NT4.2, R2.1
Other:
- moved on the sheet: C5

Commit message: Add alternative LCSC no
Parts:
- D2: LCSC C2845075 -> C180497
Other:
- note added: "L1 (PCB layout & height compatible) * Sumida 125CDMCCDS-1R0MC * BOURNS SRP1245A-1R0M L4 (probably PCB layout compatible) * Ruishen RSPQ2918-100M * FANGCHENG FC-SE2915-100M D2 * STMicro STPS40170CG-TR D12 * onsemi 1SMB5951BT3G (Vz=120V instead of 130V) Q7,Q7 * infineon BSC350N20NSFD (almost same) * infineon BSC13DN30NSFD (VDS=300V instead of 200V)"
- note removed: "L1 (PCB layout & height compatible) * Sumida 125CDMCCDS-1R0MC * BOURNS SRP1245A-1R0M L4 (probably PCB layout compatible) * Ruishen RSPQ2918-100M * FANGCHENG FC-SE2915-100M D2 * STMicro STPS40170CG-TR D12 * onsemi 1SMB5951BT3G (Vz=120V instead of 130V)"
Changed lines of the file:
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@@
 		)
 	)
-	(text "L1 (PCB layout & height compatible)\n* Sumida 125CDMCCDS-1R0MC\n* BOURNS SRP1245A-1R0M\n\nL4 (probably PCB layout compatible)\n* Ruishen RSPQ2918-100M\n* FANGCHENG FC-SE2915-100M\n\nD2\n* STMicro STPS40170CG-TR\n\nD12\n* onsemi 1SMB5951BT3G (Vz=120V instead of 130V)"
+	(text "L1 (PCB layout & height compatible)\n* Sumida 125CDMCCDS-1R0MC\n* BOURNS SRP1245A-1R0M\n\nL4 (probably PCB layout compatible)\n* Ruishen RSPQ2918-100M\n* FANGCHENG FC-SE2915-100M\n\nD2\n* STMicro STPS40170CG-TR\n\nD12\n* onsemi 1SMB5951BT3G (Vz=120V instead of 130V)\n\nQ7,Q7\n* infineon BSC350N20NSFD (almost same)\n* infineon BSC13DN30NSFD (VDS=300V instead of 200V)"
 		(exclude_from_sim no)
 		(at 231.902 107.696 0)
@@
 			)
 		)
-		(property "LCSC" "C2845075"
+		(property "LCSC" "C180497"
 			(at 157.48 69.85 0)
 			(effects
