File: pcb/PULSER-testboard-hc/PULSER-testboard-hc.kicad_pcb (KiCad board)
At the start: 4 copper layers, 100 x 100 mm, 68 parts, among them J1 Screw_Terminal 2pin, J2 Screw_Terminal 2pin, J3 Conn_01x02_Pin, J4 Conn_01x02_Pin, Q1 N-ch, Vds>=60V, low Qgs, Q2 N-ch, Vds>=60V, low Rds, U1 LT3741-1, U2 LM317_DPAK

Commit message: HC test board pcb draft ok
Parts:
- added C17: 10n, Capacitor_SMD:C_0603_1608Metric, F.Cu at (124.2, 94.0)
- added C18: 10n, Capacitor_SMD:C_0603_1608Metric, F.Cu at (124.2, 91.0)
- added G***: LOGO, LOGO, F.Cu at (128.9, 132.3)
- added JP7: Jumper_2_Small_Bridged, Jumper:SolderJumper-2_P1.3mm_Bridged_RoundedPad1.0x1.5mm, F.Cu at (127.3, 94.0)
- added JP8: Jumper_2_Small_Bridged, Jumper:SolderJumper-2_P1.3mm_Bridged_RoundedPad1.0x1.5mm, F.Cu at (127.3, 91.0)
- added R23: thermal, Resistor_SMD:R_1225_3264Metric, F.Cu at (109.8, 87.0)
- added TP10: TestPoint, TestPoint:TestPoint_Pad_D1.5mm, F.Cu at (89.9, 86.7)
- added TP11: TestPoint, TestPoint:TestPoint_Pad_D1.5mm, F.Cu at (90.8, 117.0)
- added TP12: TestPoint, TestPoint:TestPoint_Pad_D1.5mm, F.Cu at (57.0, 117.0)
- added TP13: TestPoint, TestPoint:TestPoint_Pad_D1.5mm, F.Cu at (57.0, 109.5)
- added TP14: TestPoint, TestPoint:TestPoint_Pad_D1.5mm, F.Cu at (79.0, 117.0)
- added TP9: TestPoint, TestPoint:TestPoint_Pad_D1.5mm, F.Cu at (89.9, 90.2)
- moved TP7 135.8 mm to (57.0, 104.0)
- moved TP8 110.2 mm to (77.0, 146.0)
- moved TP5 99.2 mm to (93.0, 102.5)
- moved J3 97.6 mm to (108.5, 146.0), turned to 90 degrees
- moved R11 92.5 mm to (104.7, 140.0)
- moved J4 92.2 mm to (87.5, 146.0), turned to 90 degrees
- moved TP1 90.1 mm to (96.0, 102.5)
- moved R12 81.2 mm to (96.0, 140.8), turned to 90 degrees
- moved C8 78.5 mm to (98.8, 140.0), turned to 180 degrees
- moved D3 78.4 mm to (94.3, 136.7)
- moved TP4 74.0 mm to (143.0, 86.5)
- moved TP6 70.0 mm to (143.0, 93.5)
- moved D1 57.3 mm to (124.8, 62.4), turned to 180 degrees
- moved L1 55.5 mm to (128.4, 109.0)
- moved HS1 55.4 mm to (122.6, 65.8)
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Connections:
- net Net-(U1-SENSE+) renamed /SENSE+
- net Net-(U1-SENSE-) renamed /SENSE-
- C15 pad 1: Net-(C15-Pad1) -> GND
- C16 pad 1: Net-(C15-Pad1) -> GND
- C5 pad 2: Net-(JP2-A) -> Net-(JP2-B)
- R18 pad 2: Net-(C15-Pad1) -> GND
Routing:
- net Net-(D1-A): track 0.00 -> 99.7 mm
- net +36V: track 0.00 -> 98.8 mm
- net +3V3: track 0.00 -> 96.3 mm, vias 0 -> 4
- net /CTRL1: track 0.00 -> 92.3 mm, vias 0 -> 2
- net Net-(U1-SW): track 0.00 -> 79.3 mm, vias 0 -> 2
- net Net-(U1-FB): track 0.00 -> 78.9 mm, vias 0 -> 2
- net /EN: track 0.00 -> 67.8 mm, vias 0 -> 2
- net /VREF: track 0.00 -> 65.2 mm, vias 0 -> 3
- net /SENSE+: track 0.00 -> 61.8 mm, vias 0 -> 2
- net /SENSE-: track 0.00 -> 59.7 mm, vias 0 -> 2
- net Net-(JP2-B): track 0.00 -> 49.0 mm, vias 0 -> 2
- net Net-(JP3-B): track 0.00 -> 44.1 mm
- net Net-(U1-LG): track 0.00 -> 32.1 mm, vias 0 -> 3
- net Net-(D1-K): track 0.00 -> 27.2 mm
- net GND: track 0.00 -> 25.6 mm, vias 0 -> 187
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- added copper zone on F.Cu, net +36V
- added copper zone on F.Cu, net +3V3
- added copper zone on B.Cu, net GND
- added copper zone on F.Cu, net GND
- added copper zone on In1.Cu, net GND
- added copper zone on In2.Cu, net GND
- added copper zone on F.Cu, net Net-(C1-Pad2)
- added copper zone on F.Cu, net Net-(C4-Pad2)
- added copper zone on F.Cu, net Net-(D1-A)
- added copper zone on F.Cu, net Net-(D1-K)
- added copper zone on F.Cu, net Net-(J1-Pin_2)
- added copper zone on F.Cu, net Net-(L1-Pad2)
- added copper zone on F.Cu, net Net-(U1-SW)
Other:
- board text added: "+"
- board text added: "-"
- board text added: "10A"
- board text added: "10uH"
- board text added: "2A"
- board text added: "5A"
- board text added: "CTRL2"
- board text added: "CTRL_EXT"
- board text added: "EN_OVR"
- board text added: "GND"
- board text added: "HC Test Board r1"
- board text added: "IN 36V 10A"
- board text added: "LT3741-1"
- board text added: "OPEN EXT"
- board text added: "OUT CC"
- board text added: "RT"
- board text added: "SN"
- board text added: "SS"
- board text added: "SYNC"
- board text added: "VC"
- board text added: "outer: 35um (1oz) inner: 17um (0.5oz)"
- board text added: "Φ3.2"
