File: pcb/PULSER-testboard-hc/PULSER-testboard-hc.kicad_pcb (KiCad board)
At the start: 4 copper layers, 100 x 100 mm, 80 parts, among them J1 Screw_Terminal 2pin, J2 Screw_Terminal 2pin, J3 Conn_01x02_Pin, J4 Conn_01x02_Pin, Q1 N-ch, Vds>=60V, low Qgs, Q2 N-ch, Vds>=60V, low Rds, U1 LT3741-1, U2 LM317_DPAK

Commit message: HC, HV: PCB DRC pass
Parts:
- HS1: footprint SparkAll:HS-P23D1.6 -> SparkAll:HS-P23D1.6-30x30
Changed lines of the file:
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@@
 	)
 	(paper "A4")
+	(title_block
+		(title "Pulser V2 HC Test Board")
+		(date "2026-01-14")
+		(rev "1")
+		(company "Spark Project")
+		(comment 1 "夕月霞")
+	)
 	(layers
 		(0 "F.Cu" signal)
@@
 		)
 	)
-	(footprint "SparkAll:HS-P23D1.6"
+	(footprint "SparkAll:HS-P23D1.6-30x30"
 		(layer "F.Cu")
 		(at 122.555 65.786 180)
 		(property "Reference" "HS1"
-			(at 11.555 7.286 0)
+			(at 0 -0.5 180)
 			(unlocked yes)
 			(layer "F.SilkS")
@@
 		(polygon
 			(pts
-				(xy 67 75) (xy 109.5 75) (xy 109.5 99) (xy 104.5 99) (xy 104.5 99) (xy 95 99) (xy 95 85) (xy 67 85)
+				(xy 67 75) (xy 109.5 75) (xy 109.5 99) (xy 104.5 99) (xy 95 99) (xy 95 85) (xy 67 85)
 			)
 		)
@@
 		(polygon
 			(pts
-				(xy 52.5 74.5) (xy 64.5 74.5) (xy 64.5 84) (xy 52.5 84) (xy 52.5 74.5)
+				(xy 52.5 74.5) (xy 64.5 74.5) (xy 64.5 84) (xy 52.5 84)
 			)
 		)
@@
 		(polygon
 			(pts
-				(xy 116.5 91.5) (xy 116.5 96) (xy 110 96) (xy 110 83.5) (xy 116.5 83.5) (xy 116.5 91.5)
+				(xy 116.5 91.5) (xy 116.5 96) (xy 110 96) (xy 110 83.5) (xy 116.5 83.5)
 			)
 		)

Commit message: Add I/O descs
Other:
- board text added: "IN analog/PWM 0.15V/A"
- board text added: "IN digital 3.3V - 5V"
Changed lines of the file:
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@@
 		(tags "Through hole pin header THT 1x02 2.54mm single row")
 		(property "Reference" "J3"
-			(at 0 5.54 180)
+			(at -1.25 -2.71 180)
 			(layer "F.SilkS")
 			(effects
@@
 		(tags "Through hole pin header THT 1x02 2.54mm single row")
 		(property "Reference" "J4"
-			(at 0 5.54 180)
+			(at -1 -2.96 180)
 			(layer "F.SilkS")
 			(effects
@@
 		(layer "Edge.Cuts")
 	)
+	(gr_text "IN digital\n3.3V - 5V"
+		(at 113.25 147.25 0)
+		(layer "F.SilkS")
+		(effects
+			(font
+				(size 1 1)
+				(thickness 0.25)
+			)
+			(justify left bottom)
+		)
+	)
 	(gr_text "GND"
 		(at 144 123.5 90)
@@
 			)
 			(justify left bottom)
+		)
+	)
+	(gr_text "IN analog/PWM\n0.15V/A"
+		(at 92.5 147.25 0)
+		(layer "F.SilkS")
+		(effects
+			(font
+				(size 1 1)
+				(thickness 0.25)
+			)
+			(justify left bottom)
