File: pcb/PULSER-testboard-hc/PULSER-testboard-hc.kicad_pcb (KiCad board)
At the start: 4 copper layers, 100 x 100 mm, 80 parts, among them J1 Screw_Terminal 2pin, J2 Screw_Terminal 2pin, J3 Conn_01x02_Pin, J4 Conn_01x02_Pin, Q1 N-ch, Vds>=60V, low Qgs, Q2 N-ch, Vds>=60V, low Rds, U1 LT3741-1, U2 LM317_DPAK

Commit message: HC TestBoard r2 PCB draft ok
Parts:
- removed C12, C13: 0.1u, Capacitor_SMD:C_0603_1608Metric
- removed R11: 100k, Resistor_SMD:R_0603_1608Metric
- removed R23: thermal, Resistor_SMD:R_1225_3264Metric
- removed U1: LT3741-1, Package_DFN_QFN:QFN-20-1EP_4x4mm_P0.5mm_EP2.5x2.5mm
- added C19: 10u, Capacitor_SMD:C_0805_2012Metric, F.Cu at (87.5, 94.8)
- added C20: 10u, Capacitor_SMD:C_0805_2012Metric, F.Cu at (85.5, 94.8)
- added C21: 10u, Capacitor_SMD:C_1206_3216Metric, F.Cu at (111.2, 89.4)
- added C22: 10u, Capacitor_SMD:C_1206_3216Metric, F.Cu at (80.2, 97.5)
- added C23: 10u, Capacitor_SMD:C_1206_3216Metric, F.Cu at (137.6, 113.6)
- added C24: 10u, Capacitor_SMD:C_1206_3216Metric, F.Cu at (137.6, 111.3)
- added C25: 10u, Capacitor_SMD:C_1206_3216Metric, F.Cu at (137.6, 109.0)
- added C26: 10u, Capacitor_SMD:C_1206_3216Metric, F.Cu at (137.6, 106.7)
- added C27: 10u, Capacitor_SMD:C_1206_3216Metric, F.Cu at (137.6, 104.4)
- added C28: 10u, Capacitor_SMD:C_1206_3216Metric, F.Cu at (125.5, 104.4)
- added C29: 10u, Capacitor_SMD:C_1206_3216Metric, F.Cu at (125.5, 106.7)
- added C30: 10u, Capacitor_SMD:C_1206_3216Metric, F.Cu at (125.5, 109.0)
- added C31: 10u, Capacitor_SMD:C_1206_3216Metric, F.Cu at (125.5, 111.3)
- added C32: 10u, Capacitor_SMD:C_1206_3216Metric, F.Cu at (125.5, 113.6)
- added JP10: Jumper_2_Small_Bridged, Jumper:SolderJumper-2_P1.3mm_Bridged_RoundedPad1.0x1.5mm, F.Cu at (76.6, 98.7)
- added JP11: Jumper_2_Small_Bridged, Jumper:SolderJumper-2_P1.3mm_Bridged_RoundedPad1.0x1.5mm, F.Cu at (80.6, 111.0)
- added JP12: Jumper_2_Small_Bridged, Jumper:SolderJumper-2_P1.3mm_Bridged_RoundedPad1.0x1.5mm, F.Cu at (108.0, 131.7)
- added JP13: Jumper_2_Small_Open, Jumper:SolderJumper-2_P1.3mm_Open_RoundedPad1.0x1.5mm, F.Cu at (78.4, 91.0)
- added JP9: Jumper_2_Small_Bridged, Jumper:SolderJumper-2_P1.3mm_Bridged_RoundedPad1.0x1.5mm, F.Cu at (74.1, 98.7)
- added R24: 1Ω 1W, Resistor_SMD:R_2512_6332Metric, F.Cu at (73.8, 70.5)
- added R25: 47k, Resistor_SMD:R_0603_1608Metric, F.Cu at (83.4, 93.5)
- added R26: 4.3k, Resistor_SMD:R_0603_1608Metric, F.Cu at (77.5, 87.0)
- added TP15: TestPoint, TestPoint:TestPoint_Pad_D1.5mm, F.Cu at (77.8, 103.1)
- added TP16: TestPoint, TestPoint:TestPoint_Pad_D1.5mm, F.Cu at (94.8, 111.5)
- added TP17: TestPoint, TestPoint:TestPoint_Pad_D1.5mm, F.Cu at (95.8, 101.7)
- added TP18: TestPoint, TestPoint:TestPoint_Pad_D1.5mm, F.Cu at (77.8, 105.6)
- added U3: LT3763, Package_SO:TSSOP-28-1EP_4.4x9.7mm_P0.65mm_EP2.74x4.75mm, F.Cu at (87.6, 102.0)
- C2: value 0.1u -> 220n
- C5: value 1n -> 10u; footprint Capacitor_SMD:C_0603_1608Metric -> Capacitor_SMD:C_0805_2012Metric
- C9: value 1u -> 1uF 50V; footprint Capacitor_SMD:C_1206_3216Metric -> Capacitor_SMD:C_0805_2012Metric
- R9: value 100k -> 82k
- moved C10 45.8 mm to (113.6, 89.4), turned to 90 degrees
- moved TP4 43.3 mm to (124.5, 125.7)
- moved C11 41.6 mm to (110.0, 92.9), turned to 180 degrees
- moved TP3 33.2 mm to (118.3, 125.7)
- moved C5 32.2 mm to (89.5, 94.8), turned to -90 degrees
- moved C3 32.0 mm to (121.5, 124.0), turned to 180 degrees
- moved C18 29.6 mm to (125.1, 120.6), turned to 90 degrees
- moved R4 28.9 mm to (122.3, 121.7), turned to -90 degrees
- moved R5 28.9 mm to (132.2, 119.0)
- moved R7 28.9 mm to (132.2, 121.0)
- moved R3 28.6 mm to (120.8, 121.7), turned to -90 degrees
- moved TP6 28.0 mm to (143.0, 121.5)
- moved R9 24.4 mm to (77.5, 88.5), turned to 0 degrees
- moved D4 24.1 mm to (119.5, 83.0), turned to -90 degrees
- moved R2 23.5 mm to (121.5, 118.5), turned to 0 degrees
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Connections:
- net Net-(U1-VC) renamed /VC
- C17 pad 2: Net-(JP7-A) -> /VOUT
- C18 pad 2: Net-(JP8-A) -> /VOUT
- C5 pad 2: Net-(JP2-B) -> /INTVCC
- C9 pad 1: GND -> +36V
- C9 pad 2: +36V -> Net-(C9-Pad2)
- D1 pad 2: Net-(D1-A) -> /VOUT
- D2 pad 2: Net-(D2-A) -> /INTVCC
- D4 pad 2: Net-(D1-A) -> /VOUT
- J3 pad 1: /EN -> Net-(J3-Pin_1)
- JP1 pad 2: Net-(JP1-B) -> /SYNC
- JP2 pad 2: Net-(JP2-B) -> /SS
- JP3 pad 2: Net-(JP3-B) -> /RT
- JP7 pad 2: Net-(D1-A) -> /VOUT
- JP8 pad 2: Net-(D1-A) -> /VOUT
- R2 pad 2: Net-(D1-A) -> /VOUT
- R4 pad 1: Net-(D1-A) -> /VOUT
- R5 pad 1: Net-(D1-A) -> /VOUT
- R9 pad 1: Net-(JP3-B) -> +36V
- R9 pad 2: GND -> /EN
- TP12 pad 1: Net-(JP2-B) -> /SS
- TP13 pad 1: Net-(JP3-B) -> /RT
- TP4 pad 1: Net-(D1-A) -> /VOUT
- TP9 pad 1: Net-(D2-A) -> /INTVCC
Routing:
- net Net-(D1-A): track 99.7 -> 0.00 mm
- net /VOUT: track 0.00 -> 95.0 mm
- net Net-(J3-Pin_1): track 0.00 -> 90.4 mm, vias 0 -> 2
- net +3V3: track 96.3 -> 44.2 mm, vias 4 -> 2
- net /EN: track 67.8 -> 16.6 mm
- net Net-(JP2-B): track 49.0 -> 0.00 mm, vias 2 -> 0
- net /SS: track 0.00 -> 45.0 mm, vias 0 -> 2
- net Net-(JP3-B): track 44.1 -> 0.00 mm
- net /PWM: track 0.00 -> 40.7 mm
- net /RT: track 0.00 -> 37.6 mm
- net /~{FAULT}: track 0.00 -> 27.4 mm, vias 0 -> 2
- net /INTVCC: track 0.00 -> 21.8 mm
- net Net-(U3-SW): track 79.3 -> 58.0 mm, vias 2 -> 4
- net /SENSE+: track 61.8 -> 41.0 mm
- net Net-(U3-TG): track 22.2 -> 41.4 mm
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- added copper zone on F.Cu, net /VOUT
- added copper zone on F.Cu, net Net-(JP7-A)
- added copper zone on F.Cu, net Net-(JP8-A)
- removed copper zone on F.Cu, net Net-(D1-A)
Other:
- board text added: "HC Test Board r2"
- board text added: "LT3763"
- board text removed: "CTRL2"
- board text removed: "HC Test Board r1"
- board text removed: "LT3741-1"
- board text removed: "RT"
- board text removed: "SS"
- board text removed: "SYNC"
- board text removed: "VC"
