File: pcb/PULSER-testboard-hc/PULSER-testboard-hc.kicad_pcb (KiCad board)
At the start: 4 copper layers, 100 x 100 mm, 102 parts, among them J1 Screw_Terminal 2pin, J2 Screw_Terminal 2pin, J3 Conn_01x02_Pin, J4 Conn_01x02_Pin, Q1 N-ch, Vds>=60V, low Qgs, Q2 N-ch, Vds>=60V, low Rds, U2 LM317_DPAK, U3 LT3763

Commit message: HC r3 schem draft ok
Parts:
- removed C28, C31, C32: 10u, Capacitor_SMD:C_1206_3216Metric
- removed G***: LOGO, LOGO
- removed HS1: Heatsink_Pad_2Pin, SparkAll:HS-P23D1.6-30x30
- removed J4: Conn_01x02_Pin, Connector_PinHeader_2.54mm:PinHeader_1x02_P2.54mm_Vertical
- removed JP10, JP11, JP12, JP2, JP3, JP7, JP8, JP9: Jumper_2_Small_Bridged, Jumper:SolderJumper-2_P1.3mm_Bridged_RoundedPad1.0x1.5mm
- removed JP13: Jumper_2_Small_Open, Jumper:SolderJumper-2_P1.3mm_Open_RoundedPad1.0x1.5mm
- removed JP4, JP5, JP6: ~, Connector_PinHeader_2.54mm:PinHeader_1x02_P2.54mm_Vertical
- removed R20: 1.5k, Resistor_SMD:R_0603_1608Metric
- removed R21: 1.1k, Resistor_SMD:R_0603_1608Metric
- removed R22: 1M, Resistor_SMD:R_0603_1608Metric
- removed TH1: Thermistor_NTC, Resistor_SMD:R_0603_1608Metric
- removed TP11, TP13, TP17, TP7: TestPoint, TestPoint:TestPoint_Pad_D1.5mm
- added C12: 22n, Capacitor_SMD:C_0805_2012Metric, F.Cu at (169.9, 60.0)
- added C33: 0.1u, Capacitor_SMD:C_0402_1005Metric, F.Cu at (188.4, 111.6)
- added C35: 0.1u, Capacitor_SMD:C_0402_1005Metric, F.Cu at (188.4, 114.1)
- added D5: Vz=100V, Diode_SMD:D_SMB, F.Cu at (181.4, 48.6)
- added D6: ~, SparkAll:TO-227A-2P, F.Cu at (180.3, 53.0)
- added D7: LED, LED_SMD:LED_0805_2012Metric, F.Cu at (196.8, 105.5)
- added D8: LED, LED_SMD:LED_0805_2012Metric, F.Cu at (196.8, 108.6)
- added J6: Conn_01x08_Pin, Connector_FFC-FPC:Molex_200528-0080_1x08-1MP_P1.00mm_Horizontal, F.Cu at (131.0, 56.0)
- added R11: 3.3, Resistor_SMD:R_2512_6332Metric, F.Cu at (172.1, 56.0)
- added U1: ADuM1200AR, Package_SO:SOIC-8_3.9x4.9mm_P1.27mm, F.Cu at (131.0, 64.0)
- added U4: TPSM365R6, SparkAll:TI-RDN0011A-MFG, F.Cu at (167.1, 114.0)
- C1, C15, C16, C17, C18, C3, C4, C6, C7: footprint Capacitor_SMD:C_0603_1608Metric -> Capacitor_SMD:C_0402_1005Metric
- C14, C27: footprint Capacitor_SMD:C_1206_3216Metric -> Capacitor_SMD:C_0603_1608Metric
- C26: value 10u -> 1u; footprint Capacitor_SMD:C_1206_3216Metric -> Capacitor_SMD:C_0402_1005Metric
- C29, C30: value 10u -> 1u; footprint Capacitor_SMD:C_1206_3216Metric -> Capacitor_SMD:C_0603_1608Metric
- C8: value 10n -> 220n
- C9: value 1uF 50V -> 1u
- D1: value 120V 10A -> ~; footprint Package_TO_SOT_THT:TO-220-2_Vertical -> SparkAll:VISHAY-SMPC
- D2: value 100mA -> ~
- J3: footprint Connector_PinHeader_2.54mm:PinHeader_1x02_P2.54mm_Vertical -> Connector_JST:JST_XH_B2B-XH-A_1x02_P2.50mm_Vertical
- R10, R12, R13, R17, R18, R25, R26, R3, R4, R5, R7, R8, R9: footprint Resistor_SMD:R_0603_1608Metric -> Resistor_SMD:R_0402_1005Metric
- R14: value 2.4k -> 110k; footprint Resistor_SMD:R_0603_1608Metric -> Resistor_SMD:R_0402_1005Metric
- R15: value 5.1k -> 10k; footprint Resistor_SMD:R_0603_1608Metric -> Resistor_SMD:R_0402_1005Metric
- R16: value 11k -> 1k; footprint Resistor_SMD:R_0603_1608Metric -> Resistor_SMD:R_0402_1005Metric
- R19: value 2k -> 1k; footprint Resistor_SMD:R_0603_1608Metric -> Resistor_SMD:R_0402_1005Metric
- R24: value 1Ω 1W -> 1
- moved R16 140.3 mm to (200.5, 105.0)
- moved R19 138.2 mm to (200.5, 107.0)
- moved F1 136.3 mm to (196.5, 40.0)
- moved J3 115.4 mm to (171.2, 49.2), turned to 0 degrees
- moved TP12 114.5 mm to (171.5, 116.6)
- moved TP15 114.4 mm to (189.9, 80.5)
- moved TP18 113.6 mm to (189.9, 87.6)
- moved D3 113.4 mm to (194.6, 83.7)
- moved TP14 110.7 mm to (186.4, 87.6)
- moved U2 109.4 mm to (170.7, 106.9), turned to 0 degrees
- moved R10 109.1 mm to (175.5, 80.0), turned to 0 degrees
- moved R15 108.8 mm to (171.2, 113.9)
- moved C20 108.6 mm to (194.1, 96.9), turned to 0 degrees
- moved R14 108.3 mm to (171.2, 111.9)
- moved C19 106.6 mm to (194.1, 93.9), turned to 0 degrees
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Connections:
- net /CTRL1 renamed /CURR_CTRL
- net /CTRL2 renamed /highcurrent/CTRL2
- net /INTVCC renamed /highcurrent/INTVCC
- net /SENSE+ renamed /highcurrent/SENSE+
- net /SENSE- renamed /highcurrent/SENSE-
- net /SYNC renamed /highcurrent/SYNC
- net /VC renamed /highcurrent/VC
- net /~{FAULT} renamed /highcurrent/~{FAULT}
- C14 pad 2: /VREF -> /highcurrent/VREF
- C15 pad 2: +36V -> +12V
- C17 pad 2: /VOUT -> /highcurrent/VOUT
- C18 pad 2: /VOUT -> /highcurrent/VOUT
- C23 pad 2: Net-(JP7-A) -> /highcurrent/VOUT
- C24 pad 2: Net-(JP7-A) -> /highcurrent/VOUT
- C25 pad 2: Net-(JP7-A) -> /highcurrent/VOUT
- C26 pad 1: GND -> Net-(U4-VCC)
- C26 pad 2: Net-(JP7-A) -> GND
- C27 pad 1: GND -> +12V
- C27 pad 2: Net-(JP7-A) -> GND
- C29 pad 1: GND -> +36V
- C29 pad 2: Net-(JP8-A) -> GND
- C30 pad 1: GND -> +36V
- C30 pad 2: Net-(JP8-A) -> GND
- C6 pad 2: Net-(JP2-A) -> /highcurrent/SS
- D1 pad 2: /VOUT -> /highcurrent/VOUT
- D3 pad 1: /VREF -> /highcurrent/VREF
- D4 pad 2: /VOUT -> /highcurrent/VOUT
- J3 pad 1: Net-(J3-Pin_1) -> +12V
- R10 pad 1: Net-(JP3-A) -> /highcurrent/RT
- R12 pad 1: /CTRL_RAW -> Net-(U1-VOB)
- R13 pad 1: /VREF -> /highcurrent/VREF
- R14 pad 1: +3V3 -> +12V
- R14 pad 2: Net-(JP4-A) -> Net-(U4-BIAS)
- R15 pad 1: +3V3 -> Net-(U4-BIAS)
- R15 pad 2: Net-(JP5-A) -> GND
- R16 pad 1: +3V3 -> GND
- R19 pad 2: Net-(JP4-A) -> Net-(D8-K)
- R2 pad 2: /VOUT -> /highcurrent/VOUT
- R26 pad 1: /EN -> /highcurrent/EN
- R4 pad 1: /VOUT -> /highcurrent/VOUT
- R5 pad 1: /VOUT -> /highcurrent/VOUT
- R9 pad 2: /EN -> /highcurrent/EN
- TP12 pad 1: /SS -> Net-(U4-PGOOD)
- TP4 pad 1: /VOUT -> /highcurrent/VOUT
- U2 pad 3: +36V -> +12V
- U3 pad 10: Net-(JP11-B) -> /highcurrent/VREF
- U3 pad 15: /SS -> /highcurrent/SS
- U3 pad 20: /RT -> /highcurrent/RT
- U3 pad 22: /PWM -> /EN
- U3 pad 24: Net-(U3-PWM_OUT) -> unconnected-(U3-PWM_OUT-Pad24)
- U3 pad 4: /EN -> /highcurrent/EN
- U3 pad 5: /VREF -> /highcurrent/VREF
- U3 pad 6: Net-(JP10-B) -> +36V
- U3 pad 7: Net-(JP9-B) -> +36V
Routing:
- net +36V: track 114.3 -> 0.00 mm
- net /VOUT: track 95.0 -> 0.00 mm
- net Net-(J3-Pin_1): track 90.4 -> 0.00 mm, vias 2 -> 0
- net /CURR_CTRL: track 83.6 -> 0.00 mm, vias 2 -> 0
- net Net-(U3-FB): track 73.6 -> 0.00 mm, vias 2 -> 0
- net /VREF: track 62.1 -> 0.00 mm, vias 3 -> 0
- net Net-(U3-SW): track 58.0 -> 0.00 mm, vias 4 -> 0
- net /SS: track 45.0 -> 0.00 mm, vias 2 -> 0
- net +3V3: track 44.2 -> 0.00 mm, vias 2 -> 0
- net /highcurrent/SENSE-: track 43.2 -> 0.00 mm, vias 2 -> 0
- net Net-(U3-TG): track 41.4 -> 0.00 mm, vias 3 -> 0
- net /highcurrent/SENSE+: track 41.0 -> 0.00 mm, vias 2 -> 0
- net /PWM: track 40.7 -> 0.00 mm
- net /RT: track 37.6 -> 0.00 mm
- net Net-(U3-BG): track 37.1 -> 0.00 mm, vias 2 -> 0
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- removed copper zone on F.Cu, net +36V
- removed copper zone on F.Cu, net +3V3
- removed copper zone on F.Cu, net /VOUT
- removed copper zone on B.Cu, net GND
- removed copper zone on F.Cu, net GND
- removed copper zone on F.Cu, net Net-(C1-Pad2)
- removed copper zone on F.Cu, net Net-(C4-Pad2)
- removed copper zone on F.Cu, net Net-(D1-K)
- removed copper zone on F.Cu, net Net-(J1-Pin_2)
- removed copper zone on F.Cu, net Net-(JP7-A)
- removed copper zone on F.Cu, net Net-(JP8-A)
- removed copper zone on F.Cu, net Net-(L1-Pad2)
- removed copper zone on F.Cu, net Net-(U3-SW)
Other:
- board size 100 x 100 mm -> 100 x 50 mm
- board text removed: "+"
- board text removed: "-"
- board text removed: "10A"
- board text removed: "10uH"
- board text removed: "2A"
- board text removed: "5A"
- board text removed: "CTRL_EXT"
- board text removed: "EN_OVR"
- board text removed: "GND"
- board text removed: "HC Test Board r2"
- board text removed: "IN 36V 10A"
- board text removed: "IN analog/PWM 0.15V/A"
- board text removed: "IN digital 3.3V - 5V"
- board text removed: "LT3763"
- board text removed: "OPEN EXT"
- board text removed: "OUT CC"
- board text removed: "SN"

Commit message: hc pcb draft ok
Parts:
- removed TP14, TP6: TestPoint, TestPoint:TestPoint_Pad_D1.5mm
- added G***: LOGO, LOGO, F.Cu at (136.0, 87.0)
- moved F1 136.4 mm to (63.5, 70.0)
- moved C26 127.9 mm to (60.6, 52.9), turned to 180 degrees
- moved D6 122.3 mm to (62.7, 86.5), turned to 180 degrees
- moved D4 120.7 mm to (73.0, 77.5), turned to 180 degrees
- moved D5 120.7 mm to (68.0, 89.8), turned to -90 degrees
- moved R15 120.6 mm to (67.4, 52.5), turned to 90 degrees
- moved D1 119.7 mm to (71.3, 83.0), turned to -90 degrees
- moved U4 118.9 mm to (64.2, 54.4), turned to 90 degrees
- moved R14 118.7 mm to (67.4, 54.4), turned to 90 degrees
- moved TP12 116.0 mm to (72.0, 57.0)
- moved C30 114.5 mm to (62.2, 57.5), turned to 180 degrees
- moved C29 112.6 mm to (62.2, 59.0), turned to 180 degrees
- moved C12 111.7 mm to (59.5, 76.5), turned to -90 degrees
- moved R11 109.0 mm to (65.0, 76.0)
- moved R2 108.2 mm to (81.5, 82.0), turned to 180 degrees
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Routing:
- net +12V: track 0.00 -> 85.9 mm
- net +36V: track 0.00 -> 82.6 mm, vias 0 -> 55
- net /highcurrent/SENSE-: track 0.00 -> 77.3 mm, vias 0 -> 2
- net /highcurrent/SENSE+: track 0.00 -> 73.6 mm, vias 0 -> 2
- net Net-(U3-FB): track 0.00 -> 52.5 mm, vias 0 -> 2
- net /EN: track 0.00 -> 51.0 mm, vias 0 -> 3
- net +3V3: track 0.00 -> 38.9 mm
- net Net-(U3-TG): track 0.00 -> 33.0 mm, vias 0 -> 3
- net /CURR_CTRL: track 0.00 -> 32.3 mm, vias 0 -> 2
- net Net-(U3-SW): track 0.00 -> 30.9 mm, vias 0 -> 22
- net Net-(D2-K): track 0.00 -> 29.6 mm
- net Net-(U3-BG): track 0.00 -> 23.8 mm, vias 0 -> 3
- net /highcurrent/VREF: track 0.00 -> 21.1 mm, vias 0 -> 2
- net Net-(U3-IVINMON): track 0.00 -> 18.8 mm, vias 0 -> 2
- net /highcurrent/INTVCC: track 0.00 -> 18.0 mm
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- added copper zone on B.Cu, net +36V
- added copper zone on F.Cu, net +36V
- added copper zone on F.Cu, net /highcurrent/VOUT
- added copper zone on B.Cu, net GND
- added copper zone on F.Cu, net GND
- added copper zone on In1.Cu, net GNDS
- added copper zone on In2.Cu, net GNDS
- added copper zone on B.Cu, net Net-(C12-Pad1)
- added copper zone on F.Cu, net Net-(C12-Pad1)
- added copper zone on B.Cu, net Net-(D1-K)
- added copper zone on F.Cu, net Net-(D1-K)
- added copper zone on B.Cu, net Net-(J1-Pin_2)
- added copper zone on F.Cu, net Net-(J1-Pin_2)
- added copper zone on B.Cu, net Net-(L1-Pad2)
- added copper zone on F.Cu, net Net-(L1-Pad2)
- added copper zone on B.Cu, net Net-(U3-SW)
- added copper zone on F.Cu, net Net-(U3-SW)
Other:
- board text added: "+"
- board text added: "10A"
- board text added: "CTRL"
- board text added: "EN"
- board text added: "FAN(12V)"
- board text added: "I+(36V)"
- board text added: "I-"
- board text added: "O+"
- board text added: "O-"
- board text added: "PWR"
- board text added: "SN"
- board text added: "pulser-v2/HC-r${REVISION}"
