File: pcb/PULSER-testboard-hc/PULSER-testboard-hc.kicad_sch (KiCad schematic)
At the start: 34 parts, among them J1 Screw_Terminal 2pin, J2 Screw_Terminal 2pin, J3 CTRL1, Q1 N-ch, Vds>=60V, fast switch, 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, Q2 N-ch, Vds>=60V, fast switch, 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, U1 LT3741-1, U4 LM317_DPAK

Commit message: Draft architecture for both HC & HV
Parts:
- removed J3: CTRL1, symbol Connector:Conn_01x01_Pin
- added J4, J5: Conn_01x02_Pin, symbol Connector:Conn_01x02_Pin
- added R15: 100k, symbol Device:R
- renumbered C2 to C1, C1 to C2, D4 to D2, HS2 to HS1, J2 to J1, J1 to J2, JP4 to JP1, JP1 to JP2, JP2 to JP3, JP3 to JP4, R7 to R10, R10 to R11, R14 to R13, R8 to R14, R9 to R6, R11 to R7, R13 to R8, R6 to R9, U4 to U2
Connections:
- net +3V3: now also R15.1
- net CTRL1: now also J5.1 (Pin_1)
- net GND: now also J4.2 (Pin_2), J5.2 (Pin_2)
- net EN: now reaches U1.1 (EN/UVLO)
- net EN: now also J4.1 (Pin_1), R15.2
Other:
- note removed: "current timing control"
- company: (none) -> Spark Project
- title: (none) -> Pulser V2 HV Test Board
- moved on the sheet: J2

Commit message: HC testboard: schem draft ok
Parts:
- added C1, C4, C5: 1n, Capacitor_SMD:C_0603_1608Metric, symbol Device:C_Small
- added C10, C11: 10u, Capacitor_SMD:C_1206_3216Metric, symbol Device:C_Small
- added C12, C13: 0.1u, Capacitor_SMD:C_0603_1608Metric, symbol Device:C_Small
- added C14: 2.2u, Capacitor_SMD:C_1206_3216Metric, symbol Device:C_Small
- added C3: 22n, Capacitor_SMD:C_0603_1608Metric, symbol Device:C_Small
- added C8: 10n, Capacitor_SMD:C_0603_1608Metric, symbol Device:C_Small
- added C9: 1u, Capacitor_SMD:C_1206_3216Metric, symbol Device:C_Small
- added D3: D, Diode_SMD:D_SOD-123, symbol Device:D
- added D4: Ipeak>10A, SparkAll:TO-227A-2P, symbol Device:D_Schottky
- added F1: 10A, Fuse:Fuse_Littelfuse-NANO2-451_453, symbol Device:Fuse
- added JP2, JP3: Jumper_2_Small_Bridged, Jumper:SolderJumper-2_P1.3mm_Bridged_RoundedPad1.0x1.5mm, symbol Jumper:Jumper_2_Small_Bridged
- added R1, R6: 1, Resistor_SMD:R_1206_3216Metric, symbol Device:R
- added R12: 10k, Resistor_SMD:R_0603_1608Metric, symbol Device:R
- added R13: 47k, Resistor_SMD:R_0603_1608Metric, symbol Device:R
- added R3, R4: 10, Resistor_SMD:R_0603_1608Metric, symbol Device:R
- added R9: 100k, Resistor_SMD:R_0603_1608Metric, symbol Device:R
- added TH1: Thermistor_NTC, Resistor_SMD:R_0603_1608Metric, symbol Device:Thermistor_NTC
- added TP1, TP2, TP3, TP4, TP5, TP6, TP7, TP8: TestPoint, TestPoint:TestPoint_Pad_D1.5mm, symbol Connector:TestPoint_Small
- C15: renamed from C4; footprint (none) -> Capacitor_SMD:C_0603_1608Metric; LCSC (none) -> C14663
- C16: renamed from C5; value 1u -> 0.1u; footprint (none) -> Capacitor_SMD:C_0603_1608Metric; LCSC (none) -> C14663
- C2: renamed from C1; value C_Small -> 0.1u; footprint (none) -> Capacitor_SMD:C_0603_1608Metric; LCSC (none) -> C14663
- C6: renamed from C2; footprint (none) -> Capacitor_SMD:C_0603_1608Metric; LCSC (none) -> C1620
- C7: renamed from C3; footprint (none) -> Capacitor_SMD:C_0603_1608Metric; LCSC (none) -> C53987
- D1: footprint SparkAll:D_SOD-323HE -> Package_TO_SOT_THT:TO-220-2_Vertical
- D2: value 150V 1A -> 100mA; footprint SparkAll:D_SOD-323HE -> Diode_SMD:D_SOD-123; LCSC C2842811 -> C177047
- HS1: footprint (none) -> SparkAll:HS-P23D1.6; now not fitted
- J3: renamed from J4; footprint (none) -> Connector_PinHeader_2.54mm:PinHeader_1x02_P2.54mm_Vertical; LCSC (none) -> C492401
- J4: renamed from J5; footprint (none) -> Connector_PinHeader_2.54mm:PinHeader_1x02_P2.54mm_Vertical; LCSC (none) -> C492401
- JP1: footprint (none) -> Jumper:SolderJumper-2_P1.3mm_Bridged_RoundedPad1.0x1.5mm; now left out of the parts list
- JP4: renamed from JP2; value 10A -> ~; footprint (none) -> Connector_PinHeader_2.54mm:PinHeader_1x02_P2.54mm_Vertical; LCSC (none) -> C492401
- JP5: renamed from JP3; value 5A -> ~; footprint (none) -> Connector_PinHeader_2.54mm:PinHeader_1x02_P2.54mm_Vertical; LCSC (none) -> C492401
- JP6: renamed from JP4; value 2A -> ~; footprint (none) -> Connector_PinHeader_2.54mm:PinHeader_1x02_P2.54mm_Vertical; LCSC (none) -> C492401
- L1: footprint SparkAll:BOURNS-PQ2614B -> Inductor_SMD:L_Bourns_SRP1245A; LCSC C1330029 -> C840531
- Q1: value N-ch, Vds>=60V, fast switch, low Rds -> N-ch, Vds>=60V, low Qgs; LCSC C24199 -> C3278729
- Q2: value N-ch, Vds>=60V, fast switch, low Rds -> N-ch, Vds>=60V, low Rds; LCSC C24199 -> C501503
- R10: renamed from R5; footprint (none) -> Resistor_SMD:R_0603_1608Metric
- R11: renamed from R15; footprint (none) -> Resistor_SMD:R_0603_1608Metric
- R14: renamed from R6; footprint (none) -> Resistor_SMD:R_0603_1608Metric
- R15: renamed from R7; footprint (none) -> Resistor_SMD:R_0603_1608Metric
- R16: renamed from R8; footprint (none) -> Resistor_SMD:R_0603_1608Metric
- R17: renamed from R9; footprint (none) -> Resistor_SMD:R_0603_1608Metric
- R18: renamed from R10; footprint (none) -> Resistor_SMD:R_0603_1608Metric
- R19: renamed from R11; footprint (none) -> Resistor_SMD:R_0603_1608Metric
- R2: renamed from R1; footprint (none) -> Resistor_SMD:R_1206_3216Metric; LCSC (none) -> C7419996
- R20: renamed from R12; footprint (none) -> Resistor_SMD:R_0603_1608Metric
- R21: renamed from R13; footprint (none) -> Resistor_SMD:R_0603_1608Metric
- R22: renamed from R14; value 100k -> 1M; footprint (none) -> Resistor_SMD:R_0603_1608Metric
- R5: renamed from R2; footprint (none) -> Resistor_SMD:R_0603_1608Metric
- R7: renamed from R3; footprint (none) -> Resistor_SMD:R_0603_1608Metric
- R8: renamed from R4; footprint (none) -> Resistor_SMD:R_0603_1608Metric
- renumbered J2 to J1, J1 to J2
Connections:
- net +36V: now also C10.2, C11.2, C12.2, C13.2, C9.2, D4.1 (K), F1.2, R1.1; no longer J1.2 (Pin_2)
- net +3V3: now also TP7.1
- net CTRL1: now also C8.2, D3.2 (A), R12.2, TP8.1; no longer J4.1 (Pin_1)
- net GND: now also C10.1, C11.1, C12.1, C13.1, C14.1, C4.1, C5.1, C8.1, C9.1, R9.2, TH1.2
- net at C2.1, L1.1, Q1.S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: now also C1.1, R6.1, TP2.1
- net at L1.2, R2.1: now also R3.1, TP3.1; no longer U1.8 (SENSE+)
- net at Q1.G, U1.15 (HG): now also TP1.1
- net at C6.2: now also C5.2, JP2.1 (A); no longer U1.6 (SS)
- net at D1.2 (A), R2.2, R5.1: now also D4.2 (A), R4.1, TP4.1; no longer U1.9 (SENSE-)
- net at R5.2, R7.1, U1.7 (FB): now also TP6.1
- net at R10.1: now also JP3.1 (A); no longer U1.12 (RT)
- net at Q2.G, U1.18 (LG): now also TP5.1
- net VREF: now reaches U1.2 (VREF)
- net VREF: now also C14.2, D3.1 (K), R13.1
- net CTRL2: now reaches U1.3 (CTRL2)
- net CTRL2: now also R13.2, TH1.1
- new net: F1.1, J1.2 (Pin_2)
- new net: C4.2, R6.2
- new net: JP3.2 (B), R9.1, U1.12 (RT)
- new net: C3.2, R3.2, U1.8 (SENSE+)
- new net: JP2.2 (B), U1.6 (SS)
- new net: C3.1, R4.2, U1.9 (SENSE-)
- new net: C1.2, R1.2
- new net CTRL_RAW: J4.1 (Pin_1), R12.1
Other:
- note added: "0.15V/A max 1.5V analog or PWM 1.6kHz low-pass filtered high-side clamp to 2V Zin=1kΩ"
- note added: "0.5W"
- note added: "10A"
- note added: "2A"
- note added: "5A"
- note added: "MOSFET"
- note added: "fc=1.6kHz LPF"
- note added: "fc=723kHz"
- note added: "protection"
- note added: "uC"
- note removed: "500mW"
- title: Pulser V2 HV Test Board -> Pulser V2 HC Test Board
- moved on the sheet: D1, J2, Q1, R11, R2, R5, R7

Commit message: HC test board pcb draft ok
Parts:
- added C17, C18: 10n, Capacitor_SMD:C_0603_1608Metric, symbol Device:C_Small
- added JP7, JP8: Jumper_2_Small_Bridged, Jumper:SolderJumper-2_P1.3mm_Bridged_RoundedPad1.0x1.5mm, symbol Jumper:Jumper_2_Small_Bridged
- added R23: thermal, Resistor_SMD:R_1225_3264Metric, symbol Device:R
- added TP10, TP11, TP12, TP13, TP14, TP9: TestPoint, TestPoint:TestPoint_Pad_D1.5mm, symbol Connector:TestPoint_Small
Connections:
- net +36V: now also R23.1
- net CTRL2: now also TP14.1
- net GND: now also C15.1, C16.1, R18.2, C17.1, C18.1, R23.2
- net at D1.2 (A), D4.2 (A), R2.2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: now also JP7.2 (B), JP8.2 (B)
- net at R8.1, U1.10 (VC): now also TP11.1
- net at JP3.2 (B), R9.1, U1.12 (RT): now also TP13.1
- net at C6.2, JP2.1 (A): no longer C5.2
- net SENSE+: now reaches C3.2, R3.2, U1.8 (SENSE+)
- net at C2.2, D2.1 (K), U1.17 (CBOOT): now also TP10.1
- net at D2.2 (A), U1.19 (VCC_INT): now also TP9.1
- net at JP2.2 (B), U1.6 (SS): now also C5.2, TP12.1
- net SENSE-: now reaches C3.1, R4.2, U1.9 (SENSE-)
- new net: C18.2, JP8.1 (A)
- new net: C17.2, JP7.1 (A)
Other:
- note added: "tuned to 1A ripple"
- moved on the sheet: D1, HS1, J2

Commit message: HC, HV: PCB DRC pass
Parts:
- HS1: footprint SparkAll:HS-P23D1.6 -> SparkAll:HS-P23D1.6-30x30
Changed lines of the file:
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@@
 			)
 		)
-		(property "Footprint" "SparkAll:HS-P23D1.6"
+		(property "Footprint" "SparkAll:HS-P23D1.6-30x30"
 			(at 259.3848 33.02 0)
 			(effects

Commit message: HC: add missing LCSC number
Parts:
- U1: LCSC (none) -> C671328
- U2: LCSC (none) -> C68136
Changed lines of the file:
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@@
+			)
+		)
+		(property "LCSC" "C671328"
+			(at 138.43 54.61 0)
+			(effects
+				(font
+					(size 1.27 1.27)
+				)
+				(hide yes)
 			)
 		)
@@
 			(at 62.23 154.94 0)
 			(effects
+				(font
+					(size 1.27 1.27)
+				)
+				(hide yes)
+			)
+		)
+		(property "LCSC" "C68136"
+			(at 62.23 154.94 0)
+			(effects

Commit message: HC TestBoards r2 schem draft ok
Parts:
- removed R11: 100k, Resistor_SMD:R_0603_1608Metric, symbol Device:R
- removed U1: LT3741-1, Package_DFN_QFN:QFN-20-1EP_4x4mm_P0.5mm_EP2.5x2.5mm, symbol SparkAll:LT3741-1
- added C19, C20, C22: 10u, symbol Device:C_Small
- added C21, C23, C24, C25, C26, C27, C28, C29, C30, C31, C32: 10u, Capacitor_SMD:C_1206_3216Metric, symbol Device:C_Small
- added JP10, JP11, JP12, JP9: Jumper_2_Small_Bridged, Jumper:SolderJumper-2_P1.3mm_Bridged_RoundedPad1.0x1.5mm, symbol Jumper:Jumper_2_Small_Bridged
- added JP13: Jumper_2_Small_Open, symbol Jumper:Jumper_2_Small_Open
- added R24: 1Ω 1W, symbol Device:R
- added R25: 47k, Resistor_SMD:R_0603_1608Metric, symbol Device:R
- added R26: 10k, Resistor_SMD:R_0603_1608Metric, symbol Device:R
- added TP15, TP16, TP17, TP18: TestPoint, TestPoint:TestPoint_Pad_D1.5mm, symbol Connector:TestPoint_Small
- added U3: LT3763, symbol SparkAll:LT3763
- C2: value 0.1u -> 220n; LCSC C14663 -> (none)
- C5: value 1n -> 10u; footprint Capacitor_SMD:C_0603_1608Metric -> (none); LCSC C1588 -> (none); now fitted
- C9: value 1u -> 1uF 50V; footprint Capacitor_SMD:C_1206_3216Metric -> (none); LCSC C1848 -> (none)
- R9: value 100k -> 190k; now fitted
Connections:
- net +36V: now also C9.1, R9.1, C21.2, C22.2, JP10.1 (A), JP9.1 (A), U3.3 (VIN); no longer C9.2
- net CTRL1: now also U3.14 (CTRL1)
- net CTRL2: now also U3.13 (CTRL2)
- net EN: now also R9.2, JP13.2 (B), R26.1, U3.4 (EN/UVLO); no longer J3.1 (Pin_1)
- net GND: now also C19.1, C20.1, C21.1, C22.1, C23.1, C24.1, C25.1, C26.1, C27.1, C28.1, C29.1, C30.1, C31.1, C32.1, R24.2, R26.2, U3.12 (GND), U3.23 (GND), U3.28 (GND), U3.29 (GND); no longer C9.1, R9.2
- net SENSE+: now also U3.17 (SENSE+)
- net SENSE-: now also U3.16 (SENSE-)
- net VREF: now also JP11.1 (A), U3.5 (VREF)
- net at C1.1, C2.1, L1.1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: now also U3.26 (SW)
- net at JP8.1 (A): now also C28.2, C29.2, C30.2, C31.2, C32.2; no longer C18.2
- net VOUT: now reaches D1.2 (A), D4.2 (A), JP7.2 (B), JP8.2 (B), R2.2, R4.1, R5.1, TP4.1
- net VOUT: now also C17.2, C18.2
- net at Q1.G, TP1.1: now also U3.25 (TG)
- net SS: now reaches JP2.2 (B), TP12.1
- net SS: now also U3.15 (SS); no longer C5.2
- net VC: now reaches R8.1, TP11.1
- net VC: now also U3.18 (VC)
- net RT: now reaches JP3.2 (B), TP13.1
- net RT: now also U3.20 (RT); no longer R9.1
- net at R5.2, R7.1, TP6.1: now also U3.11 (FB)
- net at JP7.1 (A): now also C23.2, C24.2, C25.2, C26.2, C27.2; no longer C17.2
- net at C2.2, D2.1 (K), TP10.1: now also U3.27 (BOOST)
- net SYNC: now reaches JP1.2 (B)
- net SYNC: now also U3.21 (SYNC)
- net at Q2.G, TP5.1: now also U3.1 (BG)
- net INTVCC: now reaches D2.2 (A), TP9.1
- net INTVCC: now also C5.2, C19.2, C20.2, R25.2, U3.2 (INTVCC)
- new net: JP9.2 (B), U3.7 (IVINP)
- new net: JP10.2 (B), U3.6 (IVINN)
- new net: J3.1 (Pin_1), JP12.1 (A), JP13.1 (A)
- new net: C9.2, R24.1
- new net: JP11.2 (B), U3.10 (FBIN)
- new net: TP16.1, U3.19 (ISMON)
- new net: TP17.1, U3.24 (PWM_OUT)
- new net: TP15.1, U3.8 (IVINMON)
- new net PWM: JP12.2 (B), U3.22 (PWM)
- new net ~{FAULT}: R25.1, TP18.1, U3.9 (~{FAULT})
Other:
- note added: "22uF is recommended in datasheet account for cap loss by DC-bias 16V+ is recommended"
- note added: "2uFx10 = 20uF is recommended 30uF is DC-bias accounted value Since 10u is big, 0.1u is closer bypass"
- note added: "IC"
- note added: "resonance damper for cable inductance"
- note removed: "tuned to 1A ripple"
- note removed: "uC"
- moved on the sheet: C10, C11, C12, C13, C14, C15, C16, C17, C18, C2, C6, C7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

Commit message: HC TestBoard r2 PCB draft ok
Parts:
- removed C12, C13: 0.1u, Capacitor_SMD:C_0603_1608Metric, symbol Device:C_Small
- removed R23: thermal, Resistor_SMD:R_1225_3264Metric, symbol Device:R
- C19, C20, C5: footprint (none) -> Capacitor_SMD:C_0805_2012Metric; LCSC (none) -> C1713
- C22: footprint (none) -> Capacitor_SMD:C_1206_3216Metric; LCSC (none) -> C89632
- C9: footprint (none) -> Capacitor_SMD:C_0805_2012Metric; LCSC (none) -> C28323
- JP13: footprint (none) -> Jumper:SolderJumper-2_P1.3mm_Open_RoundedPad1.0x1.5mm; now not fitted
- R10: LCSC (none) -> C25808
- R12: LCSC (none) -> C25804
- R13, R25: LCSC (none) -> C25819
- R14: LCSC (none) -> C22940
- R15: LCSC (none) -> C23186
- R16: LCSC (none) -> C25950
- R17: LCSC (none) -> C23350
- R18: LCSC (none) -> C23151
- R19: LCSC (none) -> C22975
- R20: LCSC (none) -> C22843
- R21: LCSC (none) -> C22764
- R22: LCSC (none) -> C22935
- R24: footprint (none) -> Resistor_SMD:R_2512_6332Metric; LCSC (none) -> C3000711
- R26: value 10k -> 4.3k; LCSC (none) -> C23159
- R5: LCSC (none) -> C23221
- R7: LCSC (none) -> C13167
- R8: LCSC (none) -> C4216
- R9: value 190k -> 82k; LCSC (none) -> C23254
- U3: footprint (none) -> Package_SO:TSSOP-28-1EP_4.4x9.7mm_P0.65mm_EP2.74x4.75mm; LCSC (none) -> C459912
Other:
- note added: "2uFx10 = 20uF is recommended 30uF is DC-bias accounted value"
- note added: "30V UVLO (1.5V thresh)"
- note removed: "2uFx10 = 20uF is recommended 30uF is DC-bias accounted value Since 10u is big, 0.1u is closer bypass"

Commit message: Record current testboard modifications as schematics
Parts:
- added C12, C13: 10nF 250V, symbol Device:C_Small
- added D5: Vz=100V, symbol Device:D_Zener
- added D6: 150V2A, symbol Device:D_Schottky
- added HS2: 20x15x5mm, symbol Mechanical:Heatsink
- added R11, R23, R27: 10Ω 2W, symbol Device:R
- C26, C27, JP8: now not fitted
Connections:
- net GND: now also D5.2 (A), D6.2 (A), R11.2, R23.2, R27.2
- net at D1.1 (K), J2.1 (Pin_1): now also C12.2, C13.2, D5.1 (K), D6.1 (K)
- new net: C12.1, C13.1, R11.1, R23.1, R27.1
Other:
- note added: "1N5378BRLG"
- note added: "Snubber (R=3.3Ω, C=20nF)"
- moved on the sheet: J2
