File: pcb/PULSER-testboard-hc/PULSER-testboard-hc.kicad_sch (KiCad schematic)
At the start: 109 parts, among them J1 Screw_Terminal 2pin, J2 Screw_Terminal 2pin, J3 Conn_01x02_Pin, J4 Conn_01x02_Pin, Q1 N-ch, Vds>=60V, low Qgs, Q2 N-ch, Vds>=60V, low Rds, U2 LM317_DPAK, U3 LT3763

Commit message: Update HC schem for new connectors (FFC & fan), w/ 12V PSU
Parts:
- removed C1, C4: 1n, Capacitor_SMD:C_0603_1608Metric, symbol Device:C_Small
- removed C10, C11, C21, C22, C23, C24, C25, C26, C27, C28, C29, C30, C31, C32: 10u, Capacitor_SMD:C_1206_3216Metric, symbol Device:C_Small
- removed C13: 10nF 250V, symbol Device:C_Small
- removed C14: 2.2u, Capacitor_SMD:C_1206_3216Metric, symbol Device:C_Small
- removed C15, C16: 0.1u, Capacitor_SMD:C_0603_1608Metric, symbol Device:C_Small
- removed C17, C18: 10n, Capacitor_SMD:C_0603_1608Metric, symbol Device:C_Small
- removed C19, C20, C5: 10u, Capacitor_SMD:C_0805_2012Metric, symbol Device:C_Small
- removed C2: 220n, Capacitor_SMD:C_0603_1608Metric, symbol Device:C_Small
- removed C3: 22n, Capacitor_SMD:C_0603_1608Metric, symbol Device:C_Small
- removed C6: 470p, Capacitor_SMD:C_0603_1608Metric, symbol Device:C_Small
- removed C7: 4.7n, Capacitor_SMD:C_0603_1608Metric, symbol Device:C_Small
- removed D2: 100mA, Diode_SMD:D_SOD-123, symbol Device:D_Schottky
- removed D3: D, Diode_SMD:D_SOD-123, symbol Device:D
- removed D4: Ipeak>10A, SparkAll:TO-227A-2P, symbol Device:D_Schottky
- removed HS1: Heatsink_Pad_2Pin, SparkAll:HS-P23D1.6-30x30, symbol Mechanical:Heatsink_Pad_2Pin
- removed HS2: 20x15x5mm, symbol Mechanical:Heatsink
- removed J4: Conn_01x02_Pin, Connector_PinHeader_2.54mm:PinHeader_1x02_P2.54mm_Vertical, symbol Connector:Conn_01x02_Pin
- removed JP1, JP10, JP11, JP12, JP2, JP3, JP7, JP8, JP9: Jumper_2_Small_Bridged, Jumper:SolderJumper-2_P1.3mm_Bridged_RoundedPad1.0x1.5mm, symbol Jumper:Jumper_2_Small_Bridged
- removed JP13: Jumper_2_Small_Open, Jumper:SolderJumper-2_P1.3mm_Open_RoundedPad1.0x1.5mm, symbol Jumper:Jumper_2_Small_Open
- removed JP4, JP5, JP6: ~, Connector_PinHeader_2.54mm:PinHeader_1x02_P2.54mm_Vertical, symbol Jumper:Jumper_2_Open
- removed L1: 10u, Inductor_SMD:L_Bourns_SRP1245A, symbol Device:L
- removed Q1: N-ch, Vds>=60V, low Qgs, SparkAll:Infineon-TG-TDSON-8-NMOS, symbol Device:Q_NMOS
- removed Q2: N-ch, Vds>=60V, low Rds, SparkAll:Infineon-TG-TDSON-8-NMOS, symbol Device:Q_NMOS
- removed R1, R6: 1, Resistor_SMD:R_1206_3216Metric, symbol Device:R
- removed R10: 120k, Resistor_SMD:R_0603_1608Metric, symbol Device:R
- removed R13, R25: 47k, Resistor_SMD:R_0603_1608Metric, symbol Device:R
- removed R14: 2.4k, Resistor_SMD:R_0603_1608Metric, symbol Device:R
- removed R15: 5.1k, Resistor_SMD:R_0603_1608Metric, symbol Device:R
- removed R16: 11k, Resistor_SMD:R_0603_1608Metric, symbol Device:R
- removed R17: 240, Resistor_SMD:R_0603_1608Metric, symbol Device:R
- removed R18: 390, Resistor_SMD:R_0603_1608Metric, symbol Device:R
- removed R19: 2k, Resistor_SMD:R_0603_1608Metric, symbol Device:R
- removed R2: 5m, Resistor_SMD:R_1206_3216Metric, symbol Device:R
- removed R20: 1.5k, Resistor_SMD:R_0603_1608Metric, symbol Device:R
- removed R21: 1.1k, Resistor_SMD:R_0603_1608Metric, symbol Device:R
- removed R22: 1M, Resistor_SMD:R_0603_1608Metric, symbol Device:R
- removed R23, R27: 10Ω 2W, symbol Device:R
- removed R26: 4.3k, Resistor_SMD:R_0603_1608Metric, symbol Device:R
- removed R3, R4: 10, Resistor_SMD:R_0603_1608Metric, symbol Device:R
- removed R5: 62k, Resistor_SMD:R_0603_1608Metric, symbol Device:R
- removed R7: 2.7k, Resistor_SMD:R_0603_1608Metric, symbol Device:R
- removed R8: 33k, Resistor_SMD:R_0603_1608Metric, symbol Device:R
- removed R9: 82k, Resistor_SMD:R_0603_1608Metric, symbol Device:R
- removed TH1: Thermistor_NTC, Resistor_SMD:R_0603_1608Metric, symbol Device:Thermistor_NTC
- removed TP1, TP10, TP11, TP12, TP13, TP14, TP15, TP16, TP17, TP18, TP2, TP3, TP4, TP5, TP6, TP7, TP9: TestPoint, TestPoint:TestPoint_Pad_D1.5mm, symbol Connector:TestPoint_Small
- removed U2: LM317_DPAK, Package_TO_SOT_SMD:TO-252-2, symbol Regulator_Linear:LM317_TO-252
- removed U3: LT3763, Package_SO:TSSOP-28-1EP_4.4x9.7mm_P0.65mm_EP2.74x4.75mm, symbol SparkAll:LT3763
- added C33, C35: 0.1u, Capacitor_SMD:C_0603_1608Metric, symbol Device:C
- added J6: Conn_01x08_Pin, Connector_FFC-FPC:Molex_200528-0080_1x08-1MP_P1.00mm_Horizontal, symbol Connector:Conn_01x08_Pin
- added U1: ADuM1200AR, Package_SO:SOIC-8_3.9x4.9mm_P1.27mm, symbol Isolator:ADuM1200AR
- C12: value 10nF 250V -> 22n; Rating (none) -> 250V
- C8: value 10n -> 220n; LCSC C57112 -> (none); Rating (none) -> 10V
- C9: value 1uF 50V -> 1u; Rating (none) -> 50V
- D5: Rating (none) -> 5W
- D6: value 150V2A -> ~; Rating (none) -> 150V 2A
- J3: footprint Connector_PinHeader_2.54mm:PinHeader_1x02_P2.54mm_Vertical -> (none); LCSC C492401 -> (none)
- R11: value 10Ω 2W -> 3.3; Rating (none) -> 200V 2W
- R12: Rating (none) -> 10V
- R24: value 1Ω 1W -> 1; Rating (none) -> 1W
Connections:
- net +3V3: now also C35.1, U1.8 (VDD2)
- net EN: now also U1.7 (VOA)
- net GND: now also C35.2, U1.5 (GND2)
- net +12V: now reaches J3.1 (Pin_1)
- net CTRL1 renamed CURR_CTRL
- net CTRL_RAW: no longer names the net of R12.1
- net CTRL_RAW: now also U1.6 (VOB)
- net VOUT renamed highcurrent/VOUT
- new net CURR_S: J6.4 (Pin_4), U1.3 (VIB)
- new net EN_S: J6.3 (Pin_3), U1.2 (VIA)
- new net GNDS: C33.2, J6.2 (Pin_2), J6.5 (Pin_5), U1.4 (GND1)
- new net VCCS: C33.1, J6.1 (Pin_1), U1.1 (VDD1)
Other:
- added sheet highcurrent (highcurrent.kicad_sch)
- added sheet powersupply (powersupply.kicad_sch)
- note added: "1.6W (at 8kHz pulse)"
- note added: "12V fan (max 200mA)"
- note added: "CURR (PWM) * accepted freq: 10kHz~200kHz * working range: 22%(5A) ~ 45% (10A) (0.22A/%) * setting delay: 10ms Below 22%: output current might be unstable compared to ripple Above 45%: clamped to 10A"
- note added: "D1 protection"
- note added: "VCCS=3.3V or 5V current draw: <5mA"
- note added: "fc=72Hz LPF (9kHz 50% -> 1%- ripple)"
- note added: "min pulse width: 1us"
- note added: "stray inductance flywheel"
- note removed: "0.15V/A max 1.5V analog or PWM 1.6kHz low-pass filtered high-side clamp to 2V Zin=1kΩ"
- note removed: "0.4W cond: 0.4W"
- note removed: "0.5W"
- note removed: "1.50V : 10A 0.75V : 5A 0.30V : 2A abs max 3V Vref 2V"
- note removed: "10A"
- note removed: "1N5378BRLG"
- note removed: "22uF is recommended in datasheet account for cap loss by DC-bias 16V+ is recommended"
- note removed: "2A"
- note removed: "2uFx10 = 20uF is recommended 30uF is DC-bias accounted value"
- note removed: "3.1W cond: 1.4W sw: 1.7W"
- note removed: "3.3V"
- note removed: "30V UVLO (1.5V thresh)"
- note removed: "5A"
- note removed: "BSC0702LS"
- note removed: "BSC094N06LS5"
- note removed: "IC"
- note removed: "Isat>12A"
- note removed: "MOSFET"
- note removed: "TO-220 heatsink RΘ<14K/W"
- note removed: "Tstart=30us"
- note removed: "computed using Vo=20V"
- note removed: "fc=1.6kHz LPF"
- note removed: "fc=723kHz"
- note removed: "fs=350kHz"
- note removed: "over-voltage protection 36V (current limited above 29V) FB(OVP)=1.5V FB(limit)=1.21V"
- note removed: "protection"
- title: Pulser V2 HC Test Board -> Pulser V2 HC Board
- moved on the sheet: C12, C8, D1, D5, D6, J2, R11, R12, TP8

Commit message: HC r3 schem draft ok
Parts:
- added D7, D8: LED, LED_SMD:LED_0805_2012Metric, symbol Device:LED
- added R16, R19: 1k, Resistor_SMD:R_0402_1005Metric, symbol Device:R
- C12: footprint (none) -> Capacitor_SMD:C_0805_2012Metric; LCSC (none) -> C5128361; Rating 250V -> 200V
- C33, C35: footprint Capacitor_SMD:C_0603_1608Metric -> Capacitor_SMD:C_0402_1005Metric; LCSC (none) -> C307331
- C8: LCSC (none) -> C21120
- D1: value 120V 10A -> ~; footprint Package_TO_SOT_THT:TO-220-2_Vertical -> SparkAll:VISHAY-SMPC; LCSC C10623 -> C968542; Rating (none) -> 120V 10A
- D5: footprint (none) -> Diode_SMD:D_SMB; LCSC (none) -> C150045; Rating 5W -> 3W
- D6: footprint (none) -> SparkAll:TO-227A-2P; LCSC (none) -> C2927414
- J3: footprint (none) -> Connector_JST:JST_XH_B2B-XH-A_1x02_P2.50mm_Vertical
- R11: footprint (none) -> Resistor_SMD:R_2512_6332Metric; LCSC (none) -> C2960811
- R12: footprint Resistor_SMD:R_0603_1608Metric -> Resistor_SMD:R_0402_1005Metric; LCSC C25804 -> C25744
Connections:
- net +3V3: now also D7.2 (A)
- net EN: now also D8.2 (A)
- net GND: now also R16.1, R19.1
- new net: D7.1 (K), R16.2
- new net: D8.1 (K), R19.2
Other:
- note added: "1.6W (at 8kHz pulse) target: Tj<100C 22 vias (assuming Tjc=20K/W)"
- note added: "6W target: Tj<100C 50 vias"
- note added: "EN"
- note added: "PWR"
- note added: "Thermal environment * via: 300K/W * backside-air: 1.7K/W (only where heatsink exists) * Tair=30C"
- note removed: "1.6W (at 8kHz pulse)"
- note removed: "6W"
