File: pcb/PULSER-testboard-hc/powersupply.kicad_sch (KiCad schematic)
At the start: 13 parts, among them U2 LM317_DPAK, U4 TPSM365R6

Commit message: HC r3 schem draft ok
Parts:
- C15, C16: footprint Capacitor_SMD:C_0603_1608Metric -> Capacitor_SMD:C_0402_1005Metric; LCSC C14663 -> C307331
- C27: LCSC (none) -> C96446
- R14: LCSC (none) -> C138065
- R15: LCSC C25744 -> C513708
- R17: footprint Resistor_SMD:R_0603_1608Metric -> Resistor_SMD:R_0402_1005Metric; LCSC C23350 -> C852660
- R18: footprint Resistor_SMD:R_0603_1608Metric -> Resistor_SMD:R_0402_1005Metric; LCSC C23151 -> C137997
Changed lines of the file:
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@@
 			)
 		)
-		(property "Footprint" "Capacitor_SMD:C_0603_1608Metric"
+		(property "Footprint" "Capacitor_SMD:C_0402_1005Metric"
 			(at 92.71 111.76 0)
 			(effects
@@
 			)
 		)
-		(property "LCSC" "C14663"
+		(property "LCSC" "C307331"
 			(at 92.71 111.76 0)
 			(effects
@@
 			)
 		)
-		(property "Footprint" "Resistor_SMD:R_0603_1608Metric"
+		(property "Footprint" "Resistor_SMD:R_0402_1005Metric"
 			(at 73.152 116.84 90)
 			(effects
@@
 			)
 		)
-		(property "LCSC" "C23151"
+		(property "LCSC" "C137997"
 			(at 74.93 116.84 0)
 			(effects
@@
 			)
 		)
-		(property "LCSC" ""
+		(property "LCSC" "C96446"
 			(at 132.08 62.23 0)
 			(effects
@@
 			)
 		)
-		(property "Footprint" "Capacitor_SMD:C_0603_1608Metric"
+		(property "Footprint" "Capacitor_SMD:C_0402_1005Metric"
 			(at 40.64 110.49 0)
 			(effects
@@
 			)
 		)
-		(property "LCSC" "C14663"
+		(property "LCSC" "C307331"
 			(at 40.64 110.49 0)
 			(effects
@@
 			)
 		)
-		(property "Footprint" "Resistor_SMD:R_0603_1608Metric"
+		(property "Footprint" "Resistor_SMD:R_0402_1005Metric"
 			(at 73.152 106.68 90)
 			(effects
@@
 			)
 		)
-		(property "LCSC" "C23350"
+		(property "LCSC" "C852660"
 			(at 74.93 106.68 0)
 			(effects
@@
 			)
 		)
-		(property "LCSC" ""
+		(property "LCSC" "C138065"
 			(at 120.65 55.88 0)
 			(effects
@@
 			)
 		)
-		(property "LCSC" "C25744"
+		(property "LCSC" "C513708"
 			(at 120.65 66.04 0)
 			(effects
