File: pcb/PULSER-testboard-hv/PULSER-testboard-hv.kicad_pcb (KiCad board)
At the start: 2 copper layers, 30 parts, among them U1 TL783, U10 LMC555xMM, U2 INA281A2, U4 TLV3201, U5 LM317_DPAK, U9 LMC555xMM

Commit message: HV lcsc & footprint assigned
Parts:
- removed the C13 at (130.6, 153.3)
- removed the C15 at (130.6, 158.4)
- added C16: 330p, Capacitor_SMD:C_0603_1608Metric, F.Cu at (234.4, 107.1)
- added C17: 330p, Capacitor_SMD:C_0603_1608Metric, F.Cu at (234.4, 109.6)
- added C18: 470p, Capacitor_SMD:C_0603_1608Metric, F.Cu at (234.4, 112.1)
- added C19: 470p, Capacitor_SMD:C_0603_1608Metric, F.Cu at (234.4, 114.6)
- added C2: 100nF 200V, Capacitor_SMD:C_1206_3216Metric, F.Cu at (221.7, 69.3)
- added C22: 0.1u, Capacitor_SMD:C_0603_1608Metric, F.Cu at (238.4, 107.1)
- added C23: 0.1u, Capacitor_SMD:C_0603_1608Metric, F.Cu at (238.4, 109.6)
- added C4: 0.1u, Capacitor_SMD:C_0603_1608Metric, F.Cu at (221.7, 71.8)
- added C5: 0.1u, Capacitor_SMD:C_0603_1608Metric, F.Cu at (221.7, 74.3)
- added C6: 0.1u, Capacitor_SMD:C_0603_1608Metric, F.Cu at (221.7, 76.8)
- added C7: 0.1u, Capacitor_SMD:C_0603_1608Metric, F.Cu at (194.2, 82.5)
- added C8: 1u, Capacitor_SMD:C_0603_1608Metric, F.Cu at (194.2, 85.0)
- added F1: 2A, Fuse:Fuse_Littelfuse-NANO2-451_453, F.Cu at (224.0, 88.0)
- added J1: Screw_Terminal 2pin, SparkAll:Wurth_TerminalBlock_2pin_P5mm_691137710002, F.Cu at (60.0, 70.9)
- added J2: Screw_Terminal 2pin, SparkAll:Wurth_TerminalBlock_2pin_P5mm_691137710002, F.Cu at (145.0, 70.0)
- added J3: Conn_01x02_Pin, Connector_PinHeader_2.54mm:PinHeader_1x02_P2.54mm_Vertical, F.Cu at (222.0, 63.2)
- added J4: Conn_01x02_Pin, Connector_PinHeader_2.54mm:PinHeader_1x02_P2.54mm_Vertical, F.Cu at (226.6, 63.2)
- added JP1: Jumper_2_Small_Open, Connector_PinHeader_2.54mm:PinHeader_1x02_P2.54mm_Vertical, F.Cu at (231.2, 63.2)
- added JP2: Jumper_2_Small_Open, Connector_PinHeader_2.54mm:PinHeader_1x02_P2.54mm_Vertical, F.Cu at (235.8, 63.2)
- added JP3: Jumper_2_Small_Bridged, Jumper:SolderJumper-2_P1.3mm_Bridged_RoundedPad1.0x1.5mm, F.Cu at (246.6, 69.8)
- added JP4: Jumper_2_Small_Open, Connector_PinHeader_2.54mm:PinHeader_1x02_P2.54mm_Vertical, F.Cu at (240.4, 63.2)
- added JP5: Jumper_2_Small_Bridged, Jumper:SolderJumper-2_P1.3mm_Bridged_RoundedPad1.0x1.5mm, F.Cu at (246.6, 73.4)
- added JP6: Jumper_2_Small_Open, Connector_PinHeader_2.54mm:PinHeader_1x02_P2.54mm_Vertical, F.Cu at (245.0, 63.2)
- added Q2: Q_NMOS_GDS, Package_TO_SOT_SMD:SOT-223-3_TabPin2, F.Cu at (176.8, 80.0)
- added R10: 3.9k, Resistor_SMD:R_0603_1608Metric, F.Cu at (225.8, 81.8)
- added R13: 10k, Resistor_SMD:R_0603_1608Metric, F.Cu at (229.8, 71.8)
- added R14: 270, Resistor_SMD:R_0603_1608Metric, F.Cu at (229.8, 74.3)
- added R15: 820, Resistor_SMD:R_0603_1608Metric, F.Cu at (229.8, 76.8)
- added R20: 2.7k, Resistor_SMD:R_0603_1608Metric, F.Cu at (238.4, 112.1)
- added R21: 5.6k, Resistor_SMD:R_0603_1608Metric, F.Cu at (238.4, 114.6)
- added R22: 10k, Resistor_SMD:R_0603_1608Metric, F.Cu at (242.4, 107.1)
- added R23: 20k, Resistor_SMD:R_0603_1608Metric, F.Cu at (242.4, 109.6)
- added R24: 910, Resistor_SMD:R_0603_1608Metric, F.Cu at (242.4, 112.1)
- added R25: 9.1k, Resistor_SMD:R_0603_1608Metric, F.Cu at (242.4, 114.6)
- added R3: 2.4Ω 120V, Resistor_SMD:R_1206_3216Metric, F.Cu at (221.7, 81.8)
- added R4: 1.3Ω 120V, Resistor_SMD:R_1206_3216Metric, F.Cu at (221.7, 84.3)
- added R5: 0.62Ω 120V, Resistor_SMD:R_1206_3216Metric, F.Cu at (225.8, 69.3)
- added R6: 75k, Resistor_SMD:R_0603_1608Metric, F.Cu at (225.8, 71.8)
- added R7: 82k, Resistor_SMD:R_0603_1608Metric, F.Cu at (225.8, 74.3)
- added R8: 36k, Resistor_SMD:R_0603_1608Metric, F.Cu at (225.8, 76.8)
- added R9: 10k, Resistor_SMD:R_0603_1608Metric, F.Cu at (225.8, 79.3)
- added SW1: SW_DIP_x04, Button_Switch_SMD:SW_DIP_SPSTx04_Slide_9.78x12.34mm_W8.61mm_P2.54mm, F.Cu at (238.1, 75.1)
- added SW2: SW_DIP_x04, Button_Switch_SMD:SW_DIP_SPSTx04_Slide_9.78x12.34mm_W8.61mm_P2.54mm, F.Cu at (220.0, 99.4)
- added SW3: SW_DIP_x02, Button_Switch_SMD:SW_DIP_SPSTx02_Slide_9.78x7.26mm_W8.61mm_P2.54mm, F.Cu at (226.0, 110.9)
- added TP1: TestPoint_Small, TestPoint:TestPoint_Pad_D1.5mm, F.Cu at (233.5, 83.8)
- added TP2: TestPoint_Small, TestPoint:TestPoint_Pad_D1.5mm, F.Cu at (233.5, 87.4)
- added TP3: TestPoint_Small, TestPoint:TestPoint_Pad_D1.5mm, F.Cu at (237.1, 83.8)
- added TP4: TestPoint_Small, TestPoint:TestPoint_Pad_D1.5mm, F.Cu at (237.1, 87.4)
- added TP5: TestPoint_Small, TestPoint:TestPoint_Pad_D1.5mm, F.Cu at (240.6, 83.8)
- added TP6: TestPoint_Small, TestPoint:TestPoint_Pad_D1.5mm, F.Cu at (240.6, 87.4)
- added U3: LTC7001, Package_SO:MSOP-10-1EP_3x3mm_P0.5mm_EP1.68x1.88mm, F.Cu at (195.9, 79.0)
- added U6: LT8365, SparkAll:AD-MSOP-LT8365, F.Cu at (194.0, 69.4)
- added U7: 74HC00, Package_SO:TSSOP-14_4.4x5mm_P0.65mm, F.Cu at (236.7, 95.8)
- added U8: 74HC00, Package_SO:TSSOP-14_4.4x5mm_P0.65mm, F.Cu at (250.0, 102.5)
- C1: value 1u -> 100nF 200V; footprint Capacitor_SMD:C_0603_1608Metric -> Capacitor_SMD:C_1206_3216Metric
- C10: renamed from C6; footprint Capacitor_SMD:C_0805_2012Metric -> Capacitor_SMD:C_1206_3216Metric
- C11: renamed from C7; value 1uF -> 1u
- C12: renamed from C8; value 0.22uF -> 0.22u
- C13: renamed from C9; value 1nF -> 1n
- C3: renamed from C2; value 0.1u -> 100nF 200V; footprint Capacitor_SMD:C_0603_1608Metric -> Capacitor_SMD:C_1206_3216Metric
- D1: value 150V 1A -> 150V 2A; footprint Diode_SMD:D_PowerDI-123 -> Diode_SMD:D_SMC
- D2: value 150V 1A, Schottky bigger -> 150V 2A; footprint Diode_SMD:D_PowerDI-123 -> Diode_SMD:D_SMC
- R1: value 100m -> 100mΩ 120V; footprint Resistor_SMD:R_0603_1608Metric -> Resistor_SMD:R_1206_3216Metric
- R11: value 8.2k -> 9.1k
- R16: renamed from R7; footprint Resistor_SMD:R_0805_2012Metric -> Resistor_SMD:R_1206_3216Metric
- R2: value 2.5 -> 6.2Ω 120V; footprint Resistor_SMD:R_0603_1608Metric -> Resistor_SMD:R_1206_3216Metric
- U1: footprint Package_TO_SOT_SMD:TO-263-3_TabPin2 -> Package_TO_SOT_THT:TO-220-3_Vertical
- U10, U9: footprint Package_SO:VSSOP-8_3x3mm_P0.65mm -> Package_SO:SOIC-8_3.9x4.9mm_P1.27mm
- moved R12 136.7 mm to (229.8, 69.3)
- moved R11 122.1 mm to (225.8, 84.3)
- moved R2 108.1 mm to (221.7, 79.3)
- moved C10 85.0 mm to (206.5, 138.6)
- moved C11 85.0 mm to (190.6, 124.1)
- moved C12 85.0 mm to (190.6, 126.6)
- moved C13 85.0 mm to (190.6, 129.2)
- moved C14 85.0 mm to (212.7, 124.1)
- moved C15 85.0 mm to (212.7, 126.6)
- moved C20 85.0 mm to (212.7, 129.2)
- moved C21 85.0 mm to (212.7, 134.2)
- moved D2 85.0 mm to (195.6, 138.9)
- moved R17 85.0 mm to (190.6, 131.7)
- moved R18 85.0 mm to (190.6, 134.2)
- moved R19 85.0 mm to (190.6, 136.7)
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- renumbered C10 to C14, C11 to C15, C12 to C20, C14 to C21, C5 to C9, R8 to R17, R9 to R18, R10 to R19
Connections:
- net Net-(D1-A) renamed /IR_AD
- C1 pad 1: Net-(U1-IN) -> /Boost Converter/VOUT
- R11 pad 1: Net-(U9-DISCH) -> /VTH_100
- R11 pad 2: +5V -> GND
- R12 pad 1: Net-(U10-DISCH) -> /VTH_200
- R12 pad 2: +5V -> GND
- R2 pad 1: Net-(U1-OUT) -> Net-(JP1-B)
- U1 pad 2: Net-(U1-OUT) -> /IR_VO
- U10 pad 6: Net-(U10-DISCH) -> /Pulse Controller/TH_CL
- U10 pad 7: Net-(U10-DISCH) -> /Pulse Controller/TH_CL
- U4 pad 4: Net-(U4--) -> /VTH
- U9 pad 6: Net-(U9-DISCH) -> /Pulse Controller/TH_P
- U9 pad 7: Net-(U9-DISCH) -> /Pulse Controller/TH_P
Other:
- board outline added: 100 x 100 mm

Commit message: HC, HV: PCB DRC pass
Parts:
- added G***: LOGO, LOGO, F.Cu at (131.4, 130.3)
- added R26: 10M, Resistor_SMD:R_0603_1608Metric, F.Cu at (76.2, 121.5)
- added R27: 10M, Resistor_SMD:R_0603_1608Metric, F.Cu at (90.5, 121.8)
- added TP10: TestPoint_Small, TestPoint:TestPoint_Pad_D1.5mm, F.Cu at (84.8, 104.3)
- added TP12: TestPoint_Small, TestPoint:TestPoint_Pad_D1.5mm, F.Cu at (135.4, 111.1)
- added TP13: TestPoint_Small, TestPoint:TestPoint_Pad_D1.5mm, F.Cu at (135.5, 117.4)
- added TP14: TestPoint_Small, TestPoint:TestPoint_Pad_D1.5mm, F.Cu at (97.1, 107.9)
- added TP7: TestPoint_Small, TestPoint:TestPoint_Pad_D1.5mm, F.Cu at (76.2, 116.0)
- added TP8: TestPoint_Small, TestPoint:TestPoint_Pad_D1.5mm, F.Cu at (90.5, 116.0)
- added TP9: TestPoint_Small, TestPoint:TestPoint_Pad_D1.5mm, F.Cu at (68.0, 104.3)
- moved R20 175.7 mm to (64.0, 133.8), turned to 90 degrees
- moved R22 174.4 mm to (70.0, 133.8), turned to 90 degrees
- moved C16 173.0 mm to (64.0, 137.4), turned to 90 degrees
- moved R21 172.4 mm to (67.0, 133.8), turned to 90 degrees
- moved R23 171.1 mm to (73.0, 133.8), turned to 90 degrees
- moved C17 169.6 mm to (67.0, 137.4), turned to 90 degrees
- moved J3 169.3 mm to (75.0, 147.0), turned to 90 degrees
- moved C18 166.3 mm to (70.0, 137.4), turned to 90 degrees
- moved R14 163.3 mm to (67.0, 88.1), turned to 90 degrees
- moved R15 163.0 mm to (67.0, 84.9), turned to 90 degrees
- moved C19 163.0 mm to (73.0, 137.4), turned to 90 degrees
- moved F1 159.2 mm to (65.0, 78.5)
- moved R24 159.2 mm to (84.7, 133.9), turned to 90 degrees
- moved C22 156.6 mm to (84.7, 137.5), turned to 90 degrees
- moved R25 155.8 mm to (87.7, 133.9), turned to 90 degrees
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- renumbered Q2 to Q1
Connections:
- C7 pad 1: Net-(C7-Pad1) -> GND
- C8 pad 1: Net-(C7-Pad1) -> GND
- R15 pad 2: Net-(C7-Pad1) -> GND
Routing:
- net /Pulse Controller/PULSE: track 0.00 -> 96.2 mm
- net +5V: track 0.00 -> 93.1 mm, vias 0 -> 22
- net /CURR: track 0.00 -> 84.2 mm, vias 0 -> 2
- net /GATE: track 0.00 -> 84.0 mm, vias 0 -> 2
- net /Pulse Controller/COOLDOWN: track 0.00 -> 69.5 mm
- net /EN: track 0.00 -> 65.8 mm
- net Net-(U2-OUT): track 0.00 -> 61.4 mm, vias 0 -> 2
- net +36V: track 0.00 -> 58.2 mm
- net /IR_VO: track 0.00 -> 48.9 mm
- net /IR_AD: track 0.00 -> 46.6 mm
- net Net-(Q1-S): track 0.00 -> 40.5 mm, vias 0 -> 2
- net /Pulse Controller/TH_P: track 0.00 -> 38.4 mm
- net /Pulse Controller/~{CURR}: track 0.00 -> 37.2 mm, vias 0 -> 3
- net /Pulse Controller/GATE_OK: track 0.00 -> 35.1 mm
- net Net-(U1-IN): track 0.00 -> 26.0 mm
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- added copper zone on F.Cu, net +36V
- added copper zone on B.Cu, net +5V
- added copper zone on F.Cu, net +5V
- added copper zone on F.Cu, net /Boost Converter/VOUT
- added copper zone on B.Cu, net GND
- added copper zone on F.Cu, net GND
- added copper zone on In1.Cu, net GND
- added copper zone on In2.Cu, net GND
- added copper zone on F.Cu, net Net-(D2-A)
- added copper zone on F.Cu, net Net-(Q1-S)
- added copper zone on F.Cu, net Net-(U1-IN)
Other:
- copper layers 2 -> 4
- board text added: "*"
- board text added: "+"
- board text added: "-"
- board text added: ".05"
- board text added: ".1"
- board text added: ".2"
- board text added: ".5"
- board text added: "1"
- board text added: "10"
- board text added: "2"
- board text added: "5"
- board text added: "COOL[ms]"
- board text added: "CURR"
- board text added: "CURR[A]"
- board text added: "CURR_th[A]"
- board text added: "EN"
- board text added: "GND"
- board text added: "HIGH VOLTAGE"
- board text added: "HV Test Board r1"
- board text added: "IN 36V 2A"
- board text added: "OUT PULSE"
- board text added: "PULSE[us]"
- board text added: "SN"
- board text added: "outer: 35um (1oz) inner: 17um (0.5oz)"
- board text added: "Φ3.2"

Commit message: Add I/O descs
Other:
- board text added: "IN digital 3.3V - 5V"
- board text added: "OUT digital 5V"
Changed lines of the file:
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@@
 		(tags "Through hole pin header THT 1x02 2.54mm single row")
 		(property "Reference" "J4"
-			(at 0 5.54 180)
+			(at 0 -2.955 180)
 			(layer "F.SilkS")
 			(effects
@@
 		(tags "Through hole pin header THT 1x02 2.54mm single row")
 		(property "Reference" "J3"
-			(at 0 5.54 180)
+			(at 0 -2.71 180)
 			(layer "F.SilkS")
 			(effects
@@
 		)
 	)
+	(gr_text "IN digital\n3.3V - 5V"
+		(at 79.75 148.25 0)
+		(layer "F.SilkS")
+		(effects
+			(font
+				(size 1 1)
+				(thickness 0.25)
+			)
+			(justify left bottom)
+		)
+	)
 	(gr_text "5"
 		(at 69 118.5 0)
@@
 		(layer "F.SilkS")
 		(effects
+			(font
+				(size 1 1)
+				(thickness 0.25)
+			)
+			(justify left bottom)
+		)
+	)
+	(gr_text "OUT digital\n5V"
+		(at 113.5 148.25 0)
+		(layer "F.SilkS")
+		(effects
