File: pcb/PULSER-testboard-hv/PULSER-testboard-hv.kicad_pcb (KiCad board)
At the start: 4 copper layers, 100 x 100 mm, 92 parts, among them J1 Screw_Terminal 2pin, J2 Screw_Terminal 2pin, J3 Conn_01x02_Pin, J4 Conn_01x02_Pin, Q1 Q_NMOS_GDS, SW1 SW_DIP_x04, SW2 SW_DIP_x04, SW3 SW_DIP_x02, U1 TL783, U10 LMC555xMM, U2 INA281A2, U3 LTC7001, U4 TLV3201, U5 LM317_DPAK, U6 LT8365, U7 74HC00, U8 74HC00, U9 LMC555xMM

Commit message: HV TestBoard r2 pcb ok
Parts:
- removed C14, C15, C20, C22, C23: 0.1u, Capacitor_SMD:C_0603_1608Metric
- removed C16, C17: 330p, Capacitor_SMD:C_0603_1608Metric
- removed C18, C19: 470p, Capacitor_SMD:C_0603_1608Metric
- removed C2: 100nF 200V, Capacitor_SMD:C_1206_3216Metric
- removed JP6: Jumper_2_Small_Open, Connector_PinHeader_2.54mm:PinHeader_1x02_P2.54mm_Vertical
- removed R10: 3.9k, Resistor_SMD:R_0603_1608Metric
- removed R11, R12, R25: 9.1k, Resistor_SMD:R_0603_1608Metric
- removed R13, R22, R9: 10k, Resistor_SMD:R_0603_1608Metric
- removed R2: 6.2Ω 120V, Resistor_SMD:R_1206_3216Metric
- removed R23: 20k, Resistor_SMD:R_0603_1608Metric
- removed R24: 910, Resistor_SMD:R_0603_1608Metric
- removed R26, R27: 10M, Resistor_SMD:R_0603_1608Metric
- removed R3: 2.4Ω 120V, Resistor_SMD:R_1206_3216Metric
- removed R4: 1.3Ω 120V, Resistor_SMD:R_1206_3216Metric
- removed R5: 0.62Ω 120V, Resistor_SMD:R_1206_3216Metric
- removed R8: 36k, Resistor_SMD:R_0603_1608Metric
- removed U1: TL783, Package_TO_SOT_THT:TO-220-3_Vertical
- removed U10, U9: LMC555xMM, Package_SO:SOIC-8_3.9x4.9mm_P1.27mm
- removed U7, U8: 74HC00, Package_SO:TSSOP-14_4.4x5mm_P0.65mm
- added D3: LED, LED_SMD:LED_0603_1608Metric, F.Cu at (98.0, 119.6)
- added D4: LED, LED_SMD:LED_0603_1608Metric, F.Cu at (94.9, 119.6)
- added D5: 150V 2A, Diode_SMD:D_SMC, F.Cu at (113.0, 72.4)
- added J5: Conn_01x02_Socket, Connector_PinSocket_2.54mm:PinSocket_1x02_P2.54mm_Vertical, F.Cu at (61.3, 107.4)
- added L2: 220u, Inductor_THT:L_Toroid_Vertical_L16.0mm_W8.0mm_P7.62mm, F.Cu at (138.5, 91.5)
- added L3: 220u, Inductor_THT:L_Toroid_Vertical_L16.0mm_W8.0mm_P7.62mm, F.Cu at (126.5, 91.5)
- added L4: 220u, Inductor_THT:L_Toroid_Vertical_L16.0mm_W8.0mm_P7.62mm, F.Cu at (118.9, 108.5)
- added L5: 220u, Inductor_THT:L_Toroid_Vertical_L16.0mm_W8.0mm_P7.62mm, F.Cu at (131.0, 108.5)
- added TP11: TestPoint_Small, TestPoint:TestPoint_Pad_D1.5mm, F.Cu at (81.0, 101.9)
- added U11: ATtiny1616-M, Package_DFN_QFN:VQFN-20-1EP_3x3mm_P0.4mm_EP1.7x1.7mm, F.Cu at (73.7, 108.8)
- R20: value 2.7k -> 100k
- R21: value 5.6k -> 100k
- R6: value 75k -> 10k
- R7: value 82k -> 10k
- SW1, SW2: value SW_DIP_x04 -> SW_DIP_x02; footprint Button_Switch_SMD:SW_DIP_SPSTx04_Slide_9.78x12.34mm_W8.61mm_P2.54mm -> Button_Switch_SMD:SW_DIP_SPSTx02_Slide_9.78x7.26mm_W8.61mm_P2.54mm
- moved TP13 61.7 mm to (75.8, 101.9), turned to 90 degrees
- moved TP12 57.7 mm to (78.4, 101.9), turned to 90 degrees
- moved JP2 35.3 mm to (134.8, 129.1), turned to 90 degrees
- moved JP1 33.0 mm to (134.8, 125.0), turned to 90 degrees
- moved R20 32.6 mm to (85.6, 109.4), turned to -90 degrees
- moved TP14 29.7 mm to (67.5, 105.5)
- moved TP9 28.5 mm to (96.5, 105.8)
- moved R21 27.5 mm to (65.0, 106.4), turned to -90 degrees
- moved SW1 27.0 mm to (74.2, 121.8)
- moved JP4 26.4 mm to (134.7, 121.0), turned to 90 degrees
- moved D1 22.9 mm to (145.0, 97.1), turned to -90 degrees
- moved TP7 21.6 mm to (96.5, 108.5)
- moved SW3 21.5 mm to (64.0, 121.8)
- moved U4 21.5 mm to (97.0, 99.2)
- moved C6 21.4 mm to (100.5, 100.4)
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Connections:
- D1 pad 2: /IR_AD -> Net-(D1-A)
- JP1 pad 1: /IR_VO -> Net-(JP1-A)
- JP1 pad 2: Net-(JP1-B) -> Net-(D1-A)
- JP2 pad 1: /IR_VO -> Net-(JP2-A)
- JP2 pad 2: Net-(JP2-B) -> Net-(D1-A)
- JP4 pad 1: /IR_VO -> Net-(JP4-A)
- JP4 pad 2: Net-(JP4-B) -> Net-(D1-A)
- R20 pad 1: /Pulse Controller/TH_P_1 -> /GATE
- R20 pad 2: +5V -> GND
- R21 pad 1: /Pulse Controller/TH_P_2 -> +5V
- R21 pad 2: +5V -> /Pulse Controller/UPDI
- R6 pad 1: +5V -> Net-(D3-K)
- R6 pad 2: /VTH_50 -> GND
- R7 pad 1: +5V -> Net-(D4-K)
- R7 pad 2: /VTH_100 -> GND
- SW1 pad 1: /VTH_50 -> Net-(U11-PB2)
- SW1 pad 2: /VTH_100 -> Net-(U11-PB3)
- SW1 pad 3: /VTH_200 -> GND
- SW1 pad 4: /VTH_500 -> GND
- SW2 pad 1: /Pulse Controller/TH_P_1 -> Net-(U11-PB4)
- SW2 pad 2: /Pulse Controller/TH_P_2 -> Net-(U11-PB5)
- SW2 pad 3: /Pulse Controller/TH_P_5 -> GND
- SW2 pad 4: /Pulse Controller/TH_P_10 -> GND
- SW3 pad 1: /Pulse Controller/TH_CL_0.1m -> Net-(U11-PB0)
- SW3 pad 2: /Pulse Controller/TH_CL_1m -> Net-(U11-PB1)
- SW3 pad 3: /Pulse Controller/TH_CL -> GND
- SW3 pad 4: /Pulse Controller/TH_CL -> GND
- TP10 pad 1: /Pulse Controller/COOLDOWN -> /CURR
- TP12 pad 1: /Pulse Controller/GATE_OK -> Net-(U11-PA2)
- TP13 pad 1: /GATE -> Net-(U11-PA3)
- TP14 pad 1: /Pulse Controller/~{CURR} -> /Pulse Controller/UPDI
- TP4 pad 1: /IR_AD -> Net-(D1-A)
- TP7 pad 1: /Pulse Controller/TH_P -> /GATE
- TP8 pad 1: /Pulse Controller/TH_CL -> /VTH
- TP9 pad 1: /Pulse Controller/PULSE -> Net-(U2-OUT)
Routing:
- net /Pulse Controller/PULSE: track 96.2 -> 0.00 mm
- net Net-(D1-A): track 0.00 -> 87.2 mm, vias 0 -> 2
- net /Pulse Controller/COOLDOWN: track 69.5 -> 0.00 mm
- net Net-(JP2-A): track 0.00 -> 55.6 mm
- net +5V: track 93.1 -> 143.7 mm, vias 22 -> 2
- net /IR_VO: track 48.9 -> 0.00 mm
- net /IR_AD: track 46.6 -> 0.00 mm
- net Net-(JP1-A): track 0.00 -> 45.4 mm
- net /Pulse Controller/TH_P: track 38.4 -> 0.00 mm
- net /Pulse Controller/~{CURR}: track 37.2 -> 0.00 mm, vias 3 -> 0
- net /Pulse Controller/GATE_OK: track 35.1 -> 0.00 mm
- net Net-(U11-PB5): track 0.00 -> 31.6 mm, vias 0 -> 2
- net Net-(D4-A): track 0.00 -> 27.9 mm, vias 0 -> 2
- net Net-(U11-PB4): track 0.00 -> 27.5 mm, vias 0 -> 2
- net Net-(U2-Vin-): track 26.0 -> 53.4 mm
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- removed copper zone on B.Cu, net +5V
- removed copper zone on B.Cu, net GND
- removed copper zone on F.Cu, net GND
Other:
- board text added: "00: .05 01: .1* 10: .2 11: .5"
- board text added: "00: .1* 01: 1 10: reserved 11: reserved"
- board text added: "00: 1 01: 2 10: 5* 11: 10"
- board text added: "5V"
- board text added: "AMP"
- board text added: "ATTiny1616"
- board text added: "CURR_max[A]"
- board text added: "GATE"
- board text added: "HV Test Board r2"
- board text added: "N/C"
- board text added: "P=10us 1.2 1.6 2.2 4.6 (risky)"
- board text added: "P=5us 0.6 0.8 1.1 2.3"
- board text added: "STAT"
- board text added: "UPDI"
- board text added: "VTH"
- board text removed: "*"
- board text removed: ".05"
- board text removed: ".1"
- board text removed: ".2"
- board text removed: ".5"
- board text removed: "1"
- board text removed: "10"
- board text removed: "2"
- board text removed: "5"
- board text removed: "CURR[A]"
- board text removed: "HV Test Board r1"

Commit message: P2HV r3 PCB
Parts:
- added C2: 1uF 200V, Capacitor_SMD:C_1812_4532Metric, F.Cu at (99.0, 61.4)
- added D6: 150V 250mA, Diode_SMD:D_TUMD2, F.Cu at (103.0, 87.7)
- added JP6: Jumper_2_Small_Open, Jumper:SolderJumper-2_P1.3mm_Open_RoundedPad1.0x1.5mm, F.Cu at (120.5, 79.1)
- added R2: 10, Resistor_SMD:R_2512_6332Metric, F.Cu at (120.6, 75.4)
- added R3: 100k, Resistor_SMD:R_1206_3216Metric, F.Cu at (138.5, 78.0)
- R6: value 10k -> 1k
- R7: value 10k -> 4.7k
- moved C1 1.19 mm to (102.6, 62.1)
- moved D5 0.20 mm to (113.2, 72.4)
Connections:
- D5 pad 2: GND -> Net-(D5-A)
Routing:
- net Net-(D5-A): track 0.00 -> 9.22 mm
- net Net-(D1-K): track 15.5 -> 20.6 mm
- net /Boost Converter/VOUT: track 17.6 -> 14.4 mm
- net GND: track 31.7 -> 34.3 mm, vias 132 -> 138
- net +5V: track 143.7 -> 146.3 mm
- net Net-(D6-K): track 8.36 -> 10.6 mm
- added copper zone on F.Cu, net GND
Other:
- board text added: "HV Test Board r${REVISION}"
- board text removed: "HV Test Board r2"
