File: pcb/PULSER-testboard-hv/PULSER-testboard-hv.kicad_pcb (KiCad board)
At the start: 4 copper layers, 100 x 100 mm, 75 parts, among them J1 Screw_Terminal 2pin, J2 Screw_Terminal 2pin, J3 Conn_01x02_Pin, J4 Conn_01x02_Pin, J5 Conn_01x02_Socket, Q1 Q_NMOS_GDS, SW1 SW_DIP_x02, SW2 SW_DIP_x02, SW3 SW_DIP_x02, U11 ATtiny1616-M, U2 INA281A2, U3 LTC7001, U4 TLV3201, U5 LM317_DPAK, U6 LT8365

Commit message: pulser v2 HV r4 pcb draft ok
Parts:
- removed J3, J4: Conn_01x02_Pin, Connector_PinHeader_2.54mm:PinHeader_1x02_P2.54mm_Vertical
- removed JP1, JP2, JP4: Jumper_2_Small_Open, Connector_PinHeader_2.54mm:PinHeader_1x02_P2.54mm_Vertical
- removed JP3, JP5: Jumper_2_Small_Bridged, Jumper:SolderJumper-2_P1.3mm_Bridged_RoundedPad1.0x1.5mm
- removed JP6: Jumper_2_Small_Open, Jumper:SolderJumper-2_P1.3mm_Open_RoundedPad1.0x1.5mm
- removed L2, L3, L4, L5: 220u, Inductor_THT:L_Toroid_Vertical_L16.0mm_W8.0mm_P7.62mm
- removed SW1, SW2, SW3: SW_DIP_x02, Button_Switch_SMD:SW_DIP_SPSTx02_Slide_9.78x7.26mm_W8.61mm_P2.54mm
- removed TP12, TP13, TP14: TestPoint_Small, TestPoint:TestPoint_Pad_D1.5mm
- added C14: 0.1u, Capacitor_SMD:C_0603_1608Metric, F.Cu at (139.1, 63.0)
- added C15: 0.1u, Capacitor_SMD:C_0603_1608Metric, F.Cu at (124.2, 63.0)
- added C16: 0.1u, Capacitor_SMD:C_0603_1608Metric, F.Cu at (139.2, 68.1)
- added C17: 0.1u, Capacitor_SMD:C_0603_1608Metric, F.Cu at (124.2, 68.0)
- added C18: 0.1u, Capacitor_SMD:C_0603_1608Metric, F.Cu at (93.1, 59.4)
- added C19: 1u, Capacitor_SMD:C_0603_1608Metric, F.Cu at (102.4, 59.3)
- added D7: LED, LED_SMD:LED_0603_1608Metric, F.Cu at (147.5, 80.0)
- added J6: Conn_01x08_Pin, Connector_FFC-FPC:Molex_200528-0080_1x08-1MP_P1.00mm_Horizontal, F.Cu at (131.5, 56.1)
- added R4: 100, SparkAll:Bourns-TO508P1229X317-3N, F.Cu at (71.0, 85.9)
- added R5: 560, Resistor_SMD:R_0603_1608Metric, F.Cu at (103.1, 56.4)
- added R8: 4.7k, Resistor_SMD:R_0603_1608Metric, F.Cu at (103.1, 53.4)
- added U1: ADuM1200AR, Package_SO:SOIC-8_3.9x4.9mm_P1.27mm, F.Cu at (134.6, 65.5)
- added U7: ADuM1200AR, Package_SO:SOIC-8_3.9x4.9mm_P1.27mm, F.Cu at (128.6, 65.5)
- added U8: LM317_DPAK, Package_TO_SOT_SMD:TO-252-2, F.Cu at (97.5, 54.9)
- L1: value 100uH, Isat=2.7A -> 150uH
- R16: value 470k 150V -> 430k
- R2: value 10 -> 4.7k; footprint Resistor_SMD:R_2512_6332Metric -> Resistor_SMD:R_0603_1608Metric
- moved J2 90.4 mm to (55.0, 84.0), turned to -90 degrees
- moved J5 88.5 mm to (147.5, 87.2)
- moved D1 83.6 mm to (63.0, 80.9)
- moved R3 83.6 mm to (55.0, 76.0), turned to 90 degrees
- moved TP4 77.5 mm to (62.5, 94.5)
- moved R7 74.0 mm to (147.5, 70.6), turned to 180 degrees
- moved D4 70.8 mm to (147.5, 72.2), turned to 180 degrees
- moved R6 69.1 mm to (147.5, 74.5), turned to 180 degrees
- moved R21 68.6 mm to (130.9, 87.5)
- moved C8 66.5 mm to (116.5, 59.3)
- moved G*** 66.1 mm to (120.0, 73.0)
- moved D3 66.0 mm to (147.5, 76.0), turned to 180 degrees
- moved TP3 65.6 mm to (68.5, 94.5)
- moved C21 61.7 mm to (131.6, 84.6), turned to 180 degrees
- moved U5 60.9 mm to (111.6, 54.9), turned to 0 degrees
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Connections:
- C4 pad 1: +5V -> +12V
- C7 pad 2: +36V -> +12V
- D5 pad 2: Net-(D5-A) -> GND
- D6 pad 2: +5V -> +12V
- R2 pad 1: Net-(D5-A) -> Net-(D7-K)
- U11 pad 1: Net-(U11-PA2) -> unconnected-(U11-PA2-Pad1)
- U11 pad 10: Net-(U11-PB4) -> unconnected-(U11-PB4-Pad10)
- U11 pad 11: Net-(U11-PB3) -> unconnected-(U11-PB3-Pad11)
- U11 pad 12: Net-(U11-PB2) -> unconnected-(U11-PB2-Pad12)
- U11 pad 13: Net-(U11-PB1) -> unconnected-(U11-PB1-Pad13)
- U11 pad 14: Net-(U11-PB0) -> /~{FAULT}
- U11 pad 17: unconnected-(U11-PC2-Pad17) -> Net-(D7-A)
- U11 pad 2: Net-(U11-PA3) -> unconnected-(U11-PA3-Pad2)
- U11 pad 9: Net-(U11-PB5) -> unconnected-(U11-PB5-Pad9)
- U3 pad 1: +5V -> +12V
- U3 pad 2: Net-(JP3-B) -> GND
- U3 pad 5: Net-(JP5-B) -> GND
- U5 pad 3: +36V -> +12V
Routing:
- net Net-(D1-A): track 87.2 -> 16.9 mm, vias 2 -> 0
- net +5V: track 146.3 -> 81.0 mm, vias 2 -> 10
- net Net-(JP2-A): track 55.6 -> 0.00 mm
- net +12V: track 0.00 -> 55.2 mm
- net Net-(JP1-A): track 45.4 -> 0.00 mm
- net /Boost Converter/VOUT: track 14.4 -> 56.0 mm, vias 0 -> 2
- net Net-(U2-Vin-): track 53.4 -> 16.4 mm
- net Net-(U2-OUT): track 68.4 -> 36.1 mm, vias 4 -> 2
- net Net-(U11-PB5): track 31.6 -> 0.00 mm, vias 2 -> 0
- net Net-(D7-A): track 0.00 -> 28.1 mm, vias 0 -> 2
- net Net-(U11-PB4): track 27.5 -> 0.00 mm, vias 2 -> 0
- net Net-(U11-PB1): track 26.6 -> 0.00 mm, vias 2 -> 0
- net Net-(U11-PB0): track 25.7 -> 0.00 mm, vias 2 -> 0
- net Net-(U11-PB2): track 22.3 -> 0.00 mm, vias 2 -> 0
- net GND: track 34.3 -> 15.3 mm, vias 138 -> 253
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- added copper zone on In2.Cu, net +5V
- added copper zone on B.Cu, net GND
- added copper zone on In1.Cu, net GNDS
- added copper zone on In2.Cu, net GNDS
- added copper zone on F.Cu, net Net-(D1-A)
- added copper zone on F.Cu, net Net-(D1-K)
- added copper zone on In2.Cu, net VCCS
- removed copper zone on F.Cu, net +5V
Other:
- board size 100 x 100 mm -> 100 x 50 mm
- board text added: "2A"
- board text added: "CTRL"
- board text added: "FLT"
- board text added: "I+(36V)"
- board text added: "I-"
- board text added: "O+"
- board text added: "O-"
- board text added: "PWR"
- board text added: "UPDI(5V)"
- board text added: "pulser-v2/HV-r${REVISION}"
- board text added: "Φ3.3"
- board text removed: "+"
- board text removed: "-"
- board text removed: "00: .05 01: .1* 10: .2 11: .5"
- board text removed: "00: .1* 01: 1 10: reserved 11: reserved"
- board text removed: "00: 1 01: 2 10: 5* 11: 10"
- board text removed: "5V"
- board text removed: "AMP"
- board text removed: "COOL[ms]"
- board text removed: "CURR_max[A]"
- board text removed: "CURR_th[A]"
- board text removed: "EN"
- board text removed: "GATE"
- board text removed: "HV Test Board r${REVISION}"
- board text removed: "IN 36V 2A"
- board text removed: "IN digital 3.3V - 5V"
- board text removed: "N/C"
- board text removed: "OUT PULSE"
- board text removed: "OUT digital 5V"
- board text removed: "P=10us 1.2 1.6 2.2 4.6 (risky)"
- board text removed: "P=5us 0.6 0.8 1.1 2.3"
- board text removed: "PULSE[us]"
- board text removed: "STAT"
- board text removed: "UPDI"
- board text removed: "VTH"
- board text removed: "Φ3.2"
