File: pcb/PULSER-testboard-hv/PULSER-testboard-hv.kicad_pcb (KiCad board)
At the start: 4 copper layers, 100 x 50 mm, 71 parts, among them J1 Screw_Terminal 2pin, J2 Screw_Terminal 2pin, J5 Conn_01x02_Socket, J6 Conn_01x08_Pin, Q1 Q_NMOS_GDS, U1 ADuM1200AR, U11 ATtiny1616-M, U2 INA281A2, U3 LTC7001, U4 TLV3201, U5 LM317_DPAK, U6 LT8365, U7 ADuM1200AR, U8 LM317_DPAK

Commit message: Add 12V fan connector & sw 12V converter to HV
Parts:
- removed C18: 0.1u, Capacitor_SMD:C_0603_1608Metric
- removed C19: 1u, Capacitor_SMD:C_0603_1608Metric
- removed R5: 560, Resistor_SMD:R_0603_1608Metric
- removed R8: 4.7k, Resistor_SMD:R_0603_1608Metric
- removed U8: LM317_DPAK, Package_TO_SOT_SMD:TO-252-2
- added C26: 1u, Capacitor_SMD:C_0402_1005Metric, F.Cu at (115.4, 53.3)
- added C27: 10u, Capacitor_SMD:C_0603_1608Metric, F.Cu at (109.1, 57.3)
- added C29: 1u, Capacitor_SMD:C_0603_1608Metric, F.Cu at (109.1, 54.1)
- added C30: 1u, Capacitor_SMD:C_0603_1608Metric, F.Cu at (109.1, 55.6)
- added J3: Conn_01x02_Pin, Connector_JST:JST_XH_B2B-XH-A_1x02_P2.50mm_Vertical, F.Cu at (97.4, 53.4)
- added R10: 10k, Resistor_SMD:R_0402_1005Metric, F.Cu at (116.6, 57.4)
- added R9: 110k, Resistor_SMD:R_0402_1005Metric, F.Cu at (115.5, 57.4)
- added TP12: TestPoint, TestPoint:TestPoint_Pad_D1.5mm, F.Cu at (105.5, 52.4)
- added U9: TPSM365R6, SparkAll:TI-RDN0011A-MFG, F.Cu at (112.8, 55.9)
- moved U5 8.58 mm to (113.0, 63.4)
- moved C8 8.43 mm to (115.8, 67.7)
- moved C7 5.75 mm to (105.8, 64.8), turned to -90 degrees
- moved R14 5.21 mm to (118.7, 61.4)
- moved R15 5.21 mm to (118.7, 58.4)
Routing:
- net +36V: track 62.9 -> 35.2 mm, vias 0 -> 2
- net +12V: track 55.2 -> 40.7 mm, vias 0 -> 6
- net Net-(U8-ADJ): track 12.7 -> 0.00 mm, vias 2 -> 0
- net Net-(U9-BIAS): track 0.00 -> 10.4 mm
- net Net-(U9-PGOOD): track 0.00 -> 6.53 mm
- net +5V: track 81.0 -> 87.2 mm
- net GND: track 15.3 -> 18.2 mm, vias 253 -> 256
- net /GATE: track 59.6 -> 57.5 mm, vias 4 -> 2
- net Net-(U9-VCC): track 0.00 -> 1.29 mm
- net Net-(U5-ADJ): track 12.7 -> 12.9 mm, vias 2 -> 0
- added copper zone on In2.Cu, net +12V
- added copper zone on In2.Cu, net +36V
Other:
- board text added: "+"
- board text added: "FAN (12V)"
