File: pcb/PULSER-testboard-hv/boost.kicad_sch (KiCad schematic)
At the start: 12 parts, among them U4 LT8365

Commit message: HV schem draft ok
Parts:
- D2: renamed from D7; value 150V 1A, Schottky bigger -> 150V 2A
- renumbered C17 to C5, C18 to C6, C20 to C7, C21 to C8, C22 to C9, L2 to L1, R22 to R10, R18 to R7, R19 to R8, R20 to R9, U4 to U6
Changed lines of the file:
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@@
 		(dnp no)
 		(fields_autoplaced yes)
-		(property "Reference" "#PWR029"
+		(property "Reference" "#PWR019"
 			(at 149.86 111.76 0)
 			(effects
@@
 			(project "PULSER-testboard-hv"
 				(path "/853931f0-9d2b-49ab-aae3-2a7153967e0f/bd7f0006-b363-44d9-a542-e4fe897a7941"
-					(reference "#PWR029")
+					(reference "#PWR019")
 					(unit 1)
 				)
@@
 		(on_board yes)
 		(dnp no)
-		(property "Reference" "C21"
+		(property "Reference" "C8"
 			(at 182.118 90.424 0)
 			(effects
@@
 			(project "PULSER-testboard-hv"
 				(path "/853931f0-9d2b-49ab-aae3-2a7153967e0f/bd7f0006-b363-44d9-a542-e4fe897a7941"
-					(reference "C21")
+					(reference "C8")
 					(unit 1)
 				)
@@
 		(dnp no)
 		(fields_autoplaced yes)
-		(property "Reference" "L2"
+		(property "Reference" "L1"
 			(at 147.32 53.34 90)
 			(effects
@@
 			(project "PULSER-testboard-hv"
 				(path "/853931f0-9d2b-49ab-aae3-2a7153967e0f/bd7f0006-b363-44d9-a542-e4fe897a7941"
-					(reference "L2")
+					(reference "L1")
 					(unit 1)
 				)
@@
 		(dnp no)
 		(fields_autoplaced yes)
-		(property "Reference" "C17"
+		(property "Reference" "C5"
 			(at 90.17 74.9299 0)
 			(effects
@@
 			(project "PULSER-testboard-hv"
 				(path "/853931f0-9d2b-49ab-aae3-2a7153967e0f/bd7f0006-b363-44d9-a542-e4fe897a7941"
-					(reference "C17")
+					(reference "C5")
 					(unit 1)
 				)
@@
 		(on_board yes)
 		(dnp no)
-		(property "Reference" "U4"
+		(property "Reference" "U6"
 			(at 149.098 92.964 0)
 			(effects
@@
 			(project "PULSER-testboard-hv"
 				(path "/853931f0-9d2b-49ab-aae3-2a7153967e0f/bd7f0006-b363-44d9-a542-e4fe897a7941"
-					(reference "U4")
+					(reference "U6")
 					(unit 1)
 				)
@@
 		(on_board yes)
 		(dnp no)
-		(property "Reference" "C20"
+		(property "Reference" "C7"
 			(at 104.648 86.36 0)
 			(effects
@@
 			(project "PULSER-testboard-hv"
 				(path "/853931f0-9d2b-49ab-aae3-2a7153967e0f/bd7f0006-b363-44d9-a542-e4fe897a7941"
-					(reference "C20")
+					(reference "C7")
 					(unit 1)
 				)
@@
 		(on_board yes)
 		(dnp no)
-		(property "Reference" "R19"
+		(property "Reference" "R8"
 			(at 118.618 86.614 0)
 			(effects
@@
 			(project "PULSER-testboard-hv"
 				(path "/853931f0-9d2b-49ab-aae3-2a7153967e0f/bd7f0006-b363-44d9-a542-e4fe897a7941"
-					(reference "R19")
+					(reference "R8")
 					(unit 1)
 				)
@@
 		(dnp no)
 		(fields_autoplaced yes)
-		(property "Reference" "C22"
+		(property "Reference" "C9"
 			(at 119.38 95.2499 0)
 			(effects
@@
 			(project "PULSER-testboard-hv"
 				(path "/853931f0-9d2b-49ab-aae3-2a7153967e0f/bd7f0006-b363-44d9-a542-e4fe897a7941"
-					(reference "C22")
+					(reference "C9")
 					(unit 1)
 				)
@@
 		(on_board yes)
 		(dnp no)
-		(property "Reference" "R22"
+		(property "Reference" "R10"
 			(at 173.228 92.202 0)
 			(effects
@@
 			(project "PULSER-testboard-hv"
 				(path "/853931f0-9d2b-49ab-aae3-2a7153967e0f/bd7f0006-b363-44d9-a542-e4fe897a7941"
-					(reference "R22")
+					(reference "R10")
 					(unit 1)
 				)
@@
 		(on_board yes)
 		(dnp no)
-		(property "Reference" "C18"
+		(property "Reference" "C6"
 			(at 219.202 75.438 0)
 			(effects
@@
 			(project "PULSER-testboard-hv"
 				(path "/853931f0-9d2b-49ab-aae3-2a7153967e0f/bd7f0006-b363-44d9-a542-e4fe897a7941"
-					(reference "C18")
+					(reference "C6")
 					(unit 1)
 				)
@@
 		(on_board yes)
 		(dnp no)
-		(property "Reference" "D7"
+		(property "Reference" "D2"
 			(at 192.0875 52.07 0)
 			(effects
@@
 			)
 		)
-		(property "Value" "150V 1A, Schottky bigger"
-			(at 197.1675 54.61 0)
+		(property "Value" "150V 2A"
+			(at 192.786 54.61 0)
 			(effects
 				(font
@@
 			(project "PULSER-testboard-hv"
 				(path "/853931f0-9d2b-49ab-aae3-2a7153967e0f/bd7f0006-b363-44d9-a542-e4fe897a7941"
-					(reference "D7")
+					(reference "D2")
 					(unit 1)
 				)
@@
 		(on_board yes)
 		(dnp no)
-		(property "Reference" "R20"
+		(property "Reference" "R9"
 			(at 202.184 87.63 0)
 			(effects
@@
 			(project "PULSER-testboard-hv"
 				(path "/853931f0-9d2b-49ab-aae3-2a7153967e0f/bd7f0006-b363-44d9-a542-e4fe897a7941"
-					(reference "R20")
+					(reference "R9")
 					(unit 1)
 				)
@@
 		(on_board yes)
 		(dnp no)
-		(property "Reference" "R18"
+		(property "Reference" "R7"
 			(at 198.882 72.644 0)
 			(effects
@@
 			(project "PULSER-testboard-hv"
 				(path "/853931f0-9d2b-49ab-aae3-2a7153967e0f/bd7f0006-b363-44d9-a542-e4fe897a7941"
-					(reference "R18")
+					(reference "R7")
 					(unit 1)
 				)

Commit message: HV lcsc & footprint assigned
Parts:
- C10: renamed from C6; footprint Capacitor_SMD:C_0805_2012Metric -> Capacitor_SMD:C_1206_3216Metric; LCSC C342865 -> C113894
- C11: renamed from C7; value 1uF -> 1u
- C12: renamed from C8; value 0.22uF -> 0.22u
- C13: renamed from C9; value 1nF -> 1n
- D2: footprint Diode_SMD:D_PowerDI-123 -> Diode_SMD:D_SMC; LCSC C156325 -> C241922
- R16: renamed from R7; footprint Resistor_SMD:R_0805_2012Metric -> Resistor_SMD:R_1206_3216Metric; LCSC C17709 -> C17997
- renumbered C5 to C9, R8 to R17, R9 to R18, R10 to R19
Changed lines of the file:
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@@
 		(dnp no)
 		(fields_autoplaced yes)
-		(property "Reference" "#PWR019"
+		(property "Reference" "#PWR029"
 			(at 149.86 111.76 0)
 			(effects
@@
 			(project "PULSER-testboard-hv"
 				(path "/853931f0-9d2b-49ab-aae3-2a7153967e0f/bd7f0006-b363-44d9-a542-e4fe897a7941"
-					(reference "#PWR019")
+					(reference "#PWR029")
 					(unit 1)
 				)
@@
 		(on_board yes)
 		(dnp no)
-		(property "Reference" "C8"
+		(property "Reference" "C12"
 			(at 182.118 90.424 0)
 			(effects
@@
 			)
 		)
-		(property "Value" "0.22uF"
+		(property "Value" "0.22u"
 			(at 181.61 95.25 0)
 			(effects
@@
 			(project "PULSER-testboard-hv"
 				(path "/853931f0-9d2b-49ab-aae3-2a7153967e0f/bd7f0006-b363-44d9-a542-e4fe897a7941"
-					(reference "C8")
+					(reference "C12")
 					(unit 1)
 				)
@@
 		(dnp no)
 		(fields_autoplaced yes)
-		(property "Reference" "C5"
+		(property "Reference" "C9"
 			(at 90.17 74.9299 0)
 			(effects
@@
 			(project "PULSER-testboard-hv"
 				(path "/853931f0-9d2b-49ab-aae3-2a7153967e0f/bd7f0006-b363-44d9-a542-e4fe897a7941"
-					(reference "C5")
+					(reference "C9")
 					(unit 1)
 				)
@@
 		(on_board yes)
 		(dnp no)
-		(property "Reference" "C7"
+		(property "Reference" "C11"
 			(at 104.648 86.36 0)
 			(effects
@@
 			)
 		)
-		(property "Value" "1uF"
+		(property "Value" "1u"
 			(at 104.648 88.392 0)
 			(effects
@@
 			(project "PULSER-testboard-hv"
 				(path "/853931f0-9d2b-49ab-aae3-2a7153967e0f/bd7f0006-b363-44d9-a542-e4fe897a7941"
-					(reference "C7")
+					(reference "C11")
 					(unit 1)
 				)
@@
 		(on_board yes)
 		(dnp no)
-		(property "Reference" "R8"
+		(property "Reference" "R17"
 			(at 118.618 86.614 0)
 			(effects
@@
 			(project "PULSER-testboard-hv"
 				(path "/853931f0-9d2b-49ab-aae3-2a7153967e0f/bd7f0006-b363-44d9-a542-e4fe897a7941"
-					(reference "R8")
+					(reference "R17")
 					(unit 1)
 				)
@@
 		(dnp no)
 		(fields_autoplaced yes)
-		(property "Reference" "C9"
+		(property "Reference" "C13"
 			(at 119.38 95.2499 0)
 			(effects
@@
 			)
 		)
-		(property "Value" "1nF"
+		(property "Value" "1n"
 			(at 119.38 97.7899 0)
 			(effects
@@
 			(project "PULSER-testboard-hv"
 				(path "/853931f0-9d2b-49ab-aae3-2a7153967e0f/bd7f0006-b363-44d9-a542-e4fe897a7941"
-					(reference "C9")
+					(reference "C13")
 					(unit 1)
 				)
@@
 		(on_board yes)
 		(dnp no)
-		(property "Reference" "R10"
+		(property "Reference" "R19"
 			(at 173.228 92.202 0)
 			(effects
@@
 			(project "PULSER-testboard-hv"
 				(path "/853931f0-9d2b-49ab-aae3-2a7153967e0f/bd7f0006-b363-44d9-a542-e4fe897a7941"
-					(reference "R10")
+					(reference "R19")
 					(unit 1)
 				)
@@
 		(on_board yes)
 		(dnp no)
-		(property "Reference" "C6"
+		(property "Reference" "C10"
 			(at 219.202 75.438 0)
 			(effects
@@
 			)
 		)
-		(property "Footprint" "Capacitor_SMD:C_0805_2012Metric"
+		(property "Footprint" "Capacitor_SMD:C_1206_3216Metric"
 			(at 219.4052 81.28 0)
 			(effects
@@
 			)
 		)
-		(property "LCSC" "C342865"
+		(property "LCSC" "C113894"
 			(at 218.44 77.47 0)
 			(effects
@@
 			(project "PULSER-testboard-hv"
 				(path "/853931f0-9d2b-49ab-aae3-2a7153967e0f/bd7f0006-b363-44d9-a542-e4fe897a7941"
-					(reference "C6")
+					(reference "C10")
 					(unit 1)
 				)
@@
 			)
 		)
-		(property "Footprint" "Diode_SMD:D_PowerDI-123"
+		(property "Footprint" "Diode_SMD:D_SMC"
 			(at 191.77 58.42 0)
 			(effects
@@
 			)
 		)
-		(property "LCSC" "C156325"
+		(property "LCSC" "C241922"
 			(at 191.77 58.42 0)
 			(effects
@@
 		(on_board yes)
 		(dnp no)
-		(property "Reference" "R9"
+		(property "Reference" "R18"
 			(at 202.184 87.63 0)
 			(effects
@@
 			(project "PULSER-testboard-hv"
 				(path "/853931f0-9d2b-49ab-aae3-2a7153967e0f/bd7f0006-b363-44d9-a542-e4fe897a7941"
-					(reference "R9")
+					(reference "R18")
 					(unit 1)
 				)
@@
 		(on_board yes)
 		(dnp no)
-		(property "Reference" "R7"
+		(property "Reference" "R16"
 			(at 198.882 72.644 0)
 			(effects
@@
 			)
 		)
-		(property "Footprint" "Resistor_SMD:R_0805_2012Metric"
+		(property "Footprint" "Resistor_SMD:R_1206_3216Metric"
 			(at 207.518 73.66 90)
 			(effects
@@
 			)
 		)
-		(property "LCSC" "C17709"
+		(property "LCSC" "C17997"
 			(at 205.74 73.66 0)
 			(effects
@@
 			(project "PULSER-testboard-hv"
 				(path "/853931f0-9d2b-49ab-aae3-2a7153967e0f/bd7f0006-b363-44d9-a542-e4fe897a7941"
-					(reference "R7")
+					(reference "R16")
 					(unit 1)
 				)
