File: pcb/PULSER-testboard-hv/boost.kicad_sch (KiCad schematic)
At the start: 12 parts, among them U6 LT8365

Commit message: pulser v2 HV r4 pcb draft ok
Parts:
- L1: value 100uH, Isat=2.7A -> 150uH; LCSC C2453104 -> C338769; Rating (none) -> Isat=1.8A
- R16: value 470k 150V -> 430k; LCSC C17997 -> (none); Rating (none) -> 1% 150V
- R18: Rating (none) -> 1%
Other:
- note added: "95V"
- note added: "FBX=1.6V results in 93V"
- note added: "spec: Vo=95V, Iomax=0.4A DMAX=62% eta=90% ILMAX=1.2A ΔISW = 0.6A L = 150uH"
- note removed: "100V"
- note removed: "DMAX=64% eta=50% ILMAX=550mA ΔISW = 0.6A (< 1.9A) L = 96uH"
- note removed: "FBX=1.6V results in 102V"
Changed lines of the file:
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@@
 	(title_block
 		(title "Pulser V2 HV Test Board")
-		(date "2026-04-15")
-		(rev "3")
+		(date "2026-07-01")
+		(rev "4")
 		(company "Spark Project")
 		(comment 1 "夕月霞")
@@
 		)
 	)
-	(text "DMAX=64%\neta=50%\nILMAX=550mA\nΔISW = 0.6A (< 1.9A)\nL = 96uH"
+	(text "spec: Vo=95V, Iomax=0.4A\nDMAX=62%\neta=90%\nILMAX=1.2A\nΔISW = 0.6A\nL = 150uH"
 		(exclude_from_sim no)
-		(at 145.542 61.976 0)
+		(at 144.78 62.23 0)
 		(effects
 			(font
@@
 		)
 	)
-	(text "FBX=1.6V\nresults in 102V"
+	(text "FBX=1.6V\nresults in 93V"
 		(exclude_from_sim no)
 		(at 205.74 104.394 0)
@@
 		)
 	)
-	(text "100V"
+	(text "95V"
 		(exclude_from_sim no)
-		(at 228.854 56.134 0)
+		(at 229.616 56.134 0)
 		(effects
 			(font
@@
 			)
 		)
+		(property "Sim.Params" ""
+			(at 181.61 92.71 0)
+			(effects
+				(font
+					(size 1.27 1.27)
+				)
+				(hide yes)
+			)
+		)
 		(pin "1"
 		)
@@
 		(on_board yes)
 		(dnp no)
-		(fields_autoplaced yes)
 		(property "Reference" "L1"
-			(at 147.32 53.34 90)
-			(effects
-				(font
-					(size 1.27 1.27)
-				)
-			)
-		)
-		(property "Value" "100uH, Isat=2.7A"
-			(at 147.32 55.88 90)
+			(at 144.78 51.562 90)
+			(effects
+				(font
+					(size 1.27 1.27)
+				)
+			)
+		)
+		(property "Value" "150uH"
+			(at 146.558 53.848 90)
 			(effects
 				(font
@@
 			)
 		)
-		(property "LCSC" "C2453104"
+		(property "LCSC" "C338769"
 			(at 147.32 58.42 90)
 			(effects
@@
 					(size 1.27 1.27)
 				)
+			)
+		)
+		(property "Rating" "Isat=1.8A"
+			(at 148.082 56.134 90)
+			(effects
+				(font
+					(size 1.27 1.27)
+				)
+			)
+		)
+		(property "Sim.Params" ""
+			(at 147.32 58.42 90)
+			(effects
+				(font
+					(size 1.27 1.27)
+				)
+				(hide yes)
 			)
 		)
@@
 			)
 		)
+		(property "Sim.Params" ""
+			(at 86.36 76.2 0)
+			(effects
+				(font
+					(size 1.27 1.27)
+				)
+				(hide yes)
+			)
+		)
 		(pin "1"
 		)
@@
 			)
 		)
+		(property "Sim.Params" ""
+			(at 119.38 71.12 0)
+			(effects
+				(font
+					(size 1.27 1.27)
+				)
+				(hide yes)
+			)
+		)
 		(pin "12"
 		)
@@
 			)
 		)
+		(property "Sim.Params" ""
+			(at 101.6 87.63 0)
+			(effects
+				(font
+					(size 1.27 1.27)
+				)
+				(hide yes)
+			)
+		)
 		(pin "1"
 		)
@@
 					(size 1.27 1.27)
 				)
+			)
+		)
+		(property "Sim.Params" ""
+			(at 115.57 87.63 0)
+			(effects
+				(font
+					(size 1.27 1.27)
+				)
+				(hide yes)
 			)
 		)
@@
 			)
 		)
+		(property "Sim.Params" ""
+			(at 115.57 96.52 0)
+			(effects
+				(font
+					(size 1.27 1.27)
+				)
+				(hide yes)
+			)
+		)
 		(pin "1"
 		)
@@
 			)
 		)
+		(property "Sim.Params" ""
+			(at 176.53 92.71 0)
+			(effects
+				(font
+					(size 1.27 1.27)
+				)
+				(hide yes)
+			)
+		)
 		(pin "1"
 		)
@@
 			)
 		)
+		(property "Sim.Params" ""
+			(at 218.44 77.47 0)
+			(effects
+				(font
+					(size 1.27 1.27)
+				)
+				(hide yes)
+			)
+		)
 		(pin "1"
 		)
@@
 			)
 		)
+		(property "Sim.Params" ""
+			(at 191.77 58.42 0)
+			(effects
+				(font
+					(size 1.27 1.27)
+				)
+				(hide yes)
+			)
+		)
 		(pin "2"
 		)
@@
 			)
 		)
+		(property "Rating" "1%"
+			(at 202.946 91.948 0)
+			(effects
+				(font
+					(size 1.27 1.27)
+				)
+			)
+		)
+		(property "Sim.Params" ""
+			(at 205.74 88.9 0)
+			(effects
+				(font
+					(size 1.27 1.27)
+				)
+				(hide yes)
+			)
+		)
 		(pin "1"
 		)
@@
 		(dnp no)
 		(property "Reference" "R16"
-			(at 198.882 72.644 0)
-			(effects
-				(font
-					(size 1.27 1.27)
-				)
-			)
-		)
-		(property "Value" "470k 150V"
-			(at 198.882 74.676 0)
+			(at 201.93 72.644 0)
+			(effects
+				(font
+					(size 1.27 1.27)
+				)
+			)
+		)
+		(property "Value" "430k"
+			(at 201.93 74.676 0)
 			(effects
 				(font
@@
 			)
 		)
-		(property "LCSC" "C17997"
+		(property "LCSC" ""
 			(at 205.74 73.66 0)
 			(effects
@@
 			)
 		)
+		(property "Rating" "1% 150V"
+			(at 200.152 76.708 0)
+			(effects
+				(font
+					(size 1.27 1.27)
+				)
+			)
+		)
+		(property "Sim.Params" ""
+			(at 205.74 73.66 0)
+			(effects
+				(font
+					(size 1.27 1.27)
+				)
+				(hide yes)
+			)
+		)
