File: pcb/PULSER-testboard-hv/PULSER-testboard-hv.kicad_sch (KiCad schematic)
At the start: 48 parts, among them J1 Screw_Terminal 2pin, J2 Screw_Terminal 2pin, J3 Conn_01x02_Pin, J4 Conn_01x02_Pin, Q1 Q_NMOS_GDS, U2 INA281A2, U3 LTC7001, U4 TLV3201, U5 LM317_DPAK

Commit message: P2HV r3 PCB
Parts:
- D6: footprint (none) -> Diode_SMD:D_TUMD2; LCSC (none) -> C509964
- JP6: footprint (none) -> Jumper:SolderJumper-2_P1.3mm_Open_RoundedPad1.0x1.5mm; now left out of the parts list
- R2: footprint (none) -> Resistor_SMD:R_2512_6332Metric; LCSC (none) -> C47019
- R3: footprint (none) -> Resistor_SMD:R_1206_3216Metric; LCSC (none) -> C17900
- R6: LCSC (none) -> C21190
Changed lines of the file:
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@@
 			)
 		)
-		(property "Footprint" ""
+		(property "Footprint" "Resistor_SMD:R_1206_3216Metric"
 			(at 252.222 50.8 90)
 			(effects
@@
 		)
 		(property "Description" "Resistor"
+			(at 254 50.8 0)
+			(effects
+				(font
+					(size 1.27 1.27)
+				)
+				(hide yes)
+			)
+		)
+		(property "LCSC" "C17900"
 			(at 254 50.8 0)
 			(effects
@@
 			)
 		)
-		(property "LCSC" ""
+		(property "LCSC" "C21190"
 			(at 196.85 115.57 0)
 			(effects
@@
 			)
 		)
-		(property "Footprint" ""
+		(property "Footprint" "Resistor_SMD:R_2512_6332Metric"
 			(at 143.002 55.88 90)
 			(effects
@@
 		)
 		(property "Description" "Resistor"
+			(at 144.78 55.88 0)
+			(effects
+				(font
+					(size 1.27 1.27)
+				)
+				(hide yes)
+			)
+		)
+		(property "LCSC" "C47019"
 			(at 144.78 55.88 0)
 			(effects
@@
 			)
 		)
-		(property "Footprint" ""
+		(property "Footprint" "Diode_SMD:D_TUMD2"
 			(at 125.73 67.31 0)
 			(effects
@@
 		(property "Sim.Pins" "1=K 2=A"
 			(at 125.73 67.31 0)
+			(effects
+				(font
+					(size 1.27 1.27)
+				)
+				(hide yes)
+			)
+		)
+		(property "LCSC" "C509964"
+			(at 125.73 67.31 90)
 			(effects
 				(font
@@
 		(unit 1)
 		(exclude_from_sim no)
-		(in_bom yes)
+		(in_bom no)
 		(on_board yes)
 		(dnp no)
@@
 			)
 		)
-		(property "Footprint" ""
+		(property "Footprint" "Jumper:SolderJumper-2_P1.3mm_Open_RoundedPad1.0x1.5mm"
 			(at 151.13 55.88 0)
 			(effects
