File: pcb/PULSER-testboard-hv/PULSER-testboard-hv.kicad_sch (KiCad schematic)
At the start: 48 parts, among them J1 Screw_Terminal 2pin, J2 Screw_Terminal 2pin, J3 Conn_01x02_Pin, J4 Conn_01x02_Pin, Q1 Q_NMOS_GDS, U2 INA281A2, U3 LTC7001, U4 TLV3201, U5 LM317_DPAK

Commit message: Record current testboard modifications as schematics
Parts:
- added E1: 12VDC, symbol Simulation_SPICE:ESOURCE
- added HS1: 20x15x5mm, symbol Mechanical:Heatsink
- added R4: 100Ω 5W, symbol Device:R
- L2, L3, L4, L5: now not fitted
Connections:
- net +36V: now also E1.3 (C+)
- net +5V: no longer D6.2 (A), U3.1 (VCC)
- net GND: now also E1.2 (N-), E1.4 (C-)
- net at D1.2 (A), JP1.2 (B), JP2.2 (B)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: now also R4.1
- net at L2.1, R1.2, TP3.1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: now also R4.2
- new net +12V: D6.2 (A), E1.1 (N+), U3.1 (VCC)
Other:
- note added: "short"
