File: pcb/PULSER-testboard-hv/PULSER-testboard-hv.kicad_sch (KiCad schematic)
At the start: 51 parts, among them J1 Screw_Terminal 2pin, J2 Screw_Terminal 2pin, J3 Conn_01x02_Pin, J4 Conn_01x02_Pin, Q1 Q_NMOS_GDS, U2 INA281A2, U3 LTC7001, U4 TLV3201, U5 LM317_DPAK

Commit message: pulser v2 HV r4 pcb draft ok
Parts:
- removed E1: 12VDC, symbol Simulation_SPICE:ESOURCE
- removed HS1: 20x15x5mm, symbol Mechanical:Heatsink
- removed J3, J4: Conn_01x02_Pin, Connector_PinHeader_2.54mm:PinHeader_1x02_P2.54mm_Vertical, symbol Connector:Conn_01x02_Pin
- removed JP1, JP2, JP4: Jumper_2_Small_Open, Connector_PinHeader_2.54mm:PinHeader_1x02_P2.54mm_Vertical, symbol Jumper:Jumper_2_Small_Open
- removed JP3, JP5: Jumper_2_Small_Bridged, Jumper:SolderJumper-2_P1.3mm_Bridged_RoundedPad1.0x1.5mm, symbol Jumper:Jumper_2_Small_Bridged
- removed JP6: Jumper_2_Small_Open, Jumper:SolderJumper-2_P1.3mm_Open_RoundedPad1.0x1.5mm, symbol Jumper:Jumper_2_Small_Open
- removed L2, L3, L4, L5: 220u, Inductor_THT:L_Toroid_Vertical_L16.0mm_W8.0mm_P7.62mm, symbol Device:L
- removed R2: 10, Resistor_SMD:R_2512_6332Metric, symbol Device:R
- added C14, C15, C16, C17: 0.1u, Capacitor_SMD:C_0603_1608Metric, symbol Device:C
- added C18: 0.1u, Capacitor_SMD:C_0603_1608Metric, symbol Device:C_Small
- added C19: 1u, Capacitor_SMD:C_0603_1608Metric, symbol Device:C_Small
- added J6: Conn_01x08_Pin, Connector_FFC-FPC:Molex_200528-0080_1x08-1MP_P1.00mm_Horizontal, symbol Connector:Conn_01x08_Pin
- added R5: 560, Resistor_SMD:R_0603_1608Metric, symbol Device:R
- added R8: 4.7k, Resistor_SMD:R_0603_1608Metric, symbol Device:R
- added U1, U7: ADuM1200AR, Package_SO:SOIC-8_3.9x4.9mm_P1.27mm, symbol Isolator:ADuM1200AR
- added U8: LM317_DPAK, Package_TO_SOT_SMD:TO-252-2, symbol Regulator_Linear:LM317_TO-252
- D3: LCSC C2286 -> (none); Rating (none) -> Amber
- R4: value 100Ω 5W -> 100; footprint (none) -> SparkAll:Bourns-TO508P1229X317-3N; LCSC (none) -> C37794578
Connections:
- net +12V: now also C4.1, C7.2, U5.3 (VI), C19.2, R5.1, U8.2 (VO)
- net +36V: now also C18.2, U8.3 (VI); no longer C7.2, U5.3 (VI)
- net +5V: now also C16.1, C17.1, U1.8 (VDD2), U7.1 (VDD1); no longer C4.1
- net CURR: now also U7.2 (VIA)
- net EN: now also U1.7 (VOA)
- net GND: now also D5.2 (A), U3.2 (VCCUV), U3.5 (OVLO), C16.2, C17.2, C18.1, C19.1, R8.2, U1.5 (GND2), U7.4 (GND1)
- new net: R5.2, R8.1, U8.1 (ADJ)
- new net CURR_S: J6.4 (Pin_4), U7.7 (VOA)
- new net EN_S: J6.3 (Pin_3), U1.2 (VIA)
- new net GNDS: C14.2, C15.2, J6.2 (Pin_2), J6.5 (Pin_5), U1.3 (VIB), U1.4 (GND1), U7.5 (GND2)
- new net VCCS: C14.1, C15.1, J6.1 (Pin_1), U1.1 (VDD1), U7.8 (VDD2)
- new net ~{FAULT}: U7.3 (VIB)
- new net ~{FAULT}_S: J6.6 (Pin_6), U7.6 (VOB)
Other:
- sheet Pulse Controller ports: added ~{FAULT}; removed none
- note added: "400mA max cont->1A pulse 1 pulse:10uC / 1uF: 95uC max duty: 40% (0.4A avg)"
- note added: "94Ω -> 1A"
- note added: "95V"
- note added: "CURR"
- note added: "bypass U2, U4"
- note added: "bypass U3"
- note added: "operation limiting factor: * avg output current * avg. boost current: 400mW * heat dissipation of limit resistor: 10W (->100mA) * boost conv output cap: duration of single pulse * 1uF (->approx 10us)"
- note added: "peak: 100W avg: 10W Rc-back: <2K/W (150+ vias)"
- note added: "peak: 600mW avg: 60mW"
- note removed: "100V"
- note removed: "5V"
- note removed: "5V digital output"
- note removed: "CURR (RED)"
- note removed: "bypass caps"
- note removed: "digital input (thresh=2V) abs max 5.3V"
- note removed: "flywheel damping"
- note removed: "peak: 400mW avg: 20mW"
- note removed: "short"
- moved on the sheet: C1, C2, C3, C4, C5, C6, C7, C8, D1, D3, D5, D6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

Commit message: Add 12V fan connector & sw 12V converter to HV
Parts:
- removed C18, C7: 0.1u, Capacitor_SMD:C_0603_1608Metric, symbol Device:C_Small
- removed C19, C8: 1u, Capacitor_SMD:C_0603_1608Metric, symbol Device:C_Small
- removed R14: 270, Resistor_SMD:R_0603_1608Metric, symbol Device:R
- removed R15: 820, Resistor_SMD:R_0603_1608Metric, symbol Device:R
- removed R5: 560, Resistor_SMD:R_0603_1608Metric, symbol Device:R
- removed R8: 4.7k, Resistor_SMD:R_0603_1608Metric, symbol Device:R
- removed U5, U8: LM317_DPAK, Package_TO_SOT_SMD:TO-252-2, symbol Regulator_Linear:LM317_TO-252
- added J3: Conn_01x02_Pin, Connector_JST:JST_XH_B2B-XH-A_1x02_P2.50mm_Vertical, symbol Connector:Conn_01x02_Pin
Connections:
- net +12V: now also J3.1 (Pin_1)
- net GND: now also J3.2 (Pin_2)
Other:
- added sheet powersupply (powersupply.kicad_sch)
- note added: "12V fan (500mA max)"
- moved on the sheet: C14, C15, C16, C17, J6, U1, U7
