File: pcb/PULSER-testboard-hv/pulse.kicad_sch (KiCad schematic)
At the start: 31 parts, among them SW2 SW_DIP_x04, SW3 SW_DIP_x02, U10 LMC555xMM, U7 74HC00, U8 74HC00, U9 LMC555xMM

Commit message: HV TestBoard r2 schem draft ok. mock firmware build env.
Parts:
- removed C14, C15, C20: 0.1u, Capacitor_SMD:C_0603_1608Metric, symbol Device:C
- removed C16, C17: 330p, Capacitor_SMD:C_0603_1608Metric, symbol Device:C_Small
- removed C18, C19: 470p, Capacitor_SMD:C_0603_1608Metric, symbol Device:C_Small
- removed C22, C23: 0.1u, Capacitor_SMD:C_0603_1608Metric, symbol Device:C_Small
- removed R22: 10k, Resistor_SMD:R_0603_1608Metric, symbol Device:R
- removed R23: 20k, Resistor_SMD:R_0603_1608Metric, symbol Device:R
- removed R24: 910, Resistor_SMD:R_0603_1608Metric, symbol Device:R
- removed R25: 9.1k, Resistor_SMD:R_0603_1608Metric, symbol Device:R
- removed R26, R27: 10M, Resistor_SMD:R_0603_1608Metric, symbol Device:R
- removed SW2: SW_DIP_x04, Button_Switch_SMD:SW_DIP_SPSTx04_Slide_9.78x12.34mm_W8.61mm_P2.54mm, symbol Switch:SW_DIP_x04
- removed TP10, TP7, TP8, TP9: TestPoint_Small, TestPoint:TestPoint_Pad_D1.5mm, symbol Connector:TestPoint_Small
- removed U10, U9: LMC555xMM, Package_SO:SOIC-8_3.9x4.9mm_P1.27mm, symbol Timer:LMC555xMM
- removed U7, U8: 74HC00, Package_SO:TSSOP-14_4.4x5mm_P0.65mm, symbol 74xx:74HC00
- added D4: LED, LED_SMD:LED_0603_1608Metric, symbol Device:LED
- added J5: Conn_01x02_Socket, Connector_PinSocket_2.54mm:PinSocket_1x02_P2.54mm_Vertical, symbol Connector:Conn_01x02_Socket
- added R7: 10k, Resistor_SMD:R_0603_1608Metric, symbol Device:R
- added SW1, SW2: SW_DIP_x02, Button_Switch_SMD:SW_DIP_SPSTx02_Slide_9.78x7.26mm_W8.61mm_P2.54mm, symbol Switch:SW_DIP_x02
- added TP11: TestPoint_Small, TestPoint:TestPoint_Pad_D1.5mm, symbol Connector:TestPoint_Small
- added U11: ATtiny1616-M, Package_DFN_QFN:VQFN-20-1EP_3x3mm_P0.4mm_EP1.7x1.7mm, symbol MCU_Microchip_ATtiny:ATtiny1616-M
- R20: value 2.7k -> 100k; LCSC C13167 -> C25803
- R21: value 5.6k -> 100k; LCSC C23189 -> C25803
Connections:
- net TH_CL is gone; now on net GND: SW3.3, SW3.4
- net TH_P_1 is gone; now on net GATE: R20.1
- net TH_P_2 is gone; now on net +5V: R21.1
- net +5V: now also U11.4 (VCC); no longer R20.2, R21.2
- net CURR: now also U11.16 (PC1)
- net EN: now also U11.15 (PC0)
- net GATE: now also U11.5 (PA4); no longer TP13.1
- net GND: now also R20.2, J5.2 (Pin_2), R7.2, SW1.3, SW1.4, SW2.3, SW2.4, U11.21 (GND), U11.3 (GND)
- net GATE_OK: no longer names the net of TP12.1
- net GATE_OK: now also U11.1 (PA2)
- net TH_CL_0.1m: no longer names the net of SW3.1
- net TH_CL_0.1m: now also U11.14 (PB0)
- net TH_CL_1m: no longer names the net of SW3.2
- net TH_CL_1m: now also U11.13 (PB1)
- net ~{CURR} renamed UPDI
- net UPDI: now also R21.2, J5.1 (Pin_1), U11.19 (~{RESET}/PA0)
- new net: D4.1 (K), R7.1
- new net: D4.2 (A), U11.18 (PC3)
- new net: TP11.1, U11.20 (PA1)
- new net: SW2.1, U11.10 (PB4)
- new net: SW2.2, U11.9 (PB5)
- new net: TP13.1, U11.2 (PA3)
- new net: SW1.2, U11.11 (PB3)
- new net: SW1.1, U11.12 (PB2)
- new net VTH: U11.7 (PA6)
Other:
- note added: "COOLDOWN 00: 100us (default) 01: 1ms 1x: unused"
- note added: "PULSE 00: 1us 01: 2us 10: 5us (default) 11: 10us"
- note added: "THRESH 00: 50mA 01: 100mA (default) 10: 200mA 11: 500mA"
- note added: "Vth = Ith * Rsense (100m) * gain (50)"
- note removed: "100us (default) 1ms (t=1.1 RC)"
- note removed: "1us 2us 5us (default) 10us (t=1.1 RC)"
- note removed: "GATE = EN & GATE_OK GATE_OK = PULSE | ~COOLDOWN = ~ (!PULSE & COOLDOWN)"
- note removed: "SW open (always cooldown)"
- note removed: "SW open (no pulse)"
- note removed: "unused"
- moved on the sheet: C21, SW3

Commit message: HV TestBoard r2 pcb ok
Other:
- note added: "STAT (GREEN)"
Changed lines of the file:
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@@
+		)
+	)
+	(text "STAT (GREEN)"
+		(exclude_from_sim no)
+		(at 74.93 86.36 0)
+		(effects
+			(font
+				(size 1 1)
+			)
+			(justify left)
 		)
 	)

Commit message: P2HV r3 schem
Parts:
- D4: LCSC C2297 -> C126319
- R7: value 10k -> 4.7k; LCSC C25804 -> (none)
Changed lines of the file:
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@@
 	(title_block
 		(title "Pulser V2 HV Test Board")
-		(date "2026-02-06")
-		(rev "2")
+		(date "2026-04-15")
+		(rev "3")
 		(company "Spark Project")
 		(comment 1 "夕月霞")
@@
 			)
 		)
-		(property "LCSC" "C2297"
+		(property "LCSC" "C126319"
 			(at 71.12 81.28 90)
 			(effects
@@
 			)
 		)
-		(property "Value" "10k"
+		(property "Value" "4.7k"
 			(at 73.66 92.7099 0)
 			(effects
@@
 			)
 		)
-		(property "LCSC" "C25804"
+		(property "LCSC" ""
 			(at 71.12 91.44 0)
 			(effects

Commit message: P2HV r3 PCB
Parts:
- R7: LCSC (none) -> C23162
Changed lines of the file:
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@@
 			)
 		)
-		(property "LCSC" ""
+		(property "LCSC" "C23162"
 			(at 71.12 91.44 0)
 			(effects
