File: pcb/PULSER-testboard-hv/pulse.kicad_sch (KiCad schematic)
At the start: 14 parts, among them J5 Conn_01x02_Socket, SW1 SW_DIP_x02, SW2 SW_DIP_x02, SW3 SW_DIP_x02, U11 ATtiny1616-M

Commit message: pulser v2 HV r4 pcb draft ok
Parts:
- removed SW1, SW2, SW3: SW_DIP_x02, Button_Switch_SMD:SW_DIP_SPSTx02_Slide_9.78x7.26mm_W8.61mm_P2.54mm, symbol Switch:SW_DIP_x02
- removed TP12, TP13, TP14: TestPoint_Small, TestPoint:TestPoint_Pad_D1.5mm, symbol Connector:TestPoint_Small
- added D7: LED, LED_SMD:LED_0603_1608Metric, symbol Device:LED
- added R2: 4.7k, Resistor_SMD:R_0603_1608Metric, symbol Device:R
- D4: Rating (none) -> Green
Connections:
- net GND: now also R2.2
- net ~{FAULT}: now reaches U11.14 (PB0)
- net at U11.17 (PC2): now also D7.2 (A)
- new net: D7.1 (K), R2.1
Other:
- note added: "FLT"
- note added: "STAT"
- note removed: "COOLDOWN 00: 100us (default) 01: 1ms 1x: unused"
- note removed: "PULSE 00: 1us 01: 2us 10: 5us (default) 11: 10us"
- note removed: "STAT (GREEN)"
- note removed: "THRESH 00: 50mA 01: 100mA (default) 10: 200mA 11: 500mA"
- note removed: "Vth = Ith * Rsense (100m) * gain (50)"
