File: pcb/PULSER-testboard-ctrl/PULSER-testboard-ctrl.kicad_sch (KiCad schematic)
At the start: 11 parts, among them J1 I2C/XH, J2 36V IN, J3 HV EN, J4 HV CURR, J5 HC EN

Commit message: Draft ctrl r2 schem
Parts:
- removed E1: 5V DCDC, symbol Simulation_SPICE:ESOURCE
- added C1: 2.2u, symbol Device:C_Small
- added C2, C6: 1u, symbol Device:C_Small
- added C3, C4, C5: 22u, symbol Device:C_Small
- added J6, J7: Conn_01x08_Pin, symbol Connector:Conn_01x08_Pin
- added J8: Conn_01x02_Pin, symbol Connector:Conn_01x02_Pin
- added PS1: MEE1S0505SC, Converter_DCDC:Converter_DCDC_Murata_MEE1SxxxxSC_THT, symbol Converter_DCDC:MEE1S0505SC
- added R5: 10k, symbol Device:R
- added R6: 40.2k, symbol Device:R
- added R7: 15.8k, symbol Device:R
- added U1: ATtiny1616-M, Package_DFN_QFN:VQFN-20-1EP_3x3mm_P0.4mm_EP1.7x1.7mm, symbol MCU_Microchip_ATtiny:ATtiny1616-M
- added U2: TPSM365R6, SparkAll:TI-RDN0011A-MFG, symbol SparkAll:TPSM365R6FRDNR
Connections:
- net GND: now also C1.2, C2.2, C3.2, C5.2, PS1.1 (-Vin), R5.2, R7.2, U2.10 (GND)
- net HC_EN: now also J7.3 (Pin_3)
- net HV_CURR: now also J6.4 (Pin_4)
- net HV_EN: now also J6.3 (Pin_3)
- net I2C_SCL: now also U1.14 (PB0)
- net I2C_SDA: now also U1.13 (PB1)
- net +36V: now reaches J2.1 (Pin_1)
- net +36V: now also C1.1, U2.2 (EN), U2.3 (VIN)
- new net: C3.1, C5.1, PS1.2 (+Vin), R6.1, U2.4 (VOUT)
- new net: R5.1, R6.2, U2.9 (BIAS)
- new net: R7.1, U2.11 (MODE_SYNC)
- new net: C2.1, U2.8 (VCC)
- new net +5VS: C4.1, C6.1, J6.1 (Pin_1), J7.1 (Pin_1), PS1.4 (+Vout), U1.4 (VCC)
- new net GNDS: C4.2, C6.2, J6.2 (Pin_2), J6.5 (Pin_5), J7.2 (Pin_2), J7.5 (Pin_5), J8.2 (Pin_2), PS1.3 (-Vout), U1.21 (GND), U1.3 (GND)
- new net HC_CURR: J7.4 (Pin_4)
- new net HV_~{FAULT}: J6.6 (Pin_6)
- new net UPDI: J8.1 (Pin_1), U1.19 (~{RESET}/PA0)
- no-connect marks 0 -> 5
Other:
- note added: "RT Fsw=1MHz"
- note added: "UPDI writer (5V)"
- note added: "non-isolated 5V"
- moved on the sheet: A1, J1, J2, J3, J4, J5, R1, R2, R3, R4
