File: pcb/PULSER-testboard-ctrl/PULSER-testboard-ctrl.kicad_sch (KiCad schematic)
At the start: 25 parts, among them J1 I2C/XH, J2 36V IN, J3 HV EN, J4 HV CURR, J5 HC EN, J6 Conn_01x08_Pin, J7 Conn_01x08_Pin, J8 Conn_01x02_Pin, U1 ATtiny1616-M, U2 TPSM365R6

Commit message: pulser-v2 / ctrl-r2 PCB draft ok
Parts:
- removed A1: RaspberryPi_Pico2, Module:RaspberryPi_Pico_Common_Unspecified, symbol MCU_Module:RaspberryPi_Pico
- removed J3: HV EN, symbol Connector:Conn_01x02_Socket
- removed J4: HV CURR, symbol Connector:Conn_01x02_Socket
- removed J5: HC EN, symbol Connector:Conn_01x02_Socket
- added C6: 1u, Capacitor_SMD:C_0603_1608Metric, symbol Device:C_Small
- added D1, D2, D3: LED, LED_SMD:LED_0603_1608Metric, symbol Device:LED
- added TP1, TP2, TP3, TP5, TP6, TP7: TestPoint, TestPoint:TestPoint_Pad_D1.5mm, symbol Connector:TestPoint_Small
- C1: renamed from C6; footprint (none) -> Capacitor_SMD:C_0402_1005Metric; LCSC (none) -> C52923
- C2: footprint (none) -> Capacitor_SMD:C_0402_1005Metric; LCSC (none) -> C52923
- C3: renamed from C4; footprint (none) -> Capacitor_SMD:C_0603_1608Metric; LCSC (none) -> C59461
- C4: renamed from C3; footprint (none) -> Capacitor_SMD:C_0603_1608Metric; LCSC (none) -> C59461
- C5: footprint (none) -> Capacitor_SMD:C_0603_1608Metric; LCSC (none) -> C59461
- C7: renamed from C1; value 2.2u -> 1u; footprint (none) -> Capacitor_SMD:C_0603_1608Metric; LCSC (none) -> C15849; Rating 100V -> 50V
- J1: footprint (none) -> Connector_JST:JST_XH_S3B-XH-A_1x03_P2.50mm_Horizontal; LCSC (none) -> C48641715
- J2: renamed from J6; footprint (none) -> SparkAll:Molex_Connector_8pin_P1mm_526100872; LCSC (none) -> C588214
- J3: renamed from J2; footprint (none) -> Connector_JST:JST_XH_B2B-XH-AM_1x02_P2.50mm_Vertical; LCSC (none) -> C42391660
- J4: renamed from J7; footprint (none) -> SparkAll:Molex_Connector_8pin_P1mm_526100872; LCSC (none) -> C588214
- J5: renamed from J8; footprint (none) -> Connector_PinSocket_2.54mm:PinSocket_1x02_P2.54mm_Vertical
- R1: value 1k -> 100k; footprint (none) -> Resistor_SMD:R_0402_1005Metric; LCSC (none) -> C25741
- R2, R3, R4: value 1k -> 10k; footprint (none) -> Resistor_SMD:R_0402_1005Metric; LCSC (none) -> C25744
- R5: renamed from R6; footprint (none) -> Resistor_SMD:R_0402_1005Metric; LCSC (none) -> C25893
- R6: renamed from R5; footprint (none) -> Resistor_SMD:R_0402_1005Metric; LCSC (none) -> C25744
- R7: footprint (none) -> Resistor_SMD:R_0402_1005Metric; LCSC (none) -> C26956
- U1: LCSC (none) -> C507118
Connections:
- net +5V is gone; now on net +5VS: R1.1
- net HV_EN_3V3 is gone; now on net GNDS: R4.2
- net +36V: now also C6.1
- net +5VS: now also TP5.1
- net GND: now also C6.2, TP1.1; no longer J1.3 (Pin_3)
- net GNDS: now also J1.3 (Pin_3), R2.2, R3.2, TP2.1
- net HC_CURR: now also U1.6 (PA5)
- net HC_EN: now also U1.5 (PA4)
- net HV_CURR: now also U1.1 (PA2)
- net HV_EN: now also U1.20 (PA1); no longer R3.2, R4.1
- net HV_~{FAULT}: now also U1.2 (PA3)
- net UPDI: now also R1.2
- net 5V_NON_ISO: now reaches C4.1, C5.1, PS1.2 (+Vin), R5.1, U2.4 (VOUT)
- net 5V_NON_ISO: now also TP6.1
- net LED_OK: now reaches U1.15 (PC0)
- net LED_OK: now also D1.2 (A)
- net LED_RUN: now reaches U1.16 (PC1)
- net LED_RUN: now also D2.2 (A)
- net LED_ERR: now reaches U1.17 (PC2)
- net LED_ERR: now also D3.2 (A)
- net at U1.18 (PC3): now also TP3.1
- net at U2.1 (PGOOD): now also TP7.1
- net at R2.1: now also D1.1 (K); no longer R1.2
- net at R3.1: now also D2.1 (K); no longer R2.2
- new net: D3.1 (K), R4.1
Other:
- note added: "TODO: confirm these pinouts"
- note removed: "Currently constructed on breardboard; no PCB yet"
- note removed: "Firmware: `firmware-test-integ/` Written via SWD connector"
- note removed: "makeshift level conveter 3.3V I/O -> 5V I/O OUT: L=1.3V, H=3.7V"
- note removed: "non-isolated 5V"
- moved on the sheet: C2, J1, J2, J3, J4, J5
