File: pcb/PULSER-testboard-ctrl/PULSER-testboard-ctrl.kicad_pcb (KiCad board)
At the start: 4 copper layers, 40 x 45 mm, 32 parts, among them J1 I2C/XH, J2 Conn_01x08_Pin, J3 36V IN, J4 Conn_01x08_Pin, J5 Conn_01x02_Pin, U1 ATtiny1616-M, U2 TPSM365R6

Commit message: pulser v2 - ctrl r2 minor update (silk)
Other:
- board text added: "FLT"
- board text removed: "ERR"
Changed lines of the file:
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@@
 	(gr_line
 		(start 73.5 75.5)
-		(end 89 75.5)
+		(end 82 75.5)
 		(stroke
 			(width 0.1)
@@
 		)
 	)
-	(gr_text "ERR"
+	(gr_text "FLT"
 		(at 65.9 98.8 0)
 		(layer "F.SilkS")

Commit message: Via-stitch ctrl
Routing:
- net GNDS: vias 29 -> 59
- net GND: vias 19 -> 28
