File: pcb/pulser-ctrl/pulser-ctrl.kicad_sch (KiCad schematic)
At the start: 22 parts, among them J1 Screw_Terminal 2pin, J2 Screw_Terminal 2pin, J3 Conn_01x02_Pin, J6 Conn_01x08_Pin, U1 ADuM1200AR

Commit message: Restructure kicad filenames
Parts:
- removed C12: 22n, Capacitor_SMD:C_0805_2012Metric, symbol Device:C_Small
- removed C33, C35: 0.1u, Capacitor_SMD:C_0402_1005Metric, symbol Device:C
- removed C8: 220n, Capacitor_SMD:C_0603_1608Metric, symbol Device:C_Small
- removed C9: 1u, Capacitor_SMD:C_0805_2012Metric, symbol Device:C_Small
- removed D1: ~, SparkAll:VISHAY-SMPC, symbol Device:D_Schottky
- removed D5: Vz=100V, Diode_SMD:D_SMB, symbol Device:D_Zener
- removed D6: ~, SparkAll:TO-227A-2P, symbol Device:D_Schottky
- removed D7, D8: LED, LED_SMD:LED_0805_2012Metric, symbol Device:LED
- removed F1: 10A, Fuse:Fuse_Littelfuse-NANO2-451_453, symbol Device:Fuse
- removed J1, J2: Screw_Terminal 2pin, SparkAll:Wurth_TerminalBlock_2pin_P5mm_691137710002, symbol Connector:Screw_Terminal_01x02
- removed J3: Conn_01x02_Pin, Connector_JST:JST_XH_B2B-XH-A_1x02_P2.50mm_Vertical, symbol Connector:Conn_01x02_Pin
- removed J6: Conn_01x08_Pin, Connector_FFC-FPC:Molex_200528-0080_1x08-1MP_P1.00mm_Horizontal, symbol Connector:Conn_01x08_Pin
- removed R11: 3.3, Resistor_SMD:R_2512_6332Metric, symbol Device:R
- removed R12: 10k, Resistor_SMD:R_0402_1005Metric, symbol Device:R
- removed R16, R19: 1k, Resistor_SMD:R_0402_1005Metric, symbol Device:R
- removed R24: 1, Resistor_SMD:R_2512_6332Metric, symbol Device:R
- removed TP8: TestPoint, TestPoint:TestPoint_Pad_D1.5mm, symbol Connector:TestPoint_Small
- removed U1: ADuM1200AR, Package_SO:SOIC-8_3.9x4.9mm_P1.27mm, symbol Isolator:ADuM1200AR
- added C1, C2: 1u, Capacitor_SMD:C_0402_1005Metric, symbol Device:C_Small
- added C3, C4, C5: 22u, Capacitor_SMD:C_0603_1608Metric, symbol Device:C_Small
- added C6, C7: 1u, Capacitor_SMD:C_0603_1608Metric, symbol Device:C_Small
- added D1, D2, D3: LED, LED_SMD:LED_0603_1608Metric, symbol Device:LED
- added J1: I2C/XH, Connector_JST:JST_XH_S3B-XH-A_1x03_P2.50mm_Horizontal, symbol Connector:Conn_01x03_Socket
- added J2, J4: Conn_01x08_Pin, SparkAll:Molex_Connector_8pin_P1mm_526100872, symbol Connector:Conn_01x08_Pin
- added J3: 36V IN, Connector_JST:JST_XH_B2B-XH-AM_1x02_P2.50mm_Vertical, symbol Connector:Conn_01x02_Socket
- added J5: Conn_01x02_Pin, Connector_PinSocket_2.54mm:PinSocket_1x02_P2.54mm_Vertical, symbol Connector:Conn_01x02_Pin
- added PS1: MEE1S0505SC, Converter_DCDC:Converter_DCDC_Murata_MEE1SxxxxSC_THT, symbol Converter_DCDC:MEE1S0505SC
- added R1: 100k, Resistor_SMD:R_0402_1005Metric, symbol Device:R
- added R2, R3, R4, R6: 10k, Resistor_SMD:R_0402_1005Metric, symbol Device:R
- added R5: 40.2k, Resistor_SMD:R_0402_1005Metric, symbol Device:R
- added R7: 15.8k, Resistor_SMD:R_0402_1005Metric, symbol Device:R
- added TP1, TP2, TP3, TP5, TP6, TP7: TestPoint, TestPoint:TestPoint_Pad_D1.5mm, symbol Connector:TestPoint_Small
- added U1: ATtiny1616-M, Package_DFN_QFN:VQFN-20-1EP_3x3mm_P0.4mm_EP1.7x1.7mm, symbol MCU_Microchip_ATtiny:ATtiny1616-M
- added U2: TPSM365R6, SparkAll:TI-RDN0011A-MFG, symbol SparkAll:TPSM365R6FRDNR
Connections:
- net +36V: now also C6.1, C7.1, J3.1 (Pin_1), U2.2 (EN), U2.3 (VIN)
- net GND: now also C2.2, C4.2, C5.2, C6.2, C7.2, J3.2 (Pin_2), PS1.1 (-Vin), R6.2, R7.2, TP1.1, U2.10 (GND)
- net GNDS: now also C1.2, C3.2, J1.3 (Pin_3), J2.2 (Pin_2), J2.5 (Pin_5), J4.2 (Pin_2), J4.5 (Pin_5), J5.2 (Pin_2), PS1.3 (-Vout), R2.2, R3.2, R4.2, TP2.1, U1.21 (GND), U1.3 (GND)
- new net: TP7.1, U2.1 (PGOOD)
- new net: TP3.1, U1.18 (PC3)
- new net: D2.1 (K), R3.1
- new net: R5.2, R6.1, U2.9 (BIAS)
- new net: R7.1, U2.11 (MODE_SYNC)
- new net: C2.1, U2.8 (VCC)
- new net: D3.1 (K), R4.1
- new net: D1.1 (K), R2.1
- new net +5VS: C1.1, C3.1, J2.1 (Pin_1), J4.1 (Pin_1), PS1.4 (+Vout), R1.1, TP5.1, U1.4 (VCC)
- new net 5V_NON_ISO: C4.1, C5.1, PS1.2 (+Vin), R5.1, TP6.1, U2.4 (VOUT)
- new net HC_CURR: J4.4 (Pin_4), U1.6 (PA5)
- new net HC_EN: J4.3 (Pin_3), U1.5 (PA4)
- new net HV_CURR: J2.4 (Pin_4), U1.1 (PA2)
- new net HV_EN: J2.3 (Pin_3), U1.20 (PA1)
- new net HV_~{FAULT}: J2.6 (Pin_6), U1.2 (PA3)
- new net I2C_SCL: J1.2 (Pin_2), U1.14 (PB0)
- new net I2C_SDA: J1.1 (Pin_1), U1.13 (PB1)
- new net LED_ERR: D3.2 (A), U1.17 (PC2)
- new net LED_OK: D1.2 (A), U1.15 (PC0)
- new net LED_RUN: D2.2 (A), U1.16 (PC1)
- new net UPDI: J5.1 (Pin_1), R1.2, U1.19 (~{RESET}/PA0)
- no-connect marks 0 -> 5
Other:
- removed sheet highcurrent
- removed sheet powersupply
- note added: "RT Fsw=1MHz"
- note added: "TODO: confirm these pinouts"
- note added: "UPDI writer (5V)"
- note added: "to HC board"
- note added: "to HV board"
- note removed: "1.6W (at 8kHz pulse) target: Tj<100C 22 vias (assuming Tjc=20K/W)"
- note removed: "12V fan (max 200mA)"
- note removed: "6W target: Tj<100C 50 vias"
- note removed: "CURR (PWM) * accepted freq: 10kHz~200kHz * working range: 22%(5A) ~ 45% (10A) (0.22A/%) * setting delay: 10ms Below 22%: output current might be unstable compared to ripple Above 45%: clamped to 10A"
- note removed: "D1 protection"
- note removed: "EN"
- note removed: "PWR"
- note removed: "Snubber (R=3.3Ω, C=20nF)"
- note removed: "Thermal environment * via: 300K/W * backside-air: 1.7K/W (only where heatsink exists) * Tair=30C"
- note removed: "VCCS=3.3V or 5V current draw: <5mA"
- note removed: "fc=72Hz LPF (9kHz 50% -> 1%- ripple)"
- note removed: "min pulse width: 1us"
- note removed: "resonance damper for cable inductance"
- note removed: "stray inductance flywheel"
- title: Pulser V2 HC Board -> Pulser V2 Controller
