File: pcb/pulser-hc/powersupply.kicad_sch (KiCad schematic)
At the start: 13 parts, among them U5 LM317_DPAK, U9 TPSM365R6

Commit message: Restructure kicad filenames
Parts:
- removed C7: 0.1u, Capacitor_SMD:C_0603_1608Metric, symbol Device:C_Small
- removed C8: 1u, Capacitor_SMD:C_0603_1608Metric, symbol Device:C_Small
- removed R10: 10k, Resistor_SMD:R_0402_1005Metric, symbol Device:R
- removed R9: 110k, Resistor_SMD:R_0402_1005Metric, symbol Device:R
- removed U5: LM317_DPAK, Package_TO_SOT_SMD:TO-252-2, symbol Regulator_Linear:LM317_TO-252
- removed U9: TPSM365R6, SparkAll:TI-RDN0011A-MFG, symbol SparkAll:TPSM365R6FRDNR
- added C15, C16: 0.1u, Capacitor_SMD:C_0402_1005Metric, symbol Device:C_Small
- added R14: 110k, Resistor_SMD:R_0402_1005Metric, symbol Device:R
- added R15: 10k, Resistor_SMD:R_0402_1005Metric, symbol Device:R
- added U2: LM317_DPAK, Package_TO_SOT_SMD:TO-252-2, symbol Regulator_Linear:LM317_TO-252
- added U4: TPSM365R6, SparkAll:TI-RDN0011A-MFG, symbol SparkAll:TPSM365R6FRDNR
- R17: renamed from R14; value 270 -> 240; footprint Resistor_SMD:R_0603_1608Metric -> Resistor_SMD:R_0402_1005Metric; LCSC C22966 -> C852660; Rating (none) -> 10V
- R18: renamed from R15; value 820 -> 390; footprint Resistor_SMD:R_0603_1608Metric -> Resistor_SMD:R_0402_1005Metric; LCSC C23253 -> C137997; Rating (none) -> 10V
Connections:
- net 12VOUT: now also C15.2, R14.1, U2.3 (VI), U4.4 (VOUT)
- net 36VIN: now also U4.2 (EN), U4.3 (VIN)
- net GND: now also C15.1, C16.1, R15.2, U4.10 (GND), U4.11 (MODE_SYNC)
- net at TP12.1: now also U4.1 (PGOOD)
- net at R17.2, R18.1: now also U2.1 (ADJ)
- net at C26.1: now also U4.8 (VCC)
- net 5VOUT renamed 3V3OUT
- net 3V3OUT: now also C16.2, U2.2 (VO)
- new net: R14.2, R15.1, U4.9 (BIAS)
Other:
- note added: "3.3V"
- title: Pulser V2 HV Test Board -> Pulser V2 HC Board
- moved on the sheet: R17, R18
