File: pcb/pulser-hc/pulser-hc.kicad_pcb (KiCad board)
At the start: 4 copper layers, 100 x 50 mm, 86 parts, among them J1 Screw_Terminal 2pin, J2 Screw_Terminal 2pin, J3 Conn_01x02_Pin, J6 Conn_01x08_Pin, Q1 N-ch, Vds>=60V, low Qgs, Q2 N-ch, Vds>=60V, low Rds, U1 ADuM1200AR, U2 LM317_DPAK, U3 LT3763, U4 TPSM365R6

Commit message: Via-stitch HC (10mm) & export as r3
Parts:
- moved C3 0.80 mm to (82.5, 86.5)
- moved R3 0.80 mm to (83.0, 85.0)
- moved R4 0.80 mm to (82.0, 85.0)
Routing:
- net +3V3: track 38.9 -> 37.6 mm
- net Net-(U3-FB): track 52.5 -> 53.3 mm
- net GNDS: vias 4 -> 12
- net GND: vias 189 -> 251
Other:
- board text added: "I+ 36V"
- board text removed: "I+(36V)"
