File: pcb/pulser-hc/pulser-hc.kicad_sch (KiCad schematic)
At the start: 31 parts, among them J1 I2C/XH, J2 Conn_01x08_Pin, J3 36V IN, J4 Conn_01x08_Pin, J5 Conn_01x02_Pin, U1 ATtiny1616-M, U2 TPSM365R6

Commit message: Restructure kicad filenames
Parts:
- removed C1, C2: 1u, Capacitor_SMD:C_0402_1005Metric, symbol Device:C_Small
- removed C3, C4, C5: 22u, Capacitor_SMD:C_0603_1608Metric, symbol Device:C_Small
- removed C6, C7: 1u, Capacitor_SMD:C_0603_1608Metric, symbol Device:C_Small
- removed D1, D2, D3: LED, LED_SMD:LED_0603_1608Metric, symbol Device:LED
- removed J1: I2C/XH, Connector_JST:JST_XH_S3B-XH-A_1x03_P2.50mm_Horizontal, symbol Connector:Conn_01x03_Socket
- removed J2, J4: Conn_01x08_Pin, SparkAll:Molex_Connector_8pin_P1mm_526100872, symbol Connector:Conn_01x08_Pin
- removed J3: 36V IN, Connector_JST:JST_XH_B2B-XH-AM_1x02_P2.50mm_Vertical, symbol Connector:Conn_01x02_Socket
- removed J5: Conn_01x02_Pin, Connector_PinSocket_2.54mm:PinSocket_1x02_P2.54mm_Vertical, symbol Connector:Conn_01x02_Pin
- removed PS1: MEE1S0505SC, Converter_DCDC:Converter_DCDC_Murata_MEE1SxxxxSC_THT, symbol Converter_DCDC:MEE1S0505SC
- removed R1: 100k, Resistor_SMD:R_0402_1005Metric, symbol Device:R
- removed R2, R3, R4, R6: 10k, Resistor_SMD:R_0402_1005Metric, symbol Device:R
- removed R5: 40.2k, Resistor_SMD:R_0402_1005Metric, symbol Device:R
- removed R7: 15.8k, Resistor_SMD:R_0402_1005Metric, symbol Device:R
- removed TP1, TP2, TP3, TP5, TP6, TP7: TestPoint, TestPoint:TestPoint_Pad_D1.5mm, symbol Connector:TestPoint_Small
- removed U1: ATtiny1616-M, Package_DFN_QFN:VQFN-20-1EP_3x3mm_P0.4mm_EP1.7x1.7mm, symbol MCU_Microchip_ATtiny:ATtiny1616-M
- removed U2: TPSM365R6, SparkAll:TI-RDN0011A-MFG, symbol SparkAll:TPSM365R6FRDNR
- added C12: 22n, Capacitor_SMD:C_0805_2012Metric, symbol Device:C_Small
- added C33, C35: 0.1u, Capacitor_SMD:C_0402_1005Metric, symbol Device:C
- added C8: 220n, Capacitor_SMD:C_0603_1608Metric, symbol Device:C_Small
- added C9: 1u, Capacitor_SMD:C_0805_2012Metric, symbol Device:C_Small
- added D1: ~, SparkAll:VISHAY-SMPC, symbol Device:D_Schottky
- added D5: Vz=100V, Diode_SMD:D_SMB, symbol Device:D_Zener
- added D6: ~, SparkAll:TO-227A-2P, symbol Device:D_Schottky
- added D7, D8: LED, LED_SMD:LED_0805_2012Metric, symbol Device:LED
- added F1: 10A, Fuse:Fuse_Littelfuse-NANO2-451_453, symbol Device:Fuse
- added J1, J2: Screw_Terminal 2pin, SparkAll:Wurth_TerminalBlock_2pin_P5mm_691137710002, symbol Connector:Screw_Terminal_01x02
- added J3: Conn_01x02_Pin, Connector_JST:JST_XH_B2B-XH-A_1x02_P2.50mm_Vertical, symbol Connector:Conn_01x02_Pin
- added J6: Conn_01x08_Pin, Connector_FFC-FPC:Molex_200528-0080_1x08-1MP_P1.00mm_Horizontal, symbol Connector:Conn_01x08_Pin
- added R11: 3.3, Resistor_SMD:R_2512_6332Metric, symbol Device:R
- added R12: 10k, Resistor_SMD:R_0402_1005Metric, symbol Device:R
- added R16, R19: 1k, Resistor_SMD:R_0402_1005Metric, symbol Device:R
- added R24: 1, Resistor_SMD:R_2512_6332Metric, symbol Device:R
- added TP8: TestPoint, TestPoint:TestPoint_Pad_D1.5mm, symbol Connector:TestPoint_Small
- added U1: ADuM1200AR, Package_SO:SOIC-8_3.9x4.9mm_P1.27mm, symbol Isolator:ADuM1200AR
Connections:
- net +36V: now also C9.1, F1.2
- net GND: now also C35.2, C8.1, D5.2 (A), D6.2 (A), J1.1 (Pin_1), J2.2 (Pin_2), J3.2 (Pin_2), R11.2, R16.1, R19.1, R24.2, U1.5 (GND2)
- net GNDS: now also C33.2, J6.2 (Pin_2), J6.5 (Pin_5), U1.4 (GND1)
- new net: D7.1 (K), R16.2
- new net: F1.1, J1.2 (Pin_2)
- new net: D8.1 (K), R19.2
- new net: C12.1, R11.1
- new net: C12.2, D1.1 (K), D5.1 (K), D6.1 (K), J2.1 (Pin_1)
- new net: C9.2, R24.1
- new net: R12.1, U1.6 (VOB)
- new net +12V: J3.1 (Pin_1)
- new net +3V3: C35.1, D7.2 (A), U1.8 (VDD2)
- new net CURR_CTRL: C8.2, R12.2, TP8.1
- new net CURR_S: J6.4 (Pin_4), U1.3 (VIB)
- new net EN: D8.2 (A), U1.7 (VOA)
- new net EN_S: J6.3 (Pin_3), U1.2 (VIA)
- new net VCCS: C33.1, J6.1 (Pin_1), U1.1 (VDD1)
- new net highcurrent/VOUT: D1.2 (A)
- no-connect marks 5 -> 0
Other:
- added sheet highcurrent (highcurrent.kicad_sch)
- added sheet powersupply (powersupply.kicad_sch)
- note added: "1.6W (at 8kHz pulse) target: Tj<100C 22 vias (assuming Tjc=20K/W)"
- note added: "12V fan (max 200mA)"
- note added: "6W target: Tj<100C 50 vias"
- note added: "CURR (PWM) * accepted freq: 10kHz~200kHz * working range: 22%(5A) ~ 45% (10A) (0.22A/%) * setting delay: 10ms Below 22%: output current might be unstable compared to ripple Above 45%: clamped to 10A"
- note added: "D1 protection"
- note added: "EN"
- note added: "PWR"
- note added: "Snubber (R=3.3Ω, C=20nF)"
- note added: "Thermal environment * via: 300K/W * backside-air: 1.7K/W (only where heatsink exists) * Tair=30C"
- note added: "VCCS=3.3V or 5V current draw: <5mA"
- note added: "fc=72Hz LPF (9kHz 50% -> 1%- ripple)"
- note added: "min pulse width: 1us"
- note added: "resonance damper for cable inductance"
- note added: "stray inductance flywheel"
- note removed: "RT Fsw=1MHz"
- note removed: "TODO: confirm these pinouts"
- note removed: "UPDI writer (5V)"
- note removed: "to HC board"
- note removed: "to HV board"
- title: Pulser V2 Controller -> Pulser V2 HC Board

Commit message: hc: Add missing LCSC no & reexport
Parts:
- J3: LCSC (none) -> C158012
Changed lines of the file:
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@@
+			)
+		)
+		(property "LCSC" "C158012"
+			(at 237.49 80.01 0)
+			(effects
+				(font
+					(size 1.27 1.27)
+				)
+				(hide yes)
 			)
 		)
