File: pcb/pulser-hv/boost.kicad_sch (KiCad schematic)
At the start: 12 parts, among them U6 LT8365

Commit message: Restructure kicad filenames
Other:
- title: Pulser V2 HV Test Board -> Pulser V2 HV Board
Changed lines of the file:
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@@
 	(paper "A4")
 	(title_block
-		(title "Pulser V2 HV Test Board")
+		(title "Pulser V2 HV Board")
 		(date "2026-07-01")
 		(rev "4")
@@
 		)
 		(instances
-			(project "PULSER-testboard-hv"
+			(project "pulser-hv"
 				(path "/853931f0-9d2b-49ab-aae3-2a7153967e0f/bd7f0006-b363-44d9-a542-e4fe897a7941"
 					(reference "#PWR029")
@@
 		)
 		(instances
-			(project "PULSER-testboard-hv"
+			(project "pulser-hv"
 				(path "/853931f0-9d2b-49ab-aae3-2a7153967e0f/bd7f0006-b363-44d9-a542-e4fe897a7941"
 					(reference "C12")
@@
 		)
 		(instances
-			(project "PULSER-testboard-hv"
+			(project "pulser-hv"
 				(path "/853931f0-9d2b-49ab-aae3-2a7153967e0f/bd7f0006-b363-44d9-a542-e4fe897a7941"
 					(reference "L1")
@@
 		)
 		(instances
-			(project "PULSER-testboard-hv"
+			(project "pulser-hv"
 				(path "/853931f0-9d2b-49ab-aae3-2a7153967e0f/bd7f0006-b363-44d9-a542-e4fe897a7941"
 					(reference "C9")
@@
 		)
 		(instances
-			(project "PULSER-testboard-hv"
+			(project "pulser-hv"
 				(path "/853931f0-9d2b-49ab-aae3-2a7153967e0f/bd7f0006-b363-44d9-a542-e4fe897a7941"
 					(reference "U6")
@@
 		)
 		(instances
-			(project "PULSER-testboard-hv"
+			(project "pulser-hv"
 				(path "/853931f0-9d2b-49ab-aae3-2a7153967e0f/bd7f0006-b363-44d9-a542-e4fe897a7941"
 					(reference "C11")
@@
 		)
 		(instances
-			(project "PULSER-testboard-hv"
+			(project "pulser-hv"
 				(path "/853931f0-9d2b-49ab-aae3-2a7153967e0f/bd7f0006-b363-44d9-a542-e4fe897a7941"
 					(reference "R17")
@@
 		)
 		(instances
-			(project "PULSER-testboard-hv"
+			(project "pulser-hv"
 				(path "/853931f0-9d2b-49ab-aae3-2a7153967e0f/bd7f0006-b363-44d9-a542-e4fe897a7941"
 					(reference "C13")
@@
 		)
 		(instances
-			(project "PULSER-testboard-hv"
+			(project "pulser-hv"
 				(path "/853931f0-9d2b-49ab-aae3-2a7153967e0f/bd7f0006-b363-44d9-a542-e4fe897a7941"
 					(reference "R19")
@@
 		)
 		(instances
-			(project "PULSER-testboard-hv"
+			(project "pulser-hv"
 				(path "/853931f0-9d2b-49ab-aae3-2a7153967e0f/bd7f0006-b363-44d9-a542-e4fe897a7941"
 					(reference "C10")
@@
 		)
 		(instances
-			(project "PULSER-testboard-hv"
+			(project "pulser-hv"
 				(path "/853931f0-9d2b-49ab-aae3-2a7153967e0f/bd7f0006-b363-44d9-a542-e4fe897a7941"
 					(reference "D2")
@@
 		)
 		(instances
-			(project "PULSER-testboard-hv"
+			(project "pulser-hv"
 				(path "/853931f0-9d2b-49ab-aae3-2a7153967e0f/bd7f0006-b363-44d9-a542-e4fe897a7941"
 					(reference "R18")
@@
 		)
 		(instances
-			(project "PULSER-testboard-hv"
+			(project "pulser-hv"
 				(path "/853931f0-9d2b-49ab-aae3-2a7153967e0f/bd7f0006-b363-44d9-a542-e4fe897a7941"
 					(reference "R16")
