File: pcb/pulser-hv/powersupply.kicad_sch (KiCad schematic)
At the start: 13 parts, among them U2 LM317_DPAK, U4 TPSM365R6

Commit message: Restructure kicad filenames
Parts:
- removed C15, C16: 0.1u, Capacitor_SMD:C_0402_1005Metric, symbol Device:C_Small
- removed R14: 110k, Resistor_SMD:R_0402_1005Metric, symbol Device:R
- removed R15: 10k, Resistor_SMD:R_0402_1005Metric, symbol Device:R
- removed U2: LM317_DPAK, Package_TO_SOT_SMD:TO-252-2, symbol Regulator_Linear:LM317_TO-252
- removed U4: TPSM365R6, SparkAll:TI-RDN0011A-MFG, symbol SparkAll:TPSM365R6FRDNR
- added C7: 0.1u, Capacitor_SMD:C_0603_1608Metric, symbol Device:C_Small
- added C8: 1u, Capacitor_SMD:C_0603_1608Metric, symbol Device:C_Small
- added R10: 10k, Resistor_SMD:R_0402_1005Metric, symbol Device:R
- added R9: 110k, Resistor_SMD:R_0402_1005Metric, symbol Device:R
- added U5: LM317_DPAK, Package_TO_SOT_SMD:TO-252-2, symbol Regulator_Linear:LM317_TO-252
- added U9: TPSM365R6, SparkAll:TI-RDN0011A-MFG, symbol SparkAll:TPSM365R6FRDNR
- R14: renamed from R17; value 240 -> 270; footprint Resistor_SMD:R_0402_1005Metric -> Resistor_SMD:R_0603_1608Metric; LCSC C852660 -> C22966; Rating 10V -> (none)
- R15: renamed from R18; value 390 -> 820; footprint Resistor_SMD:R_0402_1005Metric -> Resistor_SMD:R_0603_1608Metric; LCSC C137997 -> C23253; Rating 10V -> (none)
Connections:
- net 12VOUT: now also C7.2, R9.1, U5.3 (VI), U9.4 (VOUT)
- net 36VIN: now also U9.2 (EN), U9.3 (VIN)
- net GND: now also C7.1, C8.1, R10.2, U9.10 (GND), U9.11 (MODE_SYNC)
- net at TP12.1: now also U9.1 (PGOOD)
- net at R14.2, R15.1: now also U5.1 (ADJ)
- net at C26.1: now also U9.8 (VCC)
- net 3V3OUT renamed 5VOUT
- net 5VOUT: now also C8.2, U5.2 (VO)
- new net: R10.1, R9.2, U9.9 (BIAS)
Other:
- note removed: "3.3V"
- title: Pulser V2 HC Board -> Pulser V2 HV Board
- moved on the sheet: R14, R15
