File: pcb/pulser-hv/pulse.kicad_sch (KiCad schematic)
At the start: 10 parts, among them J5 Conn_01x02_Socket, U11 ATtiny1616-M

Commit message: Restructure kicad filenames
Other:
- title: Pulser V2 HV Test Board -> Pulser V2 HV Board
Changed lines of the file:
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@@
 	(paper "A4")
 	(title_block
-		(title "Pulser V2 HV Test Board")
+		(title "Pulser V2 HV Board")
 		(date "2026-07-01")
 		(rev "4")
@@
 		)
 		(instances
-			(project "PULSER-testboard-hv"
+			(project "pulser-hv"
 				(path "/853931f0-9d2b-49ab-aae3-2a7153967e0f/a58ab8a7-d919-4bb1-bcb6-a07722db020b"
 					(reference "D4")
@@
 		)
 		(instances
-			(project "PULSER-testboard-hv"
+			(project "pulser-hv"
 				(path "/853931f0-9d2b-49ab-aae3-2a7153967e0f/a58ab8a7-d919-4bb1-bcb6-a07722db020b"
 					(reference "#PWR054")
@@
 		)
 		(instances
-			(project "PULSER-testboard-hv"
+			(project "pulser-hv"
 				(path "/853931f0-9d2b-49ab-aae3-2a7153967e0f/a58ab8a7-d919-4bb1-bcb6-a07722db020b"
 					(reference "TP11")
@@
 		)
 		(instances
-			(project "PULSER-testboard-hv"
+			(project "pulser-hv"
 				(path "/853931f0-9d2b-49ab-aae3-2a7153967e0f/a58ab8a7-d919-4bb1-bcb6-a07722db020b"
 					(reference "R7")
@@
 		)
 		(instances
-			(project "PULSER-testboard-hv"
+			(project "pulser-hv"
 				(path "/853931f0-9d2b-49ab-aae3-2a7153967e0f/a58ab8a7-d919-4bb1-bcb6-a07722db020b"
 					(reference "#PWR032")
@@
 		)
 		(instances
-			(project "PULSER-testboard-hv"
+			(project "pulser-hv"
 				(path "/853931f0-9d2b-49ab-aae3-2a7153967e0f/a58ab8a7-d919-4bb1-bcb6-a07722db020b"
 					(reference "#PWR019")
@@
 		)
 		(instances
-			(project "PULSER-testboard-hv"
+			(project "pulser-hv"
 				(path "/853931f0-9d2b-49ab-aae3-2a7153967e0f/a58ab8a7-d919-4bb1-bcb6-a07722db020b"
 					(reference "#PWR031")
@@
 		)
 		(instances
-			(project "PULSER-testboard-hv"
+			(project "pulser-hv"
 				(path "/853931f0-9d2b-49ab-aae3-2a7153967e0f/a58ab8a7-d919-4bb1-bcb6-a07722db020b"
 					(reference "#PWR048")
@@
 		)
 		(instances
-			(project "PULSER-testboard-hv"
+			(project "pulser-hv"
 				(path "/853931f0-9d2b-49ab-aae3-2a7153967e0f/a58ab8a7-d919-4bb1-bcb6-a07722db020b"
 					(reference "#PWR034")
@@
 		)
 		(instances
-			(project "PULSER-testboard-hv"
+			(project "pulser-hv"
 				(path "/853931f0-9d2b-49ab-aae3-2a7153967e0f/a58ab8a7-d919-4bb1-bcb6-a07722db020b"
 					(reference "C21")
@@
 		)
 		(instances
-			(project "PULSER-testboard-hv"
+			(project "pulser-hv"
 				(path "/853931f0-9d2b-49ab-aae3-2a7153967e0f/a58ab8a7-d919-4bb1-bcb6-a07722db020b"
 					(reference "#PWR033")
@@
 		)
 		(instances
-			(project "PULSER-testboard-hv"
+			(project "pulser-hv"
 				(path "/853931f0-9d2b-49ab-aae3-2a7153967e0f/a58ab8a7-d919-4bb1-bcb6-a07722db020b"
 					(reference "#PWR035")
@@
 		)
 		(instances
-			(project "PULSER-testboard-hv"
+			(project "pulser-hv"
 				(path "/853931f0-9d2b-49ab-aae3-2a7153967e0f/a58ab8a7-d919-4bb1-bcb6-a07722db020b"
 					(reference "R21")
@@
 		)
 		(instances
-			(project "PULSER-testboard-hv"
+			(project "pulser-hv"
 				(path "/853931f0-9d2b-49ab-aae3-2a7153967e0f/a58ab8a7-d919-4bb1-bcb6-a07722db020b"
 					(reference "D7")
@@
 		)
 		(instances
-			(project "PULSER-testboard-hv"
+			(project "pulser-hv"
 				(path "/853931f0-9d2b-49ab-aae3-2a7153967e0f/a58ab8a7-d919-4bb1-bcb6-a07722db020b"
 					(reference "R2")
@@
 		)
 		(instances
-			(project "PULSER-testboard-hv"
+			(project "pulser-hv"
 				(path "/853931f0-9d2b-49ab-aae3-2a7153967e0f/a58ab8a7-d919-4bb1-bcb6-a07722db020b"
 					(reference "#PWR030")

Commit message: hv: add missing lcsc
Parts:
- D7: LCSC (none) -> C2286
Changed lines of the file:
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@@
 			)
 		)
-		(property "LCSC" ""
+		(property "LCSC" "C2286"
 			(at 59.69 81.28 90)
 			(effects
