File: pcb/pulser-hv/pulser-hv.kicad_pcb (KiCad board)
At the start: 4 copper layers, 100 x 50 mm, 75 parts, among them J1 Screw_Terminal 2pin, J2 Screw_Terminal 2pin, J3 Conn_01x02_Pin, J5 Conn_01x02_Socket, J6 Conn_01x08_Pin, Q1 Q_NMOS_GDS, U1 ADuM1200AR, U11 ATtiny1616-M, U2 INA281A2, U3 LTC7001, U4 TLV3201, U5 LM317_DPAK, U6 LT8365, U7 ADuM1200AR, U9 TPSM365R6

Commit message: Via-stitch HV (10mm) & export as r4
Parts:
- moved C29 0.42 mm to (108.7, 54.1)
- moved C30 0.42 mm to (108.7, 55.6)
Routing:
- net +5V: track 87.2 -> 72.5 mm
- net GNDS: vias 6 -> 10
- net GND: vias 256 -> 317

Commit message: hv: add missing lcsc
Connections:
- R4 pad 3: GND -> (no net)
Changed lines of the file:
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@@
 			)
 		)
+		(property "LCSC" "C15219"
+			(at 0 0 90)
+			(unlocked yes)
+			(layer "F.Fab")
+			(hide yes)
+			(effects
+				(font
+					(size 1 1)
+					(thickness 0.15)
+				)
+			)
+		)
 		(property ki_fp_filters "SOIC*3.9x4.9mm*P1.27mm*")
 		(sheetname "/")
@@
 			)
 		)
-		(property "LCSC" ""
+		(property "LCSC" "C165983"
 			(at 0 0 180)
 			(unlocked yes)
@@
 			)
 		)
-		(property "LCSC" ""
+		(property "LCSC" "C2286"
 			(at 0 0 180)
 			(unlocked yes)
@@
 			)
 		)
+		(property "LCSC" "C15219"
+			(at 0 0 270)
+			(unlocked yes)
+			(layer "F.Fab")
+			(hide yes)
+			(effects
+				(font
+					(size 1 1)
+					(thickness 0.15)
+				)
+			)
+		)
 		(property ki_fp_filters "SOIC*3.9x4.9mm*P1.27mm*")
 		(sheetname "/")
@@
 			(size 8.26 6.9)
 			(layers "F.Cu" "F.Mask")
-			(net 1 "GND")
 			(solder_mask_margin 0.102)
 		)

Commit message: hv: Fix TO263-resistor footprint & rework PCB & export
Parts:
- R4: footprint SparkAll:Bourns-TO508P1229X317-3N -> SparkAll:RESI-TO263
- moved TP5 11.0 mm to (102.0, 95.0)
- moved TP3 7.70 mm to (76.2, 94.5)
- moved C1 6.06 mm to (94.1, 79.8)
- moved C2 6.06 mm to (100.7, 83.2)
- moved C4 6.06 mm to (103.4, 90.6)
- moved D6 6.06 mm to (99.8, 90.8)
- moved C3 6.06 mm to (95.3, 89.8)
- moved U3 6.06 mm to (101.1, 87.8)
- moved Q1 5.93 mm to (93.0, 84.8)
- moved D5 5.74 mm to (84.8, 83.5)
- moved R1 5.20 mm to (83.3, 91.2)
- moved C5 4.70 mm to (81.2, 96.2)
- moved U2 4.70 mm to (84.1, 96.1)
- moved D2 3.55 mm to (87.9, 64.1)
- moved C10 3.55 mm to (87.6, 59.4)
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Connections:
- R4 pad 3: (no net) -> GND
Routing:
- net +36V: track 35.2 -> 15.0 mm, vias 2 -> 5
- net /Boost Converter/VOUT: track 56.0 -> 35.9 mm
- net Net-(D5-K): track 32.5 -> 18.7 mm
- net Net-(U2-Vin-): track 16.4 -> 9.77 mm
- net /GATE: track 57.5 -> 51.1 mm
- net Net-(U2-OUT): track 36.1 -> 31.4 mm
- net Net-(D1-A): track 16.9 -> 21.2 mm
- net +12V: track 40.7 -> 36.8 mm
- net Net-(J1-Pin_2): track 5.94 -> 9.60 mm
- net Net-(D1-K): track 13.7 -> 14.9 mm
- net Net-(D6-K): track 11.4 -> 12.2 mm
- net GND: vias 317 -> 334
Other:
- board text added: "I+ 36V"
- board text removed: "I+(36V)"
