File: pcb/pulser-hv/pulser-hv.kicad_sch (KiCad schematic)
At the start: 39 parts, among them J1 Screw_Terminal 2pin, J2 Screw_Terminal 2pin, J3 Conn_01x02_Pin, J6 Conn_01x08_Pin, Q1 Q_NMOS_GDS, U1 ADuM1200AR, U2 INA281A2, U3 LTC7001, U4 TLV3201, U7 ADuM1200AR

Commit message: Restructure kicad filenames
Other:
- title: Pulser V2 HV Test Board -> Pulser V2 HV Board

Commit message: hv: Add missing lcsc no & reexport
Parts:
- J3: LCSC (none) -> C158012
Changed lines of the file:
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@@
+			)
+		)
+		(property "LCSC" "C158012"
+			(at 261.62 80.01 0)
+			(effects
+				(font
+					(size 1.27 1.27)
+				)
+				(hide yes)
 			)
 		)

Commit message: hv: add missing lcsc
Parts:
- D3: LCSC (none) -> C165983
- U1, U7: LCSC (none) -> C15219
Changed lines of the file:
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@@
 			)
 		)
-		(property "LCSC" ""
+		(property "LCSC" "C165983"
 			(at 223.52 80.01 90)
 			(effects
@@
 			)
 		)
+		(property "LCSC" "C15219"
+			(at 54.61 140.97 0)
+			(effects
+				(font
+					(size 1.27 1.27)
+				)
+				(hide yes)
+			)
+		)
 		(pin "3"
 		)
@@
 			(at 54.61 107.95 0)
 			(effects
+				(font
+					(size 1.27 1.27)
+				)
+				(hide yes)
+			)
+		)
+		(property "LCSC" "C15219"
+			(at 54.61 107.95 0)
+			(effects

Commit message: hv: Fix TO263-resistor footprint & rework PCB & export
Parts:
- R4: footprint SparkAll:Bourns-TO508P1229X317-3N -> SparkAll:RESI-TO263
Changed lines of the file:
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@@
 			)
 		)
-		(property "Footprint" "SparkAll:Bourns-TO508P1229X317-3N"
+		(property "Footprint" "SparkAll:RESI-TO263"
 			(at 214.63 37.592 90)
 			(effects
